File: board/hdmi2usb.sch (KiCad schematic (older format))
At the start: 0 parts

Commit message: Issue #336
Changed lines of the file:
@@
 Sheet 1 7
 Title ""
-Date "4 jul 2013"
+Date "5 jul 2013"
 Rev ""
 Comp ""
@@
 F0 "hdmi" 50
 F1 "hdmi.sch" 50
-F2 "TMDS-RX-2_P" B L 8400 4550 60
-F3 "TMDS-RX-1_P" B L 8400 4750 60
-F4 "TMDS-RX-0_P" B L 8400 4950 60
-F5 "TMDS-RX-2_N" B L 8400 4650 60
-F6 "TMDS-RX-1_N" B L 8400 4850 60
-F7 "TMDS-RX-0_N" B L 8400 5050 60
-F8 "TMDS-RX-CLK_P" B L 8400 4350 60
-F9 "TMDS-RX-CLK_N" B L 8400 4450 60
-F10 "TMDS-RX-SCL" B L 8400 5150 60
-F11 "TMDS-RX-SDA" B L 8400 5250 60
-F12 "JA-D2_P" B L 8400 3700 60
-F13 "JA-D2_N" B L 8400 3600 60
-F14 "JA-D1_P" B L 8400 3900 60
-F15 "JA-D1_N" B L 8400 3800 60
-F16 "JA-D0_P" B L 8400 4100 60
-F17 "JA-D0_N" B L 8400 4000 60
-F18 "JA-CLK_P" B L 8400 3400 60
-F19 "JA-CLK_N" B L 8400 3500 60
-$EndSheet
-Wire Wire Line
-	7950 2650 8400 2650
-Wire Wire Line
-	7950 2550 8400 2550
-Wire Wire Line
-	7950 2450 8400 2450
-Wire Wire Line
-	7950 2350 8400 2350
-Wire Wire Line
-	7950 2250 8400 2250
-Wire Wire Line
-	7950 2150 8400 2150
-Wire Wire Line
-	7950 2050 8400 2050
-Wire Wire Line
-	7950 1950 8400 1950
-Wire Wire Line
-	7950 1850 8400 1850
-Wire Wire Line
-	7950 1750 8400 1750
-Wire Wire Line
-	7950 1650 8400 1650
-Wire Wire Line
-	7950 1550 8400 1550
-Wire Wire Line
-	7950 1450 8400 1450
-Wire Wire Line
-	7950 1350 8400 1350
-Wire Wire Line
-	7950 1250 8400 1250
-Wire Wire Line
-	7950 1150 8400 1150
+F2 "TMDS-RX1-2_P" B L 8400 4550 60
+F3 "TMDS-RX1-1_P" B L 8400 4750 60
+F4 "TMDS-RX1-0_P" B L 8400 4950 60
+F5 "TMDS-RX1-2_N" B L 8400 4650 60
+F6 "TMDS-RX1-1_N" B L 8400 4850 60
+F7 "TMDS-RX1-0_N" B L 8400 5050 60
+F8 "TMDS-RX1-CLK_P" B L 8400 4350 60
+F9 "TMDS-RX1-CLK_N" B L 8400 4450 60
+F10 "TMDS-RX1-SCL" B L 8400 5150 60
+F11 "TMDS-RX1-SDA" B L 8400 5250 60
+F12 "TMDS-TX1-2_P" B L 8400 3400 60
+F13 "TMDS-TX1-1_P" B L 8400 3600 60
+F14 "TMDS-TX1-0_P" B L 8400 3800 60
+F15 "TMDS-TX1-2_N" B L 8400 3500 60
+F16 "TMDS-TX1-1_N" B L 8400 3700 60
+F17 "TMDS-TX1-0_N" B L 8400 3900 60
+F18 "TMDS-TX1-CLK_P" B L 8400 4000 60
+F19 "TMDS-TX1-CLK_N" B L 8400 4100 60
+$EndSheet
+Wire Wire Line
+	7900 2650 8400 2650
+Wire Wire Line
+	7900 2550 8400 2550
+Wire Wire Line
+	7900 2450 8400 2450
+Wire Wire Line
+	7900 2350 8400 2350
+Wire Wire Line
+	7900 2250 8400 2250
+Wire Wire Line
+	7900 2150 8400 2150
+Wire Wire Line
+	7900 2050 8400 2050
+Wire Wire Line
+	7900 1950 8400 1950
+Wire Wire Line
+	7900 1850 8400 1850
+Wire Wire Line
+	7900 1750 8400 1750
+Wire Wire Line
+	7900 1650 8400 1650
+Wire Wire Line
+	7900 1550 8400 1550
+Wire Wire Line
+	7900 1450 8400 1450
+Wire Wire Line
+	7900 1350 8400 1350
+Wire Wire Line
+	7900 1250 8400 1250
+Wire Wire Line
+	7900 1150 8400 1150
 Wire Bus Line
-	7950 950  8400 950
+	7900 950  8400 950
 Wire Bus Line
-	7950 850  8400 850
+	7900 850  8400 850
 Wire Wire Line
 	5850 1900 5850 2000
@@
 Wire Wire Line
 	5850 5600 4250 5600
+Wire Wire Line
+	7900 3400 8400 3400
+Wire Wire Line
+	7900 3500 8400 3500
+Wire Wire Line
+	7900 3600 8400 3600
+Wire Wire Line
+	7900 3700 8400 3700
+Wire Wire Line
+	7900 3800 8400 3800
+Wire Wire Line
+	7900 3900 8400 3900
+Wire Wire Line
+	7900 4000 8400 4000
+Wire Wire Line
+	7900 4100 8400 4100
+Wire Wire Line
+	7900 4350 8400 4350
+Wire Wire Line
+	7900 4450 8400 4450
+Wire Wire Line
+	7900 4550 8400 4550
+Wire Wire Line
+	7900 4650 8400 4650
+Wire Wire Line
+	7900 4750 8400 4750
+Wire Wire Line
+	7900 4850 8400 4850
+Wire Wire Line
+	7900 4950 8400 4950
+Wire Wire Line
+	8400 5050 7900 5050
+Wire Wire Line
+	7900 5150 8400 5150
+Wire Wire Line
+	8400 5250 7900 5250
 $Sheet
 S 5850 700  2050 5650
@@
 F26 "EXP-IO12_N" B L 5850 4000 60
 F27 "EXP-IO12_P" B L 5850 3900 60
-F28 "JA-CLK_P" B R 7900 3400 60
-F29 "JA-CLK_N" B R 7900 3500 60
-F30 "EXP-IO13_P" B L 5850 4100 60
-F31 "EXP-IO13_N" B L 5850 4200 60
-F32 "EXP-IO14_P" B L 5850 4300 60
-F33 "EXP-IO14_N" B L 5850 4400 60
-F34 "JA-D2_N" B R 7900 3600 60
-F35 "JA-D2_P" B R 7900 3700 60
-F36 "JA-D1_N" B R 7900 3800 60
-F37 "JA-D1_P" B R 7900 3900 60
-F38 "JA-D0_N" B R 7900 4000 60
-F39 "JA-D0_P" B R 7900 4100 60
-F40 "EXP-IO15_P" B L 5850 4500 60
-F41 "EXP-IO15_N" B L 5850 4600 60
-F42 "EXP-IO16_P" B L 5850 4700 60
-F43 "EXP-IO16_N" B L 5850 4800 60
-F44 "EXP-IO17_N" B L 5850 4900 60
-F45 "EXP-IO17_P" B L 5850 5000 60
-F46 "EXP-IO18_P" B L 5850 5100 60
-F47 "EXP-IO18_N" B L 5850 5200 60
-F48 "EXP-IO19_P" B L 5850 5300 60
-F49 "EXP-IO19_N" B L 5850 5400 60
-F50 "EXP-IO2_P" B L 5850 2000 60
-F51 "EXP-IO2_N" B L 5850 1900 60
-F52 "EXP-IO20_N" B L 5850 5600 60
-F53 "EXP-IO20_P" B L 5850 5500 60
-F54 "EXP-IO3_N" B L 5850 2200 60
-F55 "EXP-IO3_P" B L 5850 2100 60
-F56 "EXP-IO4_N" B L 5850 2400 60
-F57 "EXP-IO4_P" B L 5850 2300 60
-F58 "EXP-IO5_N" B L 5850 2600 60
-F59 "EXP-IO5_P" B L 5850 2500 60
-F60 "EXP-IO6_N" B L 5850 2800 60
-F61 "EXP-IO6_P" B L 5850 2700 60
-F62 "EXP-IO7_N" B L 5850 3000 60
-F63 "EXP-IO7_P" B L 5850 2900 60
-F64 "EXP-IO8_N" B L 5850 3200 60
-F65 "EXP-IO8_P" B L 5850 3100 60
-F66 "EXP-IO9_N" B L 5850 3400 60
-F67 "EXP-IO9_P" B L 5850 3300 60
-F68 "TMDS-RX-CLK_P" B R 7900 4350 60
-F69 "TMDS-RX-CLK_N" B R 7900 4450 60
-F70 "TMDS-RX-2_P" B R 7900 4550 60
-F71 "TMDS-RX-2_N" B R 7900 4650 60
-F72 "TMDS-RX-0_P" B R 7900 4950 60
-F73 "TMDS-RX-0_N" B R 7900 5050 60
-F74 "TMDS-RX-1_P" B R 7900 4750 60
-F75 "TMDS-RX-1_N" B R 7900 4850 60
-F76 "TMDS-RX-SCL" B R 7900 5150 60
-F77 "TMDS-RX-SDA" B R 7900 5250 60
-F78 "TCK" B L 5850 5700 60
-F79 "TDO-USB/TDI-FPGA" I L 5850 5800 60
-F80 "TMS" B L 5850 5900 60
-F81 "TDO_FPGA/TDO-JTAG" O L 5850 6000 60
-F82 "CY-SLRD" B L 5850 6100 60
-$EndSheet
-Wire Wire Line
-	7900 3400 8400 3400
-Wire Wire Line
-	7900 3500 8400 3500
-Wire Wire Line
-	7900 3600 8400 3600
-Wire Wire Line
-	7900 3700 8400 3700
-Wire Wire Line
-	7900 3800 8400 3800
-Wire Wire Line
-	7900 3900 8400 3900
-Wire Wire Line
-	7900 4000 8400 4000
-Wire Wire Line
-	7900 4100 8400 4100
-Wire Wire Line
-	7900 4350 8400 4350
-Wire Wire Line
-	7900 4450 8400 4450
-Wire Wire Line
-	7900 4550 8400 4550
-Wire Wire Line
-	7900 4650 8400 4650
-Wire Wire Line
-	7900 4750 8400 4750
-Wire Wire Line
-	7900 4850 8400 4850
-Wire Wire Line
-	7900 4950 8400 4950
-Wire Wire Line
-	8400 5050 7900 5050
-Wire Wire Line
-	7900 5150 8400 5150
-Wire Wire Line
-	8400 5250 7900 5250
+F28 "EXP-IO13_P" B L 5850 4100 60
+F29 "EXP-IO13_N" B L 5850 4200 60
+F30 "EXP-IO14_P" B L 5850 4300 60
+F31 "EXP-IO14_N" B L 5850 4400 60
+F32 "EXP-IO15_P" B L 5850 4500 60
+F33 "EXP-IO15_N" B L 5850 4600 60
+F34 "EXP-IO16_P" B L 5850 4700 60
+F35 "EXP-IO16_N" B L 5850 4800 60
+F36 "EXP-IO17_N" B L 5850 4900 60
+F37 "EXP-IO17_P" B L 5850 5000 60
+F38 "EXP-IO18_P" B L 5850 5100 60
+F39 "EXP-IO18_N" B L 5850 5200 60
+F40 "EXP-IO19_P" B L 5850 5300 60
+F41 "EXP-IO19_N" B L 5850 5400 60
+F42 "EXP-IO2_P" B L 5850 2000 60
+F43 "EXP-IO2_N" B L 5850 1900 60
+F44 "EXP-IO20_N" B L 5850 5600 60
+F45 "EXP-IO20_P" B L 5850 5500 60
+F46 "EXP-IO3_N" B L 5850 2200 60
+F47 "EXP-IO3_P" B L 5850 2100 60
+F48 "EXP-IO4_N" B L 5850 2400 60
+F49 "EXP-IO4_P" B L 5850 2300 60
+F50 "EXP-IO5_N" B L 5850 2600 60
+F51 "EXP-IO5_P" B L 5850 2500 60
+F52 "EXP-IO6_N" B L 5850 2800 60
+F53 "EXP-IO6_P" B L 5850 2700 60
+F54 "EXP-IO7_N" B L 5850 3000 60
+F55 "EXP-IO7_P" B L 5850 2900 60
+F56 "EXP-IO8_N" B L 5850 3200 60
+F57 "EXP-IO8_P" B L 5850 3100 60
+F58 "EXP-IO9_N" B L 5850 3400 60
+F59 "EXP-IO9_P" B L 5850 3300 60
+F60 "TCK" B L 5850 5700 60
+F61 "TDO-USB/TDI-FPGA" I L 5850 5800 60
+F62 "TMS" B L 5850 5900 60
+F63 "TDO_FPGA/TDO-JTAG" O L 5850 6000 60
+F64 "CY-SLRD" B L 5850 6100 60
+F65 "TMDS-RX1-CLK_P" B R 7900 4350 60
+F66 "TMDS-RX1-CLK_N" B R 7900 4450 60
+F67 "TMDS-RX1-2_P" B R 7900 4550 60
+F68 "TMDS-RX1-2_N" B R 7900 4650 60
+F69 "TMDS-RX1-0_P" B R 7900 4950 60
+F70 "TMDS-RX1-0_N" B R 7900 5050 60
+F71 "TMDS-RX1-1_P" B R 7900 4750 60
+F72 "TMDS-RX1-1_N" B R 7900 4850 60
+F73 "TMDS-RX1-SCL" B R 7900 5150 60
+F74 "TMDS-RX1-SDA" B R 7900 5250 60
+F75 "M0/RESET" B R 7900 3000 60
+F76 "SCK" B R 7900 3100 60
+F77 "PROG" B R 7900 2900 60
+F78 "TMDS-TX1-2_P" B R 7900 3400 60
+F79 "TMDS-TX1-2_N" B R 7900 3500 60
+F80 "TMDS-TX1-1_P" B R 7900 3600 60
+F81 "TMDS-TX1-1_N" B R 7900 3700 60
+F82 "TMDS-TX1-0_P" B R 7900 3800 60
+F83 "TMDS-TX1-0_N" B R 7900 3900 60
+F84 "TMDS-TX1-CLK_P" B R 7900 4000 60
+F85 "TMDS-TX1-CLK_N" B R 7900 4100 60
+$EndSheet
 $EndSCHEMATC

Commit message: Issue #336
Changed lines of the file:
@@
 EELAYER 27 0
 EELAYER END
-$Descr A4 11693 8268
+$Descr A3 16535 11693
 encoding utf-8
 Sheet 1 7
 Title ""
-Date "5 jul 2013"
+Date "8 jul 2013"
 Rev ""
 Comp ""
@@
 $EndSheet
 $Sheet
-S 1150 6100 3850 1400
+S 11600 4350 3850 1400
 U 51BACC6F
 F0 "power" 50
@@
 $EndSheet
 $Sheet
-S 8400 3300 1750 2700
+S 8400 3300 1550 5750
 U 51CD5DED
 F0 "hdmi" 50
@@
 F18 "TMDS-TX1-CLK_P" B L 8400 4000 60
 F19 "TMDS-TX1-CLK_N" B L 8400 4100 60
+F20 "TMDS-TX2-2_P" B L 8400 5450 60
+F21 "TMDS-TX2-1_P" B L 8400 5650 60
+F22 "TMDS-TX2-0_P" B L 8400 5850 60
+F23 "TMDS-TX2-2_N" B L 8400 5550 60
+F24 "TMDS-TX2-1_N" B L 8400 5750 60
+F25 "TMDS-TX2-0_N" B L 8400 5950 60
+F26 "TMDS-TX2-CLK_P" B L 8400 6050 60
+F27 "TMDS-TX2-CLK_N" B L 8400 6150 60
+F28 "TMDS-RX2-2_P" B L 8400 6350 60
+F29 "TMDS-RX2-1_P" B L 8400 6550 60
+F30 "TMDS-RX2-0_P" B L 8400 6750 60
+F31 "TMDS-RX2-2_N" B L 8400 6450 60
+F32 "TMDS-RX2-1_N" B L 8400 6650 60
+F33 "TMDS-RX2-0_N" B L 8400 6850 60
+F34 "TMDS-RX2-CLK_P" B L 8400 6950 60
+F35 "TMDS-RX2-CLK_N" B L 8400 7050 60
 $EndSheet
 Wire Wire Line
@@
 	8400 5250 7900 5250
 $Sheet
-S 5850 700  2050 5650
+S 5850 700  2050 8300
 U 51AED6DE
 F0 "spartan6" 70
@@
 F84 "TMDS-TX1-CLK_P" B R 7900 4000 60
 F85 "TMDS-TX1-CLK_N" B R 7900 4100 60
+F86 "TMDS-TX2-2_P" B R 7900 5450 60
+F87 "TMDS-TX2-2_N" B R 7900 5550 60
+F88 "TMDS-TX2-1_P" B R 7900 5650 60
+F89 "TMDS-TX2-1_N" B R 7900 5750 60
+F90 "TMDS-TX2-0_P" B R 7900 5850 60
+F91 "TMDS-TX2-0_N" B R 7900 5950 60
+F92 "TMDS-TX2-CLK_P" B R 7900 6050 60
+F93 "TMDS-TX2-CLK_N" B R 7900 6150 60
+F94 "TMDS-RX2-2_P" B R 7900 6350 60
+F95 "TMDS-RX2-2_N" B R 7900 6450 60
+F96 "TMDS-RX2-1_P" B R 7900 6550 60
+F97 "TMDS-RX2-1_N" B R 7900 6650 60
+F98 "TMDS-RX2-0_P" B R 7900 6750 60
+F99 "TMDS-RX2-CLK_P" B R 7900 6950 60
+F100 "TMDS-RX2-CLK_N" B R 7900 7050 60
+F101 "TMDS-RX2-0_N" B R 7900 6850 60
 $EndSheet
+Wire Wire Line
+	8400 5450 7900 5450
+Wire Wire Line
+	7900 5550 8400 5550
+Wire Wire Line
+	8400 5650 7900 5650
+Wire Wire Line
+	7900 5750 8400 5750
+Wire Wire Line
+	8400 5850 7900 5850
+Wire Wire Line
+	7900 5950 8400 5950
+Wire Wire Line
+	7900 6050 8400 6050
+Wire Wire Line
+	8400 6150 7900 6150
+Wire Wire Line
+	7900 6350 8400 6350
+Wire Wire Line
+	7900 6450 8400 6450
+Wire Wire Line
+	7900 6550 8400 6550
+Wire Wire Line
+	8400 6650 7900 6650
+Wire Wire Line
+	7900 6750 8400 6750
+Wire Wire Line
+	8400 6850 7900 6850
+Wire Wire Line
+	7900 6950 8400 6950
+Wire Wire Line
+	8400 7050 7900 7050
 $EndSCHEMATC
