File: board/spartan6lxXXX.sch (KiCad schematic (older format))
At the start: 5 parts

Commit message: Issue #336
Parts:
- gave numbers to parts that had none: 1
Connections:
- net labels added: DDR-0V9, DDR-A0, DDR-A1, DDR-A10, DDR-A11, DDR-A12, DDR-A2, DDR-A3, DDR-A4, DDR-A5, DDR-A6, DDR-A7, DDR-A8, DDR-A9, DDR-A[0..12], DDR-BA0, DDR-BA1, DDR-BA2, DDR-CAS, DDR-CKE, DDR-CK_N, DDR-CK_P, DDR-D0, DDR-D1, DDR-D10, DDR-D11, DDR-D12, DDR-D13, DDR-D14, DDR-D15, DDR-D2, DDR-D3, DDR-D4, DDR-D5, DDR-D6, DDR-D7, DDR-D8, DDR-D9, DDR-D[0..15], DDR-LDM, DDR-LDQS_N, DDR-LDQS_P, DDR-ODT, DDR-RAS, DDR-UDM, DDR-UDQS_N, DDR-UDQS_P, DDR-WE
- wire segments 0 -> 40

Commit message: Issue #336
Connections:
- net labels added: DDR1V8, GCLK, JA-CLK_N, JA-CLK_P, JA-D0_N, JA-D0_P, JA-D1_N, JA-D1_P, JA-D2_N, JA-D2_P, JA-SCL, JA-SDA, TCK, TDO-USB/TDI-FPGA, TDO_FPGA/TDO-JTAG, TMDS-RX-0_N, TMDS-RX-0_P, TMDS-RX-1_N, TMDS-RX-1_P, TMDS-RX-2_N, TMDS-RX-2_P, TMDS-RX-CLK_N, TMDS-RX-CLK_P, TMDS-RX-SCL, TMDS-RX-SDA, TMS, VCC3V3, VSS
- wire segments 40 -> 143
- no-connect marks 0 -> 13

Commit message: Issue #336
Connections:
- net labels added: EXP-IO10_N, EXP-IO10_P, EXP-IO11_N, EXP-IO11_P, EXP-IO12_N, EXP-IO12_P, EXP-IO13_N, EXP-IO13_P, EXP-IO14_N, EXP-IO14_P, EXP-IO15_N, EXP-IO15_P, EXP-IO16_N, EXP-IO16_P, EXP-IO17_N, EXP-IO17_P, EXP-IO18_N, EXP-IO18_P, EXP-IO19_N, EXP-IO19_P, EXP-IO1_N, EXP-IO1_P, EXP-IO20_N, EXP-IO20_P, EXP-IO2_N, EXP-IO2_P, EXP-IO3_N, EXP-IO3_P, EXP-IO4_N, EXP-IO4_P, EXP-IO5_N, EXP-IO5_P, EXP-IO6_N, EXP-IO6_P, EXP-IO7_N, EXP-IO7_P, EXP-IO8_N, EXP-IO8_P, EXP-IO9_N, EXP-IO9_P, GND, VCC1V2
- net labels removed: VSS
- wire segments 143 -> 71
- no-connect marks 13 -> 18

Commit message: Issue #336
Parts:
- added R?: R, ~, symbol R
Connections:
- net labels added: DQ1, DQ2, DQ3, GND-T
- wire segments 71 -> 86
- no-connect marks 18 -> 12
Changed lines of the file:
@@
 $Descr A3 16535 11693
 encoding utf-8
-Sheet 7 7
+Sheet 6 7
 Title ""
-Date "27 jun 2013"
+Date "4 jul 2013"
 Rev ""
 Comp ""
@@
 $Comp
 L SPARTAN6LXXXX-CSG324 U3
-U 2 1 51B2AC95
-P 4300 4700
-F 0 "U3" H 3600 7250 60  0000 C CNN
-F 1 "SPARTAN6LXXXX-CSG324" H 4000 800 60  0000 C CNN
-F 2 "" H 4300 4700 60  0001 C CNN
-F 3 "" H 4300 4700 60  0001 C CNN
-	2    4300 4700
-	1    0    0    -1
-$EndComp
-$Comp
-L SPARTAN6LXXXX-CSG324 U3
 U 1 1 51B2AC80
 P 1700 4700
@@
 	1    0    0    -1
 $EndComp
-Text Label 11650 4300 2    60   ~ 0
+Text Label 11650 4300 2    39   ~ 0
 DDR-D0
-Text Label 11650 4400 2    60   ~ 0
+Text Label 11650 4400 2    39   ~ 0
 DDR-D1
-Text Label 11650 4500 2    60   ~ 0
+Text Label 11650 4500 2    39   ~ 0
 DDR-D2
-Text Label 11650 4600 2    60   ~ 0
+Text Label 11650 4600 2    39   ~ 0
 DDR-D3
-Text Label 11650 5100 2    60   ~ 0
+Text Label 11650 5100 2    39   ~ 0
 DDR-D4
-Text Label 11650 5200 2    60   ~ 0
+Text Label 11650 5200 2    39   ~ 0
 DDR-D5
-Text Label 11650 4900 2    60   ~ 0
+Text Label 11650 4900 2    39   ~ 0
 DDR-D6
-Text Label 11650 5000 2    60   ~ 0
+Text Label 11650 5000 2    39   ~ 0
 DDR-D7
-Text Label 11650 4100 2    60   ~ 0
+Text Label 11650 4100 2    39   ~ 0
 DDR-D8
-Text Label 11650 4200 2    60   ~ 0
+Text Label 11650 4200 2    39   ~ 0
 DDR-D9
-Text Label 11650 3900 2    60   ~ 0
+Text Label 11650 3900 2    39   ~ 0
 DDR-D10
-Text Label 11650 4000 2    60   ~ 0
+Text Label 11650 4000 2    39   ~ 0
 DDR-D11
-Text Label 11650 3500 2    60   ~ 0
+Text Label 11650 3500 2    39   ~ 0
 DDR-D12
-Text Label 11650 3600 2    60   ~ 0
+Text Label 11650 3600 2    39   ~ 0
 DDR-D13
-Text Label 11650 3300 2    60   ~ 0
+Text Label 11650 3300 2    39   ~ 0
 DDR-D14
-Text Label 11650 3400 2    60   ~ 0
+Text Label 11650 3400 2    39   ~ 0
 DDR-D15
 Entry Wire Line
@@
 Text HLabel 12150 5300 2    60   BiDi ~ 0
 DDR-D[0..15]
-Text Label 11450 6300 2    60   ~ 0
+Text Label 11450 6300 2    39   ~ 0
 DDR-A0
-Text Label 11450 6400 2    60   ~ 0
+Text Label 11450 6400 2    39   ~ 0
 DDR-A1
-Text Label 11450 6800 2    60   ~ 0
+Text Label 11450 6800 2    39   ~ 0
 DDR-A2
-Text Label 11450 5900 2    60   ~ 0
+Text Label 11450 5900 2    39   ~ 0
 DDR-A3
-Text Label 11450 7200 2    60   ~ 0
+Text Label 11450 7200 2    39   ~ 0
 DDR-A4
-Text Label 11450 5700 2    60   ~ 0
+Text Label 11450 5700 2    39   ~ 0
 DDR-A5
-Text Label 11450 5800 2    60   ~ 0
+Text Label 11450 5800 2    39   ~ 0
 DDR-A6
-Text Label 11450 6700 2    60   ~ 0
+Text Label 11450 6700 2    39   ~ 0
 DDR-A7
-Text Label 11450 7300 2    60   ~ 0
+Text Label 11450 7300 2    39   ~ 0
 DDR-A8
-Text Label 11450 7400 2    60   ~ 0
+Text Label 11450 7400 2    39   ~ 0
 DDR-A9
-Text Label 11500 7100 2    60   ~ 0
+Text Label 11450 7100 2    39   ~ 0
 DDR-A10
-Text Label 11500 7800 2    60   ~ 0
+Text Label 11500 7800 2    39   ~ 0
 DDR-A11
-Text Label 11500 7600 2    60   ~ 0
+Text Label 11500 7600 2    39   ~ 0
 DDR-A12
-Text Label 11650 3200 2    60   ~ 0
+Text Label 11650 3200 2    39   ~ 0
 DDR-0V9
-Text Label 11650 2800 2    60   ~ 0
+Text Label 11650 2800 2    39   ~ 0
 DDR-0V9
-Text Label 11650 8200 2    60   ~ 0
+Text Label 11650 8200 2    39   ~ 0
 DDR-0V9
 Entry Wire Line
@@
 Text GLabel 15350 7700 2    60   Input ~ 0
 DDR1V8
-NoConn ~ 5100 2850
-NoConn ~ 5100 2950
-NoConn ~ 5100 2750
-NoConn ~ 5100 3550
-NoConn ~ 5100 3650
-NoConn ~ 5100 2650
-NoConn ~ 5100 3050
-NoConn ~ 5100 3750
-NoConn ~ 5100 3350
-NoConn ~ 5100 3250
-NoConn ~ 5100 4050
-NoConn ~ 5100 4150
-NoConn ~ 5100 3150
 Text GLabel 5700 5450 2    60   Output ~ 0
 GCLK
@@
 Wire Wire Line
 	5100 5450 5700 5450
-Text Label 5600 5450 2    60   ~ 0
+Text Label 5600 5450 2    39   ~ 0
 GCLK
 Wire Wire Line
@@
 Wire Wire Line
 	2500 6950 2750 6950
-Text Label 2750 6950 2    60   ~ 0
+Text Label 2750 6950 2    39   ~ 0
 GND
-Text Label 12850 6150 0    60   ~ 0
+Text Label 12850 6150 0    39   ~ 0
 GND
 Wire Wire Line
 	2500 6650 2750 6650
-Text Label 2750 6650 2    60   ~ 0
+Text Label 2750 6650 2    39   ~ 0
 GND
 NoConn ~ 5100 5050
@@
 NoConn ~ 5100 4950
 NoConn ~ 5100 4850
+Text Label 2800 5950 2    39   ~ 0
+GND-T
+Wire Wire Line
+	2500 5950 2800 5950
+Text Label 2800 5650 2    39   ~ 0
+GND-T
+Wire Wire Line
+	2500 5650 2800 5650
+Text Label 2800 6150 2    39   ~ 0
+GND-T
+Wire Wire Line
+	2500 6150 2800 6150
+Text Label 2800 4450 2    39   ~ 0
+GND-T
+Wire Wire Line
+	2500 4450 2800 4450
+Text Label 2800 4350 2    39   ~ 0
+GND-T
+Wire Wire Line
+	2500 4350 2800 4350
+Text Label 2800 5250 2    39   ~ 0
+GND-T
+Wire Wire Line
+	2500 5250 2800 5250
+Text Label 2800 2950 2    39   ~ 0
+GND-T
+Wire Wire Line
+	2500 2950 2800 2950
+Text Label 2800 5350 2    39   ~ 0
+GND-T
+Wire Wire Line
+	2500 5350 2800 5350
+Text Label 2800 2550 2    39   ~ 0
+GND-T
+Wire Wire Line
+	2500 2550 2800 2550
+Text Label 2800 7750 2    39   ~ 0
+GND-T
+Wire Wire Line
+	2500 7750 2800 7750
+Text Label 900  9100 0    60   ~ 0
+GND-T
+Wire Wire Line
+	900  9100 1200 9100
+$Comp
+L R R?
+U 1 1 51CE8B12
+P 1450 9100
+F 0 "R?" V 1530 9100 40  0000 C CNN
+F 1 "R" V 1457 9101 40  0000 C CNN
+F 2 "~" V 1380 9100 30  0000 C CNN
+F 3 "~" H 1450 9100 30  0000 C CNN
+	1    1450 9100
+	0    1    1    0
+$EndComp
+Text Label 1950 9100 2    60   ~ 0
+GND
+Wire Wire Line
+	1700 9100 1950 9100
+Wire Wire Line
+	8050 3400 8350 3400
+Wire Wire Line
+	8050 3300 8350 3300
+Text Label 8350 3300 2    39   ~ 0
+DQ3
+Text Label 8350 3400 2    39   ~ 0
+DQ2
+Wire Wire Line
+	8050 2900 8350 2900
+Text Label 8350 2900 2    39   ~ 0
+DQ1
+$Comp
+L SPARTAN6LXXXX-CSG324 U3
+U 2 1 51B2AC95
+P 4300 4700
+F 0 "U3" H 3600 7250 60  0000 C CNN
+F 1 "SPARTAN6LXXXX-CSG324" H 4000 800 60  0000 C CNN
+F 2 "" H 4300 4700 60  0001 C CNN
+F 3 "" H 4300 4700 60  0001 C CNN
+	2    4300 4700
+	1    0    0    -1
+$EndComp
+NoConn ~ 2500 3650
+NoConn ~ 2500 3750
+NoConn ~ 2500 4150
+NoConn ~ 2500 4650
+NoConn ~ 2500 6250
+NoConn ~ 2500 7350
+NoConn ~ 2500 7250
 $EndSCHEMATC

Commit message: Issue #336
Parts:
- removed R?: R, ~, symbol R
- added R? (x11): R, ~, symbol R
Connections:
- net labels added: CY-SLRD, M0/RESET, PROG, SCK
- net labels removed: JA-SCL, JA-SDA
- wire segments 86 -> 97

Commit message: Issue #336
Connections:
- net labels added: TMDS-RX1-0_N, TMDS-RX1-0_P, TMDS-RX1-1_N, TMDS-RX1-1_P, TMDS-RX1-2_N, TMDS-RX1-2_P, TMDS-RX1-CLK_N, TMDS-RX1-CLK_P, TMDS-RX1-SCL, TMDS-RX1-SDA, TMDS-TX1-0_N, TMDS-TX1-0_P, TMDS-TX1-1_N, TMDS-TX1-1_P, TMDS-TX1-2_N, TMDS-TX1-2_P, TMDS-TX1-CLK_N, TMDS-TX1-CLK_P, TMDS-TX2-0_N, TMDS-TX2-0_P, TMDS-TX2-1_N, TMDS-TX2-1_P, TMDS-TX2-2_N, TMDS-TX2-2_P, TMDS-TX2-CLK_N, TMDS-TX2-CLK_P, VCC2V5
- net labels removed: JA-CLK_N, JA-CLK_P, JA-D0_N, JA-D0_P, JA-D1_N, JA-D1_P, JA-D2_N, JA-D2_P, TMDS-RX-0_N, TMDS-RX-0_P, TMDS-RX-1_N, TMDS-RX-1_P, TMDS-RX-2_N, TMDS-RX-2_P, TMDS-RX-CLK_N, TMDS-RX-CLK_P, TMDS-RX-SCL, TMDS-RX-SDA
Changed lines of the file:
@@
 $Descr A3 16535 11693
 encoding utf-8
-Sheet 6 7
+Sheet 7 7
 Title ""
-Date "4 jul 2013"
+Date "5 jul 2013"
 Rev ""
 Comp ""
@@
 	15150 7000 15350 7000
 Text GLabel 15350 3500 2    60   Input ~ 0
-VCC3V3
+VCC2V5
 Text GLabel 15550 4800 2    60   Input ~ 0
 VCC1V2
@@
 Text HLabel 8050 5500 2    60   BiDi ~ 0
 EXP-IO12_P
-Text HLabel 8050 5700 2    60   BiDi ~ 0
-JA-CLK_P
-Text HLabel 8050 5800 2    60   BiDi ~ 0
-JA-CLK_N
 Text HLabel 8050 5900 2    60   BiDi ~ 0
 EXP-IO13_P
@@
 Text HLabel 8050 6200 2    60   BiDi ~ 0
 EXP-IO14_N
-Text HLabel 8050 8200 2    60   BiDi ~ 0
-JA-D2_N
-Text HLabel 8050 8100 2    60   BiDi ~ 0
-JA-D2_P
-Text HLabel 8050 8000 2    60   BiDi ~ 0
-JA-D1_N
-Text HLabel 8050 7900 2    60   BiDi ~ 0
-JA-D1_P
-Text HLabel 8050 7800 2    60   BiDi ~ 0
-JA-D0_N
-Text HLabel 8050 7700 2    60   BiDi ~ 0
-JA-D0_P
 Text HLabel 8050 6300 2    60   BiDi ~ 0
 EXP-IO15_P
@@
 EXP-IO9_P
 Text HLabel 5100 5650 2    60   BiDi ~ 0
-TMDS-RX-CLK_P
+TMDS-RX1-CLK_P
 Text HLabel 5100 5750 2    60   BiDi ~ 0
-TMDS-RX-CLK_N
+TMDS-RX1-CLK_N
 Text HLabel 5100 5850 2    60   BiDi ~ 0
-TMDS-RX-2_P
+TMDS-RX1-2_P
 Text HLabel 5100 5950 2    60   BiDi ~ 0
-TMDS-RX-2_N
+TMDS-RX1-2_N
 Text HLabel 5100 6050 2    60   BiDi ~ 0
-TMDS-RX-0_P
+TMDS-RX1-0_P
 Text HLabel 5100 6150 2    60   BiDi ~ 0
-TMDS-RX-0_N
+TMDS-RX1-0_N
 Text HLabel 5100 6250 2    60   BiDi ~ 0
-TMDS-RX-1_P
+TMDS-RX1-1_P
 Text HLabel 5100 6350 2    60   BiDi ~ 0
-TMDS-RX-1_N
+TMDS-RX1-1_N
 Text HLabel 5100 6450 2    60   BiDi ~ 0
-TMDS-RX-SCL
+TMDS-RX1-SCL
 Text HLabel 5100 6550 2    60   BiDi ~ 0
-TMDS-RX-SDA
+TMDS-RX1-SDA
 Text Label 12850 6150 0    39   ~ 0
 GND
@@
 Text Label 15550 4800 2    39   ~ 0
 VCC1V2
+Text HLabel 8050 8100 2    60   BiDi ~ 0
+TMDS-TX1-2_P
+Text HLabel 8050 8200 2    60   BiDi ~ 0
+TMDS-TX1-2_N
+Text HLabel 8050 7900 2    60   BiDi ~ 0
+TMDS-TX1-1_P
+Text HLabel 8050 8000 2    60   BiDi ~ 0
+TMDS-TX1-1_N
+Text HLabel 8050 7700 2    60   BiDi ~ 0
+TMDS-TX1-0_P
+Text HLabel 8050 7800 2    60   BiDi ~ 0
+TMDS-TX1-0_N
+Text HLabel 8050 5700 2    60   BiDi ~ 0
+TMDS-TX1-CLK_P
+Text HLabel 8050 5800 2    60   BiDi ~ 0
+TMDS-TX1-CLK_N
+Text HLabel 2500 2650 2    60   BiDi ~ 0
+TMDS-TX2-2_P
+Text HLabel 2500 2750 2    60   BiDi ~ 0
+TMDS-TX2-2_N
+Text HLabel 2500 3050 2    60   BiDi ~ 0
+TMDS-TX2-1_P
+Text HLabel 2500 3150 2    60   BiDi ~ 0
+TMDS-TX2-1_N
+Text HLabel 2500 8250 2    60   BiDi ~ 0
+TMDS-TX2-0_P
+Text HLabel 2500 8350 2    60   BiDi ~ 0
+TMDS-TX2-0_N
+Text HLabel 2500 7850 2    60   BiDi ~ 0
+TMDS-TX2-CLK_P
+Text HLabel 2500 7950 2    60   BiDi ~ 0
+TMDS-TX2-CLK_N
 $EndSCHEMATC

Commit message: Issue #336
Connections:
- net labels added: TMDS-RX2-0_N, TMDS-RX2-0_P, TMDS-RX2-1_N, TMDS-RX2-1_P, TMDS-RX2-2_N, TMDS-RX2-2_P, TMDS-RX2-CLK_N, TMDS-RX2-CLK_P
- wire segments 97 -> 89
Changed lines of the file:
@@
 Sheet 7 7
 Title ""
-Date "5 jul 2013"
+Date "8 jul 2013"
 Rev ""
 Comp ""
@@
 Text GLabel 12850 6150 0    60   Input ~ 0
 GND
-Wire Wire Line
-	5100 8150 5450 8150
-Wire Wire Line
-	5100 8050 5450 8050
-Wire Wire Line
-	5100 7950 5450 7950
-Wire Wire Line
-	5100 7850 5450 7850
-Wire Wire Line
-	5100 7750 5450 7750
-Wire Wire Line
-	5100 7650 5450 7650
-Wire Wire Line
-	5100 7550 5450 7550
-Wire Wire Line
-	5100 7450 5450 7450
 Wire Wire Line
 	8050 8400 8400 8400
@@
 Text Label 15550 4800 2    39   ~ 0
 VCC1V2
-Text HLabel 8050 8100 2    60   BiDi ~ 0
-TMDS-TX1-2_P
-Text HLabel 8050 8200 2    60   BiDi ~ 0
-TMDS-TX1-2_N
 Text HLabel 8050 7900 2    60   BiDi ~ 0
 TMDS-TX1-1_P
@@
 Text HLabel 2500 7950 2    60   BiDi ~ 0
 TMDS-TX2-CLK_N
+Text HLabel 5100 7950 2    60   BiDi ~ 0
+TMDS-RX2-2_P
+Text HLabel 5100 7550 2    60   BiDi ~ 0
+TMDS-RX2-2_N
+Text HLabel 5100 2650 2    60   BiDi ~ 0
+TMDS-RX2-1_P
+Text HLabel 5100 2750 2    60   BiDi ~ 0
+TMDS-RX2-1_N
+Text HLabel 5100 4050 2    60   BiDi ~ 0
+TMDS-RX2-0_P
+Text HLabel 5100 4150 2    60   BiDi ~ 0
+TMDS-RX2-0_N
+Text HLabel 5100 4450 2    60   BiDi ~ 0
+TMDS-RX2-CLK_P
+Text HLabel 5100 4550 2    60   BiDi ~ 0
+TMDS-RX2-CLK_N
+Text HLabel 8050 7300 2    60   BiDi ~ 0
+TMDS-TX1-2_P
+Text HLabel 8050 7400 2    60   BiDi ~ 0
+TMDS-TX1-2_N
 $EndSCHEMATC
