File: board/DDR2.sch (KiCad schematic (older format))
At the start: 79 parts, among them P10 CONN_1, P11 CONN_1, P12 CONN_1, P13 CONN_1, P14 CONN_1, P15 CONN_1, P16 CONN_1, P17 CONN_1, P18 CONN_1, P19 CONN_1, P2 CONN_1, P20 CONN_1, P21 CONN_1, P22 CONN_1, P23 CONN_1, P24 CONN_1, P25 CONN_1, P26 CONN_1, P27 CONN_1, P28 CONN_1, P29 CONN_1, P3 CONN_1, P30 CONN_1, P31 CONN_1, P32 CONN_1, P33 CONN_1, P34 CONN_1, P35 CONN_1, P36 CONN_1, P37 CONN_1, P38 CONN_1, P39 CONN_1, P4 CONN_1, P40 CONN_1, P41 CONN_1, P42 CONN_1, P43 CONN_1, P44 CONN_1, P45 CONN_1, P46 CONN_1, P5 CONN_1, P6 CONN_1, P7 CONN_1, P8 CONN_1, P9 CONN_1, U7 MT47H64M16HR

Commit message: Issue #1022 - Power supply & pic& SCHEMATIC SECTION.
Parts:
- added C184, C185, C186, C187, C188, C189, C190, C191, C192, C193: 0.1MFD, ~, symbol C
Connections:
- net DDR0V9: now also C184.1, C185.1, C186.1, C187.1, C188.1, C189.1, C190.1, C191.1, C192.1, C193.1
- net GND: now also C184.2, C185.2, C186.2, C187.2, C188.2, C189.2, C190.2, C191.2, C192.2, C193.2
Changed lines of the file:
@@
 Sheet 3 8
 Title ""
-Date "14 mar 2014"
+Date "18 mar 2014"
 Rev ""
 Comp ""
@@
 	6250 2800 6250 3000
 Connection ~ 6250 3000
+$Comp
+L C C184
+U 1 1 5335B417
+P 4800 6700
+F 0 "C184" H 4800 6800 40  0000 L CNN
+F 1 "0.1MFD" H 4806 6615 40  0000 L CNN
+F 2 "~" H 4838 6550 30  0000 C CNN
+F 3 "~" H 4800 6700 60  0000 C CNN
+	1    4800 6700
+	1    0    0    -1
+$EndComp
+$Comp
+L C C185
+U 1 1 5335B41D
+P 5100 6700
+F 0 "C185" H 5100 6800 40  0000 L CNN
+F 1 "0.1MFD" H 5106 6615 40  0000 L CNN
+F 2 "~" H 5138 6550 30  0000 C CNN
+F 3 "~" H 5100 6700 60  0000 C CNN
+	1    5100 6700
+	1    0    0    -1
+$EndComp
+$Comp
+L C C186
+U 1 1 5335B423
+P 5400 6700
+F 0 "C186" H 5400 6800 40  0000 L CNN
+F 1 "0.1MFD" H 5406 6615 40  0000 L CNN
+F 2 "~" H 5438 6550 30  0000 C CNN
+F 3 "~" H 5400 6700 60  0000 C CNN
+	1    5400 6700
+	1    0    0    -1
+$EndComp
+$Comp
+L C C187
+U 1 1 5335B429
+P 5700 6700
+F 0 "C187" H 5700 6800 40  0000 L CNN
+F 1 "0.1MFD" H 5706 6615 40  0000 L CNN
+F 2 "~" H 5738 6550 30  0000 C CNN
+F 3 "~" H 5700 6700 60  0000 C CNN
+	1    5700 6700
+	1    0    0    -1
+$EndComp
+$Comp
+L C C188
+U 1 1 5335B42F
+P 5950 6700
+F 0 "C188" H 5950 6800 40  0000 L CNN
+F 1 "0.1MFD" H 5956 6615 40  0000 L CNN
+F 2 "~" H 5988 6550 30  0000 C CNN
+F 3 "~" H 5950 6700 60  0000 C CNN
+	1    5950 6700
+	1    0    0    -1
+$EndComp
+$Comp
+L C C189
+U 1 1 5335B435
+P 6200 6700
+F 0 "C189" H 6200 6800 40  0000 L CNN
+F 1 "0.1MFD" H 6206 6615 40  0000 L CNN
+F 2 "~" H 6238 6550 30  0000 C CNN
+F 3 "~" H 6200 6700 60  0000 C CNN
+	1    6200 6700
+	1    0    0    -1
+$EndComp
+$Comp
+L C C190
+U 1 1 5335B43B
+P 6450 6700
+F 0 "C190" H 6450 6800 40  0000 L CNN
+F 1 "0.1MFD" H 6456 6615 40  0000 L CNN
+F 2 "~" H 6488 6550 30  0000 C CNN
+F 3 "~" H 6450 6700 60  0000 C CNN
+	1    6450 6700
+	1    0    0    -1
+$EndComp
+$Comp
+L C C191
+U 1 1 5335B441
+P 6700 6700
+F 0 "C191" H 6700 6800 40  0000 L CNN
+F 1 "0.1MFD" H 6706 6615 40  0000 L CNN
+F 2 "~" H 6738 6550 30  0000 C CNN
+F 3 "~" H 6700 6700 60  0000 C CNN
+	1    6700 6700
+	1    0    0    -1
+$EndComp
+$Comp
+L C C192
+U 1 1 5335B447
+P 7000 6700
+F 0 "C192" H 7000 6800 40  0000 L CNN
+F 1 "0.1MFD" H 7006 6615 40  0000 L CNN
+F 2 "~" H 7038 6550 30  0000 C CNN
+F 3 "~" H 7000 6700 60  0000 C CNN
+	1    7000 6700
+	1    0    0    -1
+$EndComp
+$Comp
+L C C193
+U 1 1 5335B44D
+P 7300 6700
+F 0 "C193" H 7300 6800 40  0000 L CNN
+F 1 "0.1MFD" H 7306 6615 40  0000 L CNN
+F 2 "~" H 7338 6550 30  0000 C CNN
+F 3 "~" H 7300 6700 60  0000 C CNN
+	1    7300 6700
+	1    0    0    -1
+$EndComp
+Text Label 4600 6900 0    60   ~ 0
+VSS
+Wire Wire Line
+	4600 6900 7300 6900
+Connection ~ 4800 6900
+Connection ~ 5100 6900
+Connection ~ 5400 6900
+Connection ~ 5700 6900
+Connection ~ 5950 6900
+Connection ~ 6200 6900
+Connection ~ 6450 6900
+Connection ~ 6700 6900
+Connection ~ 7000 6900
+Connection ~ 7000 6500
+Connection ~ 6700 6500
+Connection ~ 6450 6500
+Connection ~ 6200 6500
+Connection ~ 5950 6500
+Connection ~ 5700 6500
+Connection ~ 5400 6500
+Connection ~ 5100 6500
+Connection ~ 4800 6500
+Wire Wire Line
+	4350 6500 7300 6500
+Text Label 4350 6500 0    60   ~ 0
+DDR0V9
 $EndSCHEMATC

Commit message: Issue #1022 - Schematics final.
Changed lines of the file:
@@
 Sheet 3 8
 Title ""
-Date "28 mar 2014"
+Date "31 mar 2014"
 Rev ""
 Comp ""
@@
 VSS
 $Comp
-L GND #PWR2
+L GND #PWR02
 U 1 1 51C148F4
 P 4400 5950
-F 0 "#PWR2" H 4400 5950 30  0001 C CNN
+F 0 "#PWR02" H 4400 5950 30  0001 C CNN
 F 1 "GND" H 4400 5880 30  0001 C CNN
 F 2 "" H 4400 5950 60  0000 C CNN
@@
 	2700 5000 2150 5000
 Wire Wire Line
-	2500 3300 2500 4850
+	2500 3250 2500 4850
 Wire Wire Line
 	2300 5850 5800 5850
@@
 Text Label 4350 6500 0    60   ~ 0
 DDR0V9
+$Comp
+L PWR_FLAG #FLG03
+U 1 1 533EEDE3
+P 2500 3250
+F 0 "#FLG03" H 2500 3345 30  0001 C CNN
+F 1 "PWR_FLAG" H 2500 3430 30  0000 C CNN
+F 2 "" H 2500 3250 60  0000 C CNN
+F 3 "" H 2500 3250 60  0000 C CNN
+	1    2500 3250
+	1    0    0    -1
+$EndComp
+Connection ~ 2500 3300
 $EndSCHEMATC

Commit message: Issue #993
Parts:
- C184, C185, C186, C187, C188, C189, C190, C191, C192, C193, C28, C29, C30, C31, C32, C33, C34, C35, C36, C37, C38, C39, C40, C41, C42, C43: value 0.1MFD -> 0.1mfd
Changed lines of the file:
@@
 $Descr A4 11693 8268
 encoding utf-8
-Sheet 3 8
-Title ""
-Date "31 mar 2014"
+Sheet 2 8
+Title "HDMI2USB"
+Date "3 apr 2014"
 Rev ""
 Comp ""
@@
 VSS
 $Comp
-L GND #PWR02
+L GND #PWR01
 U 1 1 51C148F4
 P 4400 5950
-F 0 "#PWR02" H 4400 5950 30  0001 C CNN
+F 0 "#PWR01" H 4400 5950 30  0001 C CNN
 F 1 "GND" H 4400 5880 30  0001 C CNN
 F 2 "" H 4400 5950 60  0000 C CNN
@@
 P 2800 7450
 F 0 "C29" H 2800 7550 40  0000 L CNN
-F 1 "0.1MFD" H 2806 7365 40  0000 L CNN
+F 1 "0.1mfd" H 2806 7365 40  0000 L CNN
 F 2 "~" H 2838 7300 30  0000 C CNN
 F 3 "~" H 2800 7450 60  0000 C CNN
@@
 P 3100 7450
 F 0 "C31" H 3100 7550 40  0000 L CNN
-F 1 "0.1MFD" H 3106 7365 40  0000 L CNN
+F 1 "0.1mfd" H 3106 7365 40  0000 L CNN
 F 2 "~" H 3138 7300 30  0000 C CNN
 F 3 "~" H 3100 7450 60  0000 C CNN
@@
 P 3400 7450
 F 0 "C33" H 3400 7550 40  0000 L CNN
-F 1 "0.1MFD" H 3406 7365 40  0000 L CNN
+F 1 "0.1mfd" H 3406 7365 40  0000 L CNN
 F 2 "~" H 3438 7300 30  0000 C CNN
 F 3 "~" H 3400 7450 60  0000 C CNN
@@
 P 3700 7450
 F 0 "C35" H 3700 7550 40  0000 L CNN
-F 1 "0.1MFD" H 3706 7365 40  0000 L CNN
+F 1 "0.1mfd" H 3706 7365 40  0000 L CNN
 F 2 "~" H 3738 7300 30  0000 C CNN
 F 3 "~" H 3700 7450 60  0000 C CNN
@@
 P 3950 7450
 F 0 "C37" H 3950 7550 40  0000 L CNN
-F 1 "0.1MFD" H 3956 7365 40  0000 L CNN
+F 1 "0.1mfd" H 3956 7365 40  0000 L CNN
 F 2 "~" H 3988 7300 30  0000 C CNN
 F 3 "~" H 3950 7450 60  0000 C CNN
@@
 P 4200 7450
 F 0 "C39" H 4200 7550 40  0000 L CNN
-F 1 "0.1MFD" H 4206 7365 40  0000 L CNN
+F 1 "0.1mfd" H 4206 7365 40  0000 L CNN
 F 2 "~" H 4238 7300 30  0000 C CNN
 F 3 "~" H 4200 7450 60  0000 C CNN
@@
 P 4450 7450
 F 0 "C40" H 4450 7550 40  0000 L CNN
-F 1 "0.1MFD" H 4456 7365 40  0000 L CNN
+F 1 "0.1mfd" H 4456 7365 40  0000 L CNN
 F 2 "~" H 4488 7300 30  0000 C CNN
 F 3 "~" H 4450 7450 60  0000 C CNN
@@
 P 4700 7450
 F 0 "C41" H 4700 7550 40  0000 L CNN
-F 1 "0.1MFD" H 4706 7365 40  0000 L CNN
+F 1 "0.1mfd" H 4706 7365 40  0000 L CNN
 F 2 "~" H 4738 7300 30  0000 C CNN
 F 3 "~" H 4700 7450 60  0000 C CNN
@@
 P 5000 7450
 F 0 "C42" H 5000 7550 40  0000 L CNN
-F 1 "0.1MFD" H 5006 7365 40  0000 L CNN
+F 1 "0.1mfd" H 5006 7365 40  0000 L CNN
 F 2 "~" H 5038 7300 30  0000 C CNN
 F 3 "~" H 5000 7450 60  0000 C CNN
@@
 P 5300 7450
 F 0 "C43" H 5300 7550 40  0000 L CNN
-F 1 "0.1MFD" H 5306 7365 40  0000 L CNN
+F 1 "0.1mfd" H 5306 7365 40  0000 L CNN
 F 2 "~" H 5338 7300 30  0000 C CNN
 F 3 "~" H 5300 7450 60  0000 C CNN
@@
 P 2800 6850
 F 0 "C28" H 2800 6950 40  0000 L CNN
-F 1 "0.1MFD" H 2806 6765 40  0000 L CNN
+F 1 "0.1mfd" H 2806 6765 40  0000 L CNN
 F 2 "~" H 2838 6700 30  0000 C CNN
 F 3 "~" H 2800 6850 60  0000 C CNN
@@
 P 3050 6850
 F 0 "C30" H 3050 6950 40  0000 L CNN
-F 1 "0.1MFD" H 3056 6765 40  0000 L CNN
+F 1 "0.1mfd" H 3056 6765 40  0000 L CNN
 F 2 "~" H 3088 6700 30  0000 C CNN
 F 3 "~" H 3050 6850 60  0000 C CNN
@@
 P 3550 6850
 F 0 "C34" H 3550 6950 40  0000 L CNN
-F 1 "0.1MFD" H 3556 6765 40  0000 L CNN
+F 1 "0.1mfd" H 3556 6765 40  0000 L CNN
 F 2 "~" H 3588 6700 30  0000 C CNN
 F 3 "~" H 3550 6850 60  0000 C CNN
@@
 P 3850 6850
 F 0 "C36" H 3850 6950 40  0000 L CNN
-F 1 "0.1MFD" H 3856 6765 40  0000 L CNN
+F 1 "0.1mfd" H 3856 6765 40  0000 L CNN
 F 2 "~" H 3888 6700 30  0000 C CNN
 F 3 "~" H 3850 6850 60  0000 C CNN
@@
 P 4150 6850
 F 0 "C38" H 4150 6950 40  0000 L CNN
-F 1 "0.1MFD" H 4156 6765 40  0000 L CNN
+F 1 "0.1mfd" H 4156 6765 40  0000 L CNN
 F 2 "~" H 4188 6700 30  0000 C CNN
 F 3 "~" H 4150 6850 60  0000 C CNN
@@
 P 3300 6850
 F 0 "C32" H 3300 6950 40  0000 L CNN
-F 1 "0.1MFD" H 3306 6765 40  0000 L CNN
+F 1 "0.1mfd" H 3306 6765 40  0000 L CNN
 F 2 "~" H 3338 6700 30  0000 C CNN
 F 3 "~" H 3300 6850 60  0000 C CNN
@@
 P 4800 6700
 F 0 "C184" H 4800 6800 40  0000 L CNN
-F 1 "0.1MFD" H 4806 6615 40  0000 L CNN
+F 1 "0.1mfd" H 4806 6615 40  0000 L CNN
 F 2 "~" H 4838 6550 30  0000 C CNN
 F 3 "~" H 4800 6700 60  0000 C CNN
@@
 P 5100 6700
 F 0 "C185" H 5100 6800 40  0000 L CNN
-F 1 "0.1MFD" H 5106 6615 40  0000 L CNN
+F 1 "0.1mfd" H 5106 6615 40  0000 L CNN
 F 2 "~" H 5138 6550 30  0000 C CNN
 F 3 "~" H 5100 6700 60  0000 C CNN
@@
 P 5400 6700
 F 0 "C186" H 5400 6800 40  0000 L CNN
-F 1 "0.1MFD" H 5406 6615 40  0000 L CNN
+F 1 "0.1mfd" H 5406 6615 40  0000 L CNN
 F 2 "~" H 5438 6550 30  0000 C CNN
 F 3 "~" H 5400 6700 60  0000 C CNN
@@
 P 5700 6700
 F 0 "C187" H 5700 6800 40  0000 L CNN
-F 1 "0.1MFD" H 5706 6615 40  0000 L CNN
+F 1 "0.1mfd" H 5706 6615 40  0000 L CNN
 F 2 "~" H 5738 6550 30  0000 C CNN
 F 3 "~" H 5700 6700 60  0000 C CNN
@@
 P 5950 6700
 F 0 "C188" H 5950 6800 40  0000 L CNN
-F 1 "0.1MFD" H 5956 6615 40  0000 L CNN
+F 1 "0.1mfd" H 5956 6615 40  0000 L CNN
 F 2 "~" H 5988 6550 30  0000 C CNN
 F 3 "~" H 5950 6700 60  0000 C CNN
@@
 P 6200 6700
 F 0 "C189" H 6200 6800 40  0000 L CNN
-F 1 "0.1MFD" H 6206 6615 40  0000 L CNN
+F 1 "0.1mfd" H 6206 6615 40  0000 L CNN
 F 2 "~" H 6238 6550 30  0000 C CNN
 F 3 "~" H 6200 6700 60  0000 C CNN
@@
 P 6450 6700
 F 0 "C190" H 6450 6800 40  0000 L CNN
-F 1 "0.1MFD" H 6456 6615 40  0000 L CNN
+F 1 "0.1mfd" H 6456 6615 40  0000 L CNN
 F 2 "~" H 6488 6550 30  0000 C CNN
 F 3 "~" H 6450 6700 60  0000 C CNN
@@
 P 6700 6700
 F 0 "C191" H 6700 6800 40  0000 L CNN
-F 1 "0.1MFD" H 6706 6615 40  0000 L CNN
+F 1 "0.1mfd" H 6706 6615 40  0000 L CNN
 F 2 "~" H 6738 6550 30  0000 C CNN
 F 3 "~" H 6700 6700 60  0000 C CNN
@@
 P 7000 6700
 F 0 "C192" H 7000 6800 40  0000 L CNN
-F 1 "0.1MFD" H 7006 6615 40  0000 L CNN
+F 1 "0.1mfd" H 7006 6615 40  0000 L CNN
 F 2 "~" H 7038 6550 30  0000 C CNN
 F 3 "~" H 7000 6700 60  0000 C CNN
@@
 P 7300 6700
 F 0 "C193" H 7300 6800 40  0000 L CNN
-F 1 "0.1MFD" H 7306 6615 40  0000 L CNN
+F 1 "0.1mfd" H 7306 6615 40  0000 L CNN
 F 2 "~" H 7338 6550 30  0000 C CNN
 F 3 "~" H 7300 6700 60  0000 C CNN
@@
 DDR0V9
 $Comp
-L PWR_FLAG #FLG03
+L PWR_FLAG #FLG02
 U 1 1 533EEDE3
 P 2500 3250
-F 0 "#FLG03" H 2500 3345 30  0001 C CNN
+F 0 "#FLG02" H 2500 3345 30  0001 C CNN
 F 1 "PWR_FLAG" H 2500 3430 30  0000 C CNN
 F 2 "" H 2500 3250 60  0000 C CNN
