File: board/cypress.sch (KiCad schematic (older format))
At the start: 5 parts

Commit message: Issue #336
Parts:
- gave numbers to parts that had none: 1
Changed lines of the file:
@@
 Sheet 3 5
 Title ""
-Date "19 jun 2013"
+Date "24 jun 2013"
 Rev ""
 Comp ""
@@
 $EndDescr
 $Comp
-L CY7C68013A U?
+L CY7C68013A U2
 U 5 1 51B6A1F5
 P 5500 4250
-F 0 "U?" H 5100 4900 60  0000 C CNN
+F 0 "U2" H 5100 4900 60  0000 C CNN
 F 1 "CY7C68013A" H 5300 3650 60  0000 C CNN
 F 2 "" H 5500 4250 60  0001 C CNN
@@
 $EndComp
 $Comp
-L CY7C68013A U?
+L CY7C68013A U2
 U 4 1 51B6A1E4
 P 7350 2200
-F 0 "U?" H 6950 2850 60  0000 C CNN
+F 0 "U2" H 6950 2850 60  0000 C CNN
 F 1 "CY7C68013A" H 7150 1600 60  0000 C CNN
 F 2 "" H 7350 2200 60  0001 C CNN
@@
 $EndComp
 $Comp
-L CY7C68013A U?
+L CY7C68013A U2
 U 3 1 51B6A1D7
 P 4900 2200
-F 0 "U?" H 4500 2850 60  0000 C CNN
+F 0 "U2" H 4500 2850 60  0000 C CNN
 F 1 "CY7C68013A" H 4700 1600 60  0000 C CNN
 F 2 "" H 4900 2200 60  0001 C CNN
@@
 $EndComp
 $Comp
-L CY7C68013A U?
+L CY7C68013A U2
 U 2 1 51B6A1CC
 P 2600 4300
-F 0 "U?" H 2200 4950 60  0000 C CNN
+F 0 "U2" H 2200 4950 60  0000 C CNN
 F 1 "CY7C68013A" H 2400 3700 60  0000 C CNN
 F 2 "" H 2600 4300 60  0001 C CNN
@@
 $EndComp
 $Comp
-L CY7C68013A U?
+L CY7C68013A U2
 U 1 1 51B6A1BD
 P 2550 2200
-F 0 "U?" H 2150 2850 60  0000 C CNN
+F 0 "U2" H 2150 2850 60  0000 C CNN
 F 1 "CY7C68013A" H 2350 1600 60  0000 C CNN
 F 2 "" H 2550 2200 60  0001 C CNN

Commit message: Issue #336
Parts:
- added C? (x8): 0.1MFD, ~, symbol C
- added C?: 47nF, ~, symbol C
- added C? (x2): 12pF, ~, symbol C
- added J?: USB_MICRO_B, ~, symbol USB_MICRO_B
- added R?: 100K, ~, symbol R
- added R? (x3): 75R, ~, symbol R
- added R? (x2): 10K, ~, symbol R
- added X?: CRYSTAL, ~, symbol CRYSTAL
Connections:
- net labels added: CY-FLAGA, CY-FLAGB, CY-FLAGC, CY-IFCLK, CY-SLRD, D_N, D_P, GND, VCC3V3
- wire segments 0 -> 53
Other:
- moved on the sheet: U2A, U2B, U2C, U2D, U2E

Commit message: Issue #336
Parts:
- gave numbers to parts that had none: 19
- renumbered U2 to U1
Changed lines of the file:
@@
 Sheet 2 7
 Title ""
-Date "27 jun 2013"
+Date "4 jul 2013"
 Rev ""
 Comp ""
@@
 $EndDescr
 $Comp
-L CY7C68013A U2
+L CY7C68013A U1
 U 5 1 51B6A1F5
 P 2100 6100
-F 0 "U2" H 1700 6750 60  0000 C CNN
+F 0 "U1" H 1700 6750 60  0000 C CNN
 F 1 "CY7C68013A" H 1900 5500 60  0000 C CNN
 F 2 "" H 2100 6100 60  0001 C CNN
@@
 $EndComp
 $Comp
-L CY7C68013A U2
+L CY7C68013A U1
 U 4 1 51B6A1E4
 P 8350 2300
-F 0 "U2" H 7950 2950 60  0000 C CNN
+F 0 "U1" H 7950 2950 60  0000 C CNN
 F 1 "CY7C68013A" H 8150 1700 60  0000 C CNN
 F 2 "" H 8350 2300 60  0001 C CNN
@@
 $EndComp
 $Comp
-L CY7C68013A U2
+L CY7C68013A U1
 U 3 1 51B6A1D7
 P 4450 2250
-F 0 "U2" H 4050 2900 60  0000 C CNN
+F 0 "U1" H 4050 2900 60  0000 C CNN
 F 1 "CY7C68013A" H 4250 1650 60  0000 C CNN
 F 2 "" H 4450 2250 60  0001 C CNN
@@
 $EndComp
 $Comp
-L CY7C68013A U2
+L CY7C68013A U1
 U 2 1 51B6A1CC
 P 2050 4300
-F 0 "U2" H 1650 4950 60  0000 C CNN
+F 0 "U1" H 1650 4950 60  0000 C CNN
 F 1 "CY7C68013A" H 1850 3700 60  0000 C CNN
 F 2 "" H 2050 4300 60  0001 C CNN
@@
 $EndComp
 $Comp
-L CY7C68013A U2
+L CY7C68013A U1
 U 1 1 51B6A1BD
 P 2100 2250
-F 0 "U2" H 1700 2900 60  0000 C CNN
+F 0 "U1" H 1700 2900 60  0000 C CNN
 F 1 "CY7C68013A" H 1900 1650 60  0000 C CNN
 F 2 "" H 2100 2250 60  0001 C CNN
@@
 Connection ~ 2850 6350
 $Comp
-L C C?
+L C C1
 U 1 1 51CCFF80
 P 3100 6700
-F 0 "C?" H 3100 6800 40  0000 L CNN
+F 0 "C1" H 3100 6800 40  0000 L CNN
 F 1 "0.1MFD" H 3106 6615 40  0000 L CNN
 F 2 "~" H 3138 6550 30  0000 C CNN
@@
 $EndComp
 $Comp
-L C C?
+L C C2
 U 1 1 51CCFFA2
 P 3350 6700
-F 0 "C?" H 3350 6800 40  0000 L CNN
+F 0 "C2" H 3350 6800 40  0000 L CNN
 F 1 "0.1MFD" H 3356 6615 40  0000 L CNN
 F 2 "~" H 3388 6550 30  0000 C CNN
@@
 $EndComp
 $Comp
-L C C?
+L C C3
 U 1 1 51CCFFA8
 P 3600 6700
-F 0 "C?" H 3600 6800 40  0000 L CNN
+F 0 "C3" H 3600 6800 40  0000 L CNN
 F 1 "0.1MFD" H 3606 6615 40  0000 L CNN
 F 2 "~" H 3638 6550 30  0000 C CNN
@@
 $EndComp
 $Comp
-L C C?
+L C C4
 U 1 1 51CCFFAE
 P 3850 6700
-F 0 "C?" H 3850 6800 40  0000 L CNN
+F 0 "C4" H 3850 6800 40  0000 L CNN
 F 1 "0.1MFD" H 3856 6615 40  0000 L CNN
 F 2 "~" H 3888 6550 30  0000 C CNN
@@
 $EndComp
 $Comp
-L C C?
+L C C5
 U 1 1 51CCFFB4
 P 4100 6700
-F 0 "C?" H 4100 6800 40  0000 L CNN
+F 0 "C5" H 4100 6800 40  0000 L CNN
 F 1 "0.1MFD" H 4106 6615 40  0000 L CNN
 F 2 "~" H 4138 6550 30  0000 C CNN
@@
 $EndComp
 $Comp
-L C C?
+L C C6
 U 1 1 51CCFFBA
 P 4350 6700
-F 0 "C?" H 4350 6800 40  0000 L CNN
+F 0 "C6" H 4350 6800 40  0000 L CNN
 F 1 "0.1MFD" H 4356 6615 40  0000 L CNN
 F 2 "~" H 4388 6550 30  0000 C CNN
@@
 $EndComp
 $Comp
-L C C?
+L C C7
 U 1 1 51CCFFC0
 P 4600 6700
-F 0 "C?" H 4600 6800 40  0000 L CNN
+F 0 "C7" H 4600 6800 40  0000 L CNN
 F 1 "0.1MFD" H 4606 6615 40  0000 L CNN
 F 2 "~" H 4638 6550 30  0000 C CNN
@@
 $EndComp
 $Comp
-L C C?
+L C C8
 U 1 1 51CCFFC6
 P 4850 6700
-F 0 "C?" H 4850 6800 40  0000 L CNN
+F 0 "C8" H 4850 6800 40  0000 L CNN
 F 1 "0.1MFD" H 4856 6615 40  0000 L CNN
 F 2 "~" H 4888 6550 30  0000 C CNN
@@
 Connection ~ 1300 6500
 $Comp
-L USB_MICRO_B J?
+L USB_MICRO_B J1
 U 1 1 51CD031B
 P 8400 3950
-F 0 "J?" H 8550 4350 60  0000 C CNN
+F 0 "J1" H 8550 4350 60  0000 C CNN
 F 1 "USB_MICRO_B" V 8200 3950 60  0000 C CNN
 F 2 "~" H 8400 3950 60  0000 C CNN
@@
 	8000 4150 7800 4150
 $Comp
-L GND #PWR?
+L GND #PWR01
 U 1 1 51CD0377
 P 3100 6950
-F 0 "#PWR?" H 3100 6950 30  0001 C CNN
+F 0 "#PWR01" H 3100 6950 30  0001 C CNN
 F 1 "GND" H 3100 6880 30  0001 C CNN
 F 2 "" H 3100 6950 60  0000 C CNN
@@
 	9100 2150 10350 2150
 $Comp
-L R R?
+L R R6
 U 1 1 51CD0685
 P 9900 1750
-F 0 "R?" V 9980 1750 40  0000 C CNN
+F 0 "R6" V 9980 1750 40  0000 C CNN
 F 1 "100K" V 9907 1751 40  0000 C CNN
 F 2 "~" V 9830 1750 30  0000 C CNN
@@
 $EndComp
 $Comp
-L C C?
+L C C11
 U 1 1 51CD06BB
 P 10550 2150
-F 0 "C?" H 10550 2250 40  0000 L CNN
+F 0 "C11" H 10550 2250 40  0000 L CNN
 F 1 "47nF" H 10556 2065 40  0000 L CNN
 F 2 "~" H 10588 2000 30  0000 C CNN
@@
 	10750 2150 10950 2150
 $Comp
-L C C?
+L C C9
 U 1 1 51CD0718
 P 6400 1800
-F 0 "C?" H 6400 1900 40  0000 L CNN
+F 0 "C9" H 6400 1900 40  0000 L CNN
 F 1 "12pF" H 6406 1715 40  0000 L CNN
 F 2 "~" H 6438 1650 30  0000 C CNN
@@
 	7150 2400 7150 2150
 $Comp
-L C C?
+L C C10
 U 1 1 51CD0AF0
 P 6400 2400
-F 0 "C?" H 6400 2500 40  0000 L CNN
+F 0 "C10" H 6400 2500 40  0000 L CNN
 F 1 "12pF" H 6406 2315 40  0000 L CNN
 F 2 "~" H 6438 2250 30  0000 C CNN
@@
 $EndComp
 $Comp
-L CRYSTAL X?
+L CRYSTAL X1
 U 1 1 51CD0B75
 P 6850 2100
-F 0 "X?" H 6850 2250 60  0000 C CNN
+F 0 "X1" H 6850 2250 60  0000 C CNN
 F 1 "CRYSTAL" H 6850 1950 60  0000 C CNN
 F 2 "~" H 6850 2100 60  0000 C CNN
@@
 	9100 2500 9250 2500
 $Comp
-L R R?
+L R R2
 U 1 1 51CD107F
 P 9500 2300
-F 0 "R?" V 9550 2100 40  0000 C CNN
+F 0 "R2" V 9550 2100 40  0000 C CNN
 F 1 "75R" V 9507 2301 40  0000 C CNN
 F 2 "~" V 9430 2300 30  0000 C CNN
@@
 	9900 2000 9900 2150
 $Comp
-L R R?
+L R R3
 U 1 1 51CD1113
 P 9500 2400
-F 0 "R?" V 9550 2200 40  0000 C CNN
+F 0 "R3" V 9550 2200 40  0000 C CNN
 F 1 "75R" V 9507 2401 40  0000 C CNN
 F 2 "~" V 9430 2400 30  0000 C CNN
@@
 $EndComp
 $Comp
-L R R?
+L R R4
 U 1 1 51CD1119
 P 9500 2500
-F 0 "R?" V 9550 2300 40  0000 C CNN
+F 0 "R4" V 9550 2300 40  0000 C CNN
 F 1 "75R" V 9507 2501 40  0000 C CNN
 F 2 "~" V 9430 2500 30  0000 C CNN
@@
 	7350 1400 7350 1800
 $Comp
-L R R?
+L R R1
 U 1 1 51CD1460
 P 7350 1150
-F 0 "R?" V 7430 1150 40  0000 C CNN
+F 0 "R1" V 7430 1150 40  0000 C CNN
 F 1 "10K" V 7357 1151 40  0000 C CNN
 F 2 "~" V 7280 1150 30  0000 C CNN
@@
 CY-SLRD
 $Comp
-L R R?
+L R R5
 U 1 1 51CD177C
 P 9750 1750
-F 0 "R?" V 9830 1750 40  0000 C CNN
+F 0 "R5" V 9830 1750 40  0000 C CNN
 F 1 "10K" V 9757 1751 40  0000 C CNN
 F 2 "~" V 9680 1750 30  0000 C CNN

Commit message: Issue #336
Connections:
- net labels added: U1-FLAGA, U1-FLAGB, U1-FLAGC, U1-IFCLK
- net labels removed: CY-FLAGA, CY-FLAGB, CY-FLAGC, CY-IFCLK, CY-SLRD
Changed lines of the file:
@@
 Sheet 2 7
 Title ""
-Date "8 jul 2013"
+Date "11 jul 2013"
 Rev ""
 Comp ""
@@
 	9750 2400 10200 2400
 Text Label 10200 2300 2    60   ~ 0
-CY-FLAGC
+U1-FLAGC
 Text Label 10200 2400 2    60   ~ 0
-CY-FLAGB
+U1-FLAGB
 Text Label 10200 2500 2    60   ~ 0
-CY-FLAGA
+U1-FLAGA
 Wire Wire Line
 	7550 2550 7350 2550
 Wire Wire Line
 	7350 1800 7550 1800
-Wire Wire Line
-	7350 1400 7350 1800
 $Comp
 L R R1
@@
 Text Label 6850 800  0    60   ~ 0
 VCC3V3
-Text Label 7350 1800 1    60   ~ 0
-CY-SLRD
 $Comp
 L R R5
@@
 	9100 1900 9550 1900
 Text Label 9550 1900 2    60   ~ 0
-CY-IFCLK
+U1-IFCLK
 Wire Wire Line
 	2800 3900 3150 3900
@@
 Text Label 5450 6900 2    60   ~ 0
 GND
+Wire Wire Line
+	7350 1400 7350 1800
 $EndSCHEMATC
