File: board/cypress.sch (KiCad schematic (older format))
At the start: 40 parts, among them J1 USB_MICRO_B, U1 CY7C68013A, X1 CRYSTAL

Commit message: Issue #336
Parts:
- added C34: 0.1MFD, ~, symbol C
- added R146: 4.7K, ~, symbol R
- added R147, R153: 1.8K, ~, symbol R
- added R151, R152, R154: 100R, ~, symbol R
- added U4: M25P16, symbol M25P16
- gave numbers to parts that had none: 20
Connections:
- net GND: now also C34.2, U4.4 (VSS)
- net VCC3V3: now also C34.1, R146.1, R147.1, R153.1, U4.8 (VCC)
- new net: R146.2, R151.2, U4.1 (~S)
- new net: R152.2, U4.2 (DQ1)
- new net: R153.2, U4.3 (~W)
- new net: R154.1, U4.5 (DQ0)
- new net: R147.2, U4.7 (~HOLD)
- new net SCK: U4.6 (C)
- new net SPI-CS-FLASH: R151.1
- new net SPI-SDI: R152.1
- new net SPI-SDO: R154.2
Changed lines of the file:
@@
 Sheet 2 7
 Title ""
-Date "13 jul 2013"
+Date "16 jul 2013"
 Rev ""
 Comp ""
@@
 GND
 $Comp
-L R R?
+L R R90
 U 1 1 520A85AA
 P 7250 1150
-F 0 "R?" V 7150 1150 40  0000 C CNN
+F 0 "R90" V 7150 1150 40  0000 C CNN
 F 1 "10K" V 7257 1151 40  0000 C CNN
 F 2 "~" V 7180 1150 30  0000 C CNN
@@
 U1-IFCLK
 $Comp
-L R R?
+L R R91
 U 1 1 520AAF05
 P 9600 1650
-F 0 "R?" V 9650 1450 40  0000 C CNN
+F 0 "R91" V 9650 1450 40  0000 C CNN
 F 1 "75R" V 9607 1651 40  0000 C CNN
 F 2 "~" V 9530 1650 30  0000 C CNN
@@
 $EndComp
 $Comp
-L R R?
+L R R84
 U 1 1 520AEFB9
 P 3850 2050
-F 0 "R?" V 3900 1850 40  0000 C CNN
+F 0 "R84" V 3900 1850 40  0000 C CNN
 F 1 "75R" V 3857 2051 40  0000 C CNN
 F 2 "~" V 3780 2050 30  0000 C CNN
@@
 $EndComp
 $Comp
-L R R?
+L R R86
 U 1 1 520AEFCF
 P 3850 2450
-F 0 "R?" V 3900 2250 40  0000 C CNN
+F 0 "R86" V 3900 2250 40  0000 C CNN
 F 1 "75R" V 3857 2451 40  0000 C CNN
 F 2 "~" V 3780 2450 30  0000 C CNN
@@
 $EndComp
 $Comp
-L R R?
+L R R87
 U 1 1 520AEFD5
 P 3850 2650
-F 0 "R?" V 3900 2450 40  0000 C CNN
+F 0 "R87" V 3900 2450 40  0000 C CNN
 F 1 "75R" V 3857 2651 40  0000 C CNN
 F 2 "~" V 3780 2650 30  0000 C CNN
@@
 $EndComp
 $Comp
-L R R?
+L R R83
 U 1 1 520AEFDB
 P 3850 1850
-F 0 "R?" V 3900 1650 40  0000 C CNN
+F 0 "R83" V 3900 1650 40  0000 C CNN
 F 1 "75R" V 3857 1851 40  0000 C CNN
 F 2 "~" V 3780 1850 30  0000 C CNN
@@
 $EndComp
 $Comp
-L R R?
+L R R88
 U 1 1 520AEFE1
 P 3850 2850
-F 0 "R?" V 3900 2650 40  0000 C CNN
+F 0 "R88" V 3900 2650 40  0000 C CNN
 F 1 "75R" V 3857 2851 40  0000 C CNN
 F 2 "~" V 3780 2850 30  0000 C CNN
@@
 $EndComp
 $Comp
-L R R?
+L R R85
 U 1 1 520AF4FA
 P 3850 2250
-F 0 "R?" V 3900 2050 40  0000 C CNN
+F 0 "R85" V 3900 2050 40  0000 C CNN
 F 1 "75R" V 3857 2251 40  0000 C CNN
 F 2 "~" V 3780 2250 30  0000 C CNN
@@
 $EndComp
 $Comp
-L R R?
+L R R74
 U 1 1 520AF91D
 P 3350 1450
-F 0 "R?" V 3300 1250 40  0000 C CNN
+F 0 "R74" V 3300 1250 40  0000 C CNN
 F 1 "10K" V 3357 1451 40  0000 C CNN
 F 2 "~" V 3280 1450 30  0000 C CNN
@@
 VCC3V3
 $Comp
-L R R?
+L R R73
 U 1 1 520AF926
 P 3250 1450
-F 0 "R?" V 3200 1250 40  0000 C CNN
+F 0 "R73" V 3200 1250 40  0000 C CNN
 F 1 "10K" V 3257 1451 40  0000 C CNN
 F 2 "~" V 3180 1450 30  0000 C CNN
@@
 $EndComp
 $Comp
-L R R?
+L R R72
 U 1 1 520AF92E
 P 3150 1450
-F 0 "R?" V 3100 1250 40  0000 C CNN
+F 0 "R72" V 3100 1250 40  0000 C CNN
 F 1 "10K" V 3157 1451 40  0000 C CNN
 F 2 "~" V 3080 1450 30  0000 C CNN
@@
 U1-SLCS
 $Comp
-L R R?
+L R R89
 U 1 1 520B2327
 P 3850 3100
-F 0 "R?" V 3800 2900 40  0000 C CNN
+F 0 "R89" V 3800 2900 40  0000 C CNN
 F 1 "10K" V 3857 3101 40  0000 C CNN
 F 2 "~" V 3780 3100 30  0000 C CNN
@@
 GND
 $Comp
-L R R?
+L R R75
 U 1 1 520B33A4
 P 3400 3550
-F 0 "R?" V 3450 3350 40  0000 C CNN
+F 0 "R75" V 3450 3350 40  0000 C CNN
 F 1 "75R" V 3407 3551 40  0000 C CNN
 F 2 "~" V 3330 3550 30  0000 C CNN
@@
 $EndComp
 $Comp
-L R R?
+L R R76
 U 1 1 520B33B9
 P 3400 3750
-F 0 "R?" V 3450 3550 40  0000 C CNN
+F 0 "R76" V 3450 3550 40  0000 C CNN
 F 1 "75R" V 3407 3751 40  0000 C CNN
 F 2 "~" V 3330 3750 30  0000 C CNN
@@
 $EndComp
 $Comp
-L R R?
+L R R77
 U 1 1 520B33BF
 P 3400 3950
-F 0 "R?" V 3450 3750 40  0000 C CNN
+F 0 "R77" V 3450 3750 40  0000 C CNN
 F 1 "75R" V 3407 3951 40  0000 C CNN
 F 2 "~" V 3330 3950 30  0000 C CNN
@@
 $EndComp
 $Comp
-L R R?
+L R R78
 U 1 1 520B33C5
 P 3400 4150
-F 0 "R?" V 3450 3950 40  0000 C CNN
+F 0 "R78" V 3450 3950 40  0000 C CNN
 F 1 "75R" V 3407 4151 40  0000 C CNN
 F 2 "~" V 3330 4150 30  0000 C CNN
@@
 $EndComp
 $Comp
-L R R?
+L R R79
 U 1 1 520B33CB
 P 3400 4350
-F 0 "R?" V 3450 4150 40  0000 C CNN
+F 0 "R79" V 3450 4150 40  0000 C CNN
 F 1 "75R" V 3407 4351 40  0000 C CNN
 F 2 "~" V 3330 4350 30  0000 C CNN
@@
 $EndComp
 $Comp
-L R R?
+L R R80
 U 1 1 520B33D1
 P 3400 4550
-F 0 "R?" V 3450 4350 40  0000 C CNN
+F 0 "R80" V 3450 4350 40  0000 C CNN
 F 1 "75R" V 3407 4551 40  0000 C CNN
 F 2 "~" V 3330 4550 30  0000 C CNN
@@
 $EndComp
 $Comp
-L R R?
+L R R81
 U 1 1 520B33E7
 P 3400 4750
-F 0 "R?" V 3450 4550 40  0000 C CNN
+F 0 "R81" V 3450 4550 40  0000 C CNN
 F 1 "75R" V 3407 4751 40  0000 C CNN
 F 2 "~" V 3330 4750 30  0000 C CNN
@@
 $EndComp
 $Comp
-L R R?
+L R R82
 U 1 1 520B33ED
 P 3400 4950
-F 0 "R?" V 3450 4750 40  0000 C CNN
+F 0 "R82" V 3450 4750 40  0000 C CNN
 F 1 "75R" V 3407 4951 40  0000 C CNN
 F 2 "~" V 3330 4950 30  0000 C CNN
@@
 NoConn ~ 8000 4050
 NoConn ~ 9100 1800
+$Comp
+L M25P16 U4
+U 1 1 51E42548
+P 8250 5550
+F 0 "U4" H 8250 5050 60  0000 C CNN
+F 1 "M25P16" H 8250 6000 60  0000 C CNN
+F 2 "" H 8250 5550 60  0000 C CNN
+F 3 "" H 8250 5550 60  0000 C CNN
+	1    8250 5550
+	1    0    0    -1
+$EndComp
+$Comp
+L C C34
+U 1 1 51E7848B
+P 9150 4900
+F 0 "C34" H 9150 5000 40  0000 L CNN
+F 1 "0.1MFD" H 9156 4815 40  0000 L CNN
+F 2 "~" H 9188 4750 30  0000 C CNN
+F 3 "~" H 9150 4900 60  0000 C CNN
+	1    9150 4900
+	1    0    0    -1
+$EndComp
+Wire Wire Line
+	9150 4600 9150 4700
+Connection ~ 9150 4600
+Wire Wire Line
+	9150 5100 9400 5100
+Text Label 9400 5100 2    60   ~ 0
+GND
+$Comp
+L R R147
+U 1 1 51E78785
+P 9500 4950
+F 0 "R147" V 9400 5000 40  0000 C CNN
+F 1 "1.8K" V 9507 4951 40  0000 C CNN
+F 2 "~" V 9430 4950 30  0000 C CNN
+F 3 "~" H 9500 4950 30  0000 C CNN
+	1    9500 4950
+	1    0    0    -1
+$EndComp
+Wire Wire Line
+	9500 4700 9500 4600
+Connection ~ 9500 4600
+Wire Wire Line
+	8950 5500 9500 5500
+Wire Wire Line
+	9500 5500 9500 5200
+$Comp
+L R R146
+U 1 1 51E785B7
+P 7550 4950
+F 0 "R146" V 7630 4950 40  0000 C CNN
+F 1 "4.7K" V 7557 4951 40  0000 C CNN
+F 2 "~" V 7480 4950 30  0000 C CNN
+F 3 "~" H 7550 4950 30  0000 C CNN
+	1    7550 4950
+	1    0    0    -1
+$EndComp
+Wire Wire Line
+	7550 5350 7550 5200
+Wire Wire Line
+	7550 4700 7550 4600
+Wire Wire Line
+	7350 4600 9850 4600
+Text Label 9850 4600 2    60   ~ 0
+VCC3V3
+Wire Wire Line
+	8950 5350 8950 4600
+Connection ~ 8950 4600
+Wire Wire Line
+	7550 5800 7300 5800
+Text Label 7300 5800 0    60   ~ 0
+GND
+$Comp
+L R R153
+U 1 1 51E60F08
+P 7350 4950
+F 0 "R153" V 7430 4950 40  0000 C CNN
+F 1 "1.8K" V 7357 4951 40  0000 C CNN
+F 2 "~" V 7280 4950 30  0000 C CNN
+F 3 "~" H 7350 4950 30  0000 C CNN
+	1    7350 4950
+	1    0    0    -1
+$EndComp
+Wire Wire Line
+	7550 5650 7350 5650
+Wire Wire Line
+	7350 4700 7350 4600
+Connection ~ 7550 4600
+Text HLabel 6600 5500 0    60   BiDi ~ 0
+SPI-SDI
+Text HLabel 9600 5800 2    60   BiDi ~ 0
+SPI-SDO
+Wire Wire Line
+	7350 5650 7350 5200
+Text HLabel 8950 5650 2    60   BiDi ~ 0
+SCK
+Wire Wire Line
+	7550 5500 7200 5500
+Wire Wire Line
+	7550 5350 7200 5350
+Text HLabel 6600 5350 0    60   BiDi ~ 0
+SPI-CS-FLASH
+$Comp
+L R R151
+U 1 1 51E8D361
+P 6950 5350
+F 0 "R151" V 7030 5350 40  0000 C CNN
+F 1 "100R" V 6957 5351 40  0000 C CNN
+F 2 "~" V 6880 5350 30  0000 C CNN
+F 3 "~" H 6950 5350 30  0000 C CNN
+	1    6950 5350
+	0    -1   -1   0
+$EndComp
+Wire Wire Line
+	6700 5350 6600 5350
+$Comp
+L R R152
+U 1 1 51E8DB9E
+P 6950 5500
+F 0 "R152" V 7030 5500 40  0000 C CNN
+F 1 "100R" V 6957 5501 40  0000 C CNN
+F 2 "~" V 6880 5500 30  0000 C CNN
+F 3 "~" H 6950 5500 30  0000 C CNN
+	1    6950 5500
+	0    -1   -1   0
+$EndComp
+Wire Wire Line
+	6700 5500 6600 5500
+$Comp
+L R R154
+U 1 1 51E8DC4B
+P 9300 5800
+F 0 "R154" V 9380 5800 40  0000 C CNN
+F 1 "100R" V 9307 5801 40  0000 C CNN
+F 2 "~" V 9230 5800 30  0000 C CNN
+F 3 "~" H 9300 5800 30  0000 C CNN
+	1    9300 5800
+	0    -1   -1   0
+$EndComp
+Wire Wire Line
+	9050 5800 8950 5800
+Wire Wire Line
+	9550 5800 9600 5800
 $EndSCHEMATC

Commit message: Issue #336
Parts:
- added R? (x2): 2.2K, ~, symbol R
Connections:
- net VCC3V3: now also R?.2, R?.2
- net U1-SCL: now reaches U1.15 (SCL)
- net U1-SCL: now also R?.1
- net U1-SDA: now reaches U1.16 (SDA)
- net U1-SDA: now also R?.1
Other:
- moved on the sheet: C10, C11, C34, C9, J1, R1, R146, R147, R151, R152, R153, R154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

Commit message: Issue #346
Parts:
- gave numbers to parts that had none: 2
Changed lines of the file:
@@
 Sheet 2 7
 Title ""
-Date "18 jul 2013"
+Date "30 jul 2013"
 Rev ""
 Comp ""
@@
 $EndComp
 $Comp
-L R R?
+L R R174
 U 1 1 51E6C161
 P 7450 3000
-F 0 "R?" V 7530 3000 40  0000 C CNN
+F 0 "R174" V 7530 3000 40  0000 C CNN
 F 1 "2.2K" V 7457 3001 40  0000 C CNN
 F 2 "~" V 7380 3000 30  0000 C CNN
@@
 $EndComp
 $Comp
-L R R?
+L R R175
 U 1 1 51E6C171
 P 7650 3000
-F 0 "R?" V 7730 3000 40  0000 C CNN
+F 0 "R175" V 7730 3000 40  0000 C CNN
 F 1 "2.2K" V 7657 3001 40  0000 C CNN
 F 2 "~" V 7580 3000 30  0000 C CNN

Commit message: Issue #344
Parts:
- renumbered C8 to C10, C34 to C12, C9 to C7, C10 to C8, C7 to C9, R72 to R1, R81 to R10, R82 to R11, R83 to R12, R84 to R13, R85 to R14, R86 to R15, R87 to R16, R88 to R17, R89 to R18, R90 to R19, R73 to R2, R1 to R20, R151 to R21, R152 to R22, R174 to R23, R153 to R24, R2 to R25, R3 to R26, R4 to R27, R175 to R28, R91 to R29, R74 to R3, R146 to R30, R5 to R31, R6 to R32, R154 to R33, R147 to R34, R75 to R4, R76 to R5, R77 to R6, R78 to R7, R79 to R8, R80 to R9, U4 to U2
Connections:
- net GND: now also C2.2, C3.2, C4.2, C5.2, C6.2, C9.2
- no-connect marks 2 -> 4
Changed lines of the file:
@@
 Sheet 2 7
 Title ""
-Date "30 jul 2013"
+Date "31 jul 2013"
 Rev ""
 Comp ""
@@
 $EndComp
 $Comp
-L C C7
+L C C9
 U 1 1 51CCFFC0
 P 4600 6700
-F 0 "C7" H 4600 6800 40  0000 L CNN
+F 0 "C9" H 4600 6800 40  0000 L CNN
 F 1 "0.1MFD" H 4606 6615 40  0000 L CNN
 F 2 "~" H 4638 6550 30  0000 C CNN
@@
 $EndComp
 $Comp
-L C C8
+L C C10
 U 1 1 51CCFFC6
 P 4850 6700
-F 0 "C8" H 4850 6800 40  0000 L CNN
+F 0 "C10" H 4850 6800 40  0000 L CNN
 F 1 "0.1MFD" H 4856 6615 40  0000 L CNN
 F 2 "~" H 4888 6550 30  0000 C CNN
@@
 VCC3V3
 $Comp
-L R R6
+L R R32
 U 1 1 51CD0685
 P 8050 1650
-F 0 "R6" V 8130 1650 40  0000 C CNN
+F 0 "R32" V 8130 1650 40  0000 C CNN
 F 1 "100K" V 8057 1651 40  0000 C CNN
 F 2 "~" V 7980 1650 30  0000 C CNN
@@
 $EndComp
 $Comp
-L C C9
+L C C7
 U 1 1 51CD0718
 P 4550 1700
-F 0 "C9" H 4550 1800 40  0000 L CNN
+F 0 "C7" H 4550 1800 40  0000 L CNN
 F 1 "12pF" H 4556 1615 40  0000 L CNN
 F 2 "~" H 4588 1550 30  0000 C CNN
@@
 VCC3V3
 $Comp
-L C C10
+L C C8
 U 1 1 51CD0AF0
 P 4550 2300
-F 0 "C10" H 4550 2400 40  0000 L CNN
+F 0 "C8" H 4550 2400 40  0000 L CNN
 F 1 "12pF" H 4556 2215 40  0000 L CNN
 F 2 "~" H 4588 2150 30  0000 C CNN
@@
 D_P
 $Comp
-L R R2
+L R R25
 U 1 1 51CD107F
 P 7650 2200
-F 0 "R2" V 7700 2000 40  0000 C CNN
+F 0 "R25" V 7700 2000 40  0000 C CNN
 F 1 "75R" V 7657 2201 40  0000 C CNN
 F 2 "~" V 7580 2200 30  0000 C CNN
@@
 $EndComp
 $Comp
-L R R3
+L R R26
 U 1 1 51CD1113
 P 7650 2300
-F 0 "R3" V 7700 2100 40  0000 C CNN
+F 0 "R26" V 7700 2100 40  0000 C CNN
 F 1 "75R" V 7657 2301 40  0000 C CNN
 F 2 "~" V 7580 2300 30  0000 C CNN
@@
 $EndComp
 $Comp
-L R R4
+L R R27
 U 1 1 51CD1119
 P 7650 2400
-F 0 "R4" V 7700 2200 40  0000 C CNN
+F 0 "R27" V 7700 2200 40  0000 C CNN
 F 1 "75R" V 7657 2401 40  0000 C CNN
 F 2 "~" V 7580 2400 30  0000 C CNN
@@
 $EndComp
 $Comp
-L R R1
+L R R20
 U 1 1 51CD1460
 P 5500 1050
-F 0 "R1" V 5580 1050 40  0000 C CNN
+F 0 "R20" V 5580 1050 40  0000 C CNN
 F 1 "10K" V 5507 1051 40  0000 C CNN
 F 2 "~" V 5430 1050 30  0000 C CNN
@@
 VCC3V3
 $Comp
-L R R5
+L R R31
 U 1 1 51CD177C
 P 7900 1650
-F 0 "R5" V 7980 1650 40  0000 C CNN
+F 0 "R31" V 7980 1650 40  0000 C CNN
 F 1 "10K" V 7907 1651 40  0000 C CNN
 F 2 "~" V 7830 1650 30  0000 C CNN
@@
 GND
 $Comp
-L R R90
+L R R19
 U 1 1 520A85AA
 P 5400 1050
-F 0 "R90" V 5300 1050 40  0000 C CNN
+F 0 "R19" V 5300 1050 40  0000 C CNN
 F 1 "10K" V 5407 1051 40  0000 C CNN
 F 2 "~" V 5330 1050 30  0000 C CNN
@@
 U1-IFCLK
 $Comp
-L R R91
+L R R29
 U 1 1 520AAF05
 P 7750 1550
-F 0 "R91" V 7800 1350 40  0000 C CNN
+F 0 "R29" V 7800 1350 40  0000 C CNN
 F 1 "75R" V 7757 1551 40  0000 C CNN
 F 2 "~" V 7680 1550 30  0000 C CNN
@@
 $EndComp
 $Comp
-L R R84
+L R R13
 U 1 1 520AEFB9
 P 2900 1550
-F 0 "R84" V 2950 1350 40  0000 C CNN
+F 0 "R13" V 2950 1350 40  0000 C CNN
 F 1 "75R" V 2907 1551 40  0000 C CNN
 F 2 "~" V 2830 1550 30  0000 C CNN
@@
 $EndComp
 $Comp
-L R R86
+L R R15
 U 1 1 520AEFCF
 P 2900 1950
-F 0 "R86" V 2950 1750 40  0000 C CNN
+F 0 "R15" V 2950 1750 40  0000 C CNN
 F 1 "75R" V 2907 1951 40  0000 C CNN
 F 2 "~" V 2830 1950 30  0000 C CNN
@@
 $EndComp
 $Comp
-L R R87
+L R R16
 U 1 1 520AEFD5
 P 2900 2150
-F 0 "R87" V 2950 1950 40  0000 C CNN
+F 0 "R16" V 2950 1950 40  0000 C CNN
 F 1 "75R" V 2907 2151 40  0000 C CNN
 F 2 "~" V 2830 2150 30  0000 C CNN
@@
 $EndComp
 $Comp
-L R R83
+L R R12
 U 1 1 520AEFDB
 P 2900 1350
-F 0 "R83" V 2950 1150 40  0000 C CNN
+F 0 "R12" V 2950 1150 40  0000 C CNN
 F 1 "75R" V 2907 1351 40  0000 C CNN
 F 2 "~" V 2830 1350 30  0000 C CNN
@@
 $EndComp
 $Comp
-L R R88
+L R R17
 U 1 1 520AEFE1
 P 2900 2350
-F 0 "R88" V 2950 2150 40  0000 C CNN
+F 0 "R17" V 2950 2150 40  0000 C CNN
 F 1 "75R" V 2907 2351 40  0000 C CNN
 F 2 "~" V 2830 2350 30  0000 C CNN
@@
 $EndComp
 $Comp
-L R R85
+L R R14
 U 1 1 520AF4FA
 P 2900 1750
-F 0 "R85" V 2950 1550 40  0000 C CNN
+F 0 "R14" V 2950 1550 40  0000 C CNN
 F 1 "75R" V 2907 1751 40  0000 C CNN
 F 2 "~" V 2830 1750 30  0000 C CNN
@@
 $EndComp
 $Comp
-L R R74
+L R R3
 U 1 1 520AF91D
 P 2400 950
-F 0 "R74" V 2350 750 40  0000 C CNN
+F 0 "R3" V 2350 750 40  0000 C CNN
 F 1 "10K" V 2407 951 40  0000 C CNN
 F 2 "~" V 2330 950 30  0000 C CNN
@@
 VCC3V3
 $Comp
-L R R73
+L R R2
 U 1 1 520AF926
 P 2300 950
-F 0 "R73" V 2250 750 40  0000 C CNN
+F 0 "R2" V 2250 750 40  0000 C CNN
 F 1 "10K" V 2307 951 40  0000 C CNN
 F 2 "~" V 2230 950 30  0000 C CNN
@@
 $EndComp
 $Comp
-L R R72
+L R R1
 U 1 1 520AF92E
 P 2200 950
-F 0 "R72" V 2150 750 40  0000 C CNN
+F 0 "R1" V 2150 750 40  0000 C CNN
 F 1 "10K" V 2207 951 40  0000 C CNN
 F 2 "~" V 2130 950 30  0000 C CNN
@@
 U1-SLCS
 $Comp
-L R R89
+L R R18
 U 1 1 520B2327
 P 2900 2600
-F 0 "R89" V 2850 2400 40  0000 C CNN
+F 0 "R18" V 2850 2400 40  0000 C CNN
 F 1 "10K" V 2907 2601 40  0000 C CNN
 F 2 "~" V 2830 2600 30  0000 C CNN
@@
 GND
 $Comp
-L R R75
+L R R4
 U 1 1 520B33A4
 P 2650 2900
-F 0 "R75" V 2700 2700 40  0000 C CNN
+F 0 "R4" V 2700 2700 40  0000 C CNN
 F 1 "75R" V 2657 2901 40  0000 C CNN
 F 2 "~" V 2580 2900 30  0000 C CNN
@@
 $EndComp
 $Comp
-L R R76
+L R R5
 U 1 1 520B33B9
 P 2650 3100
-F 0 "R76" V 2700 2900 40  0000 C CNN
+F 0 "R5" V 2700 2900 40  0000 C CNN
 F 1 "75R" V 2657 3101 40  0000 C CNN
 F 2 "~" V 2580 3100 30  0000 C CNN
@@
 $EndComp
 $Comp
-L R R77
+L R R6
 U 1 1 520B33BF
 P 2650 3300
-F 0 "R77" V 2700 3100 40  0000 C CNN
+F 0 "R6" V 2700 3100 40  0000 C CNN
 F 1 "75R" V 2657 3301 40  0000 C CNN
 F 2 "~" V 2580 3300 30  0000 C CNN
@@
 $EndComp
 $Comp
-L R R78
+L R R7
 U 1 1 520B33C5
 P 2650 3500
-F 0 "R78" V 2700 3300 40  0000 C CNN
+F 0 "R7" V 2700 3300 40  0000 C CNN
 F 1 "75R" V 2657 3501 40  0000 C CNN
 F 2 "~" V 2580 3500 30  0000 C CNN
@@
 $EndComp
 $Comp
-L R R79
+L R R8
 U 1 1 520B33CB
 P 2650 3700
-F 0 "R79" V 2700 3500 40  0000 C CNN
+F 0 "R8" V 2700 3500 40  0000 C CNN
 F 1 "75R" V 2657 3701 40  0000 C CNN
 F 2 "~" V 2580 3700 30  0000 C CNN
@@
 $EndComp
 $Comp
-L R R80
+L R R9
 U 1 1 520B33D1
 P 2650 3900
-F 0 "R80" V 2700 3700 40  0000 C CNN
+F 0 "R9" V 2700 3700 40  0000 C CNN
 F 1 "75R" V 2657 3901 40  0000 C CNN
 F 2 "~" V 2580 3900 30  0000 C CNN
@@
 $EndComp
 $Comp
-L R R81
+L R R10
 U 1 1 520B33E7
 P 2650 4100
-F 0 "R81" V 2700 3900 40  0000 C CNN
+F 0 "R10" V 2700 3900 40  0000 C CNN
 F 1 "75R" V 2657 4101 40  0000 C CNN
 F 2 "~" V 2580 4100 30  0000 C CNN
@@
 $EndComp
 $Comp
-L R R82
+L R R11
 U 1 1 520B33ED
 P 2650 4300
-F 0 "R82" V 2700 4100 40  0000 C CNN
+F 0 "R11" V 2700 4100 40  0000 C CNN
 F 1 "75R" V 2657 4301 40  0000 C CNN
 F 2 "~" V 2580 4300 30  0000 C CNN
@@
 NoConn ~ 7250 1700
 $Comp
-L M25P16 U4
+L M25P16 U2
 U 1 1 51E42548
 P 8500 5350
-F 0 "U4" H 8500 4850 60  0000 C CNN
+F 0 "U2" H 8500 4850 60  0000 C CNN
 F 1 "M25P16" H 8500 5800 60  0000 C CNN
 F 2 "" H 8500 5350 60  0000 C CNN
@@
 $EndComp
 $Comp
-L C C34
+L C C12
 U 1 1 51E7848B
 P 9400 4700
-F 0 "C34" H 9400 4800 40  0000 L CNN
+F 0 "C12" H 9400 4800 40  0000 L CNN
 F 1 "0.1MFD" H 9406 4615 40  0000 L CNN
 F 2 "~" H 9438 4550 30  0000 C CNN
@@
 GND
 $Comp
-L R R147
+L R R34
 U 1 1 51E78785
 P 9750 4750
-F 0 "R147" V 9650 4800 40  0000 C CNN
+F 0 "R34" V 9650 4800 40  0000 C CNN
 F 1 "1.8K" V 9757 4751 40  0000 C CNN
 F 2 "~" V 9680 4750 30  0000 C CNN
@@
 $EndComp
 $Comp
-L R R146
+L R R30
 U 1 1 51E785B7
 P 7800 4750
-F 0 "R146" V 7880 4750 40  0000 C CNN
+F 0 "R30" V 7880 4750 40  0000 C CNN
 F 1 "4.7K" V 7807 4751 40  0000 C CNN
 F 2 "~" V 7730 4750 30  0000 C CNN
@@
 GND
 $Comp
-L R R153
+L R R24
 U 1 1 51E60F08
 P 7600 4750
-F 0 "R153" V 7680 4750 40  0000 C CNN
+F 0 "R24" V 7680 4750 40  0000 C CNN
 F 1 "1.8K" V 7607 4751 40  0000 C CNN
 F 2 "~" V 7530 4750 30  0000 C CNN
@@
 SPI-CS-FLASH
 $Comp
-L R R151
+L R R21
 U 1 1 51E8D361
 P 7200 5150
-F 0 "R151" V 7280 5150 40  0000 C CNN
+F 0 "R21" V 7280 5150 40  0000 C CNN
 F 1 "100R" V 7207 5151 40  0000 C CNN
 F 2 "~" V 7130 5150 30  0000 C CNN
@@
 $EndComp
 $Comp
-L R R152
+L R R22
 U 1 1 51E8DB9E
 P 7200 5300
-F 0 "R152" V 7280 5300 40  0000 C CNN
+F 0 "R22" V 7280 5300 40  0000 C CNN
 F 1 "100R" V 7207 5301 40  0000 C CNN
 F 2 "~" V 7130 5300 30  0000 C CNN
@@
 $EndComp
 $Comp
-L R R154
+L R R33
 U 1 1 51E8DC4B
 P 9550 5600
-F 0 "R154" V 9630 5600 40  0000 C CNN
+F 0 "R33" V 9630 5600 40  0000 C CNN
 F 1 "100R" V 9557 5601 40  0000 C CNN
 F 2 "~" V 9480 5600 30  0000 C CNN
@@
 $EndComp
 $Comp
-L R R174
+L R R23
 U 1 1 51E6C161
 P 7450 3000
-F 0 "R174" V 7530 3000 40  0000 C CNN
+F 0 "R23" V 7530 3000 40  0000 C CNN
 F 1 "2.2K" V 7457 3001 40  0000 C CNN
 F 2 "~" V 7380 3000 30  0000 C CNN
@@
 $EndComp
 $Comp
-L R R175
+L R R28
 U 1 1 51E6C171
 P 7650 3000
-F 0 "R175" V 7730 3000 40  0000 C CNN
+F 0 "R28" V 7730 3000 40  0000 C CNN
 F 1 "2.2K" V 7657 3001 40  0000 C CNN
 F 2 "~" V 7580 3000 30  0000 C CNN
@@
 	7450 3250 7450 3300
 Connection ~ 7450 3300
+NoConn ~ 10100 1400
+Connection ~ 3350 6900
+Connection ~ 3600 6900
+Connection ~ 3850 6900
+Connection ~ 4100 6900
+Connection ~ 4350 6900
+Connection ~ 4600 6900
+NoConn ~ 2050 1650
 $EndSCHEMATC
