File: board/hdmi.sch (KiCad schematic (older format))
At the start: 0 parts

Commit message: Issue #336
Parts:
- added J?: HDMI, ~, symbol HDMI
- added U?: IP4776CZ38, symbol IP4776CZ38
Connections:
- new net GND: J?.11 (CLKS), J?.17 (DDC/CEC/HEC), J?.2 (D2S), J?.5 (D1S), J?.8 (D0S), U?.11 (TMDS_GND), U?.14 (TMDS_GND), U?.25 (TMDS_GND), U?.28 (TMDS_GND), U?.3 (GND), U?.31 (TMDS_GND), U?.34 (TMDS_GND), U?.36 (GND), U?.5 (TMDS_GND), U?.8 (TMDS_GND)
Other:
- note added: "HDMI IN"
Changed lines of the file:
@@
 $Descr A4 11693 8268
 encoding utf-8
-Sheet 6 7
+Sheet 5 7
 Title ""
-Date "27 jun 2013"
+Date "4 jul 2013"
 Rev ""
 Comp ""
@@
 Comment4 ""
 $EndDescr
+$Comp
+L HDMI J?
+U 1 1 51D80ADD
+P 9450 2450
+F 0 "J?" H 9150 3500 60  0000 C CNN
+F 1 "HDMI" V 9600 2450 60  0000 C CNN
+F 2 "~" H 9400 2450 60  0000 C CNN
+F 3 "~" H 9400 2450 60  0000 C CNN
+	1    9450 2450
+	1    0    0    -1
+$EndComp
+$Comp
+L IP4776CZ38 U?
+U 1 1 51D81222
+P 6200 2250
+F 0 "U?" H 5550 3400 60  0000 C CNN
+F 1 "IP4776CZ38" H 5750 1100 60  0000 C CNN
+F 2 "" H 6200 2250 60  0000 C CNN
+F 3 "" H 6200 2250 60  0000 C CNN
+	1    6200 2250
+	1    0    0    -1
+$EndComp
+Text Notes 9400 1300 0    60   ~ 0
+HDMI IN
+Wire Wire Line
+	8900 2250 8800 2250
+Connection ~ 8800 2250
+Wire Wire Line
+	8900 2550 8800 2550
+Connection ~ 8800 2550
+Wire Wire Line
+	8900 3150 8800 3150
+Connection ~ 8800 3150
+Wire Wire Line
+	8800 3650 9000 3650
+Text Label 9000 3650 2    60   ~ 0
+GND
+Wire Wire Line
+	7150 1600 7250 1600
+Wire Wire Line
+	7250 1600 7250 3600
+Wire Wire Line
+	7150 2700 7250 2700
+Connection ~ 7250 2700
+Wire Wire Line
+	7150 2400 7250 2400
+Connection ~ 7250 2400
+Wire Wire Line
+	7150 2100 7250 2100
+Connection ~ 7250 2100
+Wire Wire Line
+	7150 1800 7250 1800
+Connection ~ 7250 1800
+Wire Wire Line
+	5300 1600 5150 1600
+Wire Wire Line
+	5150 1600 5150 3450
+Wire Wire Line
+	5300 1800 5150 1800
+Connection ~ 5150 1800
+Wire Wire Line
+	5300 2100 5150 2100
+Connection ~ 5150 2100
+Wire Wire Line
+	5300 2400 5150 2400
+Connection ~ 5150 2400
+Wire Wire Line
+	5300 2700 5150 2700
+Connection ~ 5150 2700
+Text Label 7450 3600 2    60   ~ 0
+GND
+Wire Wire Line
+	7250 3600 7450 3600
+Wire Wire Line
+	5150 3450 7250 3450
+Connection ~ 7250 3450
+Wire Wire Line
+	8900 1650 8800 1650
+Wire Wire Line
+	8800 1650 8800 3650
+Wire Wire Line
+	8900 1950 8800 1950
+Connection ~ 8800 1950
 $EndSCHEMATC

Commit message: Issue #336
Parts:
- added C?: C, ~, symbol C
- added J?: HDMI, ~, symbol HDMI
- added R? (x8): R, ~, symbol R
- added R? (x2): 1.5K, ~, symbol R
- added R? (x2): 47K, ~, symbol R
Connections:
- net TMDS-RX-2_P: now reaches J?.1 (D2+)
- net TMDS-RX-2_P: now also U?.4 (TMDS_D2+)
- net TMDS-RX-CLK_P: now reaches J?.10 (CLK+)
- net TMDS-RX-CLK_P: now also U?.13 (TMDS_CLK+)
- net TMDS-RX-CLK_N: now reaches J?.12 (CLK-)
- net TMDS-RX-CLK_N: now also U?.24 (TMDS_CLK-)
- net DDC-SCL: now reaches J?.15 (SCL)
- net DDC-SCL: now also U?.22 (DDC_CLK_OUT), R?.2
- net DDC-SDA: now reaches J?.16 (SDA)
- net DDC-SDA: now also U?.21 (DDC_DAT_OUT), R?.2
- net TMDS-RX-2_N: now reaches J?.3 (D2-)
- net TMDS-RX-2_N: now also U?.33 (TMDS_D2-)
- net TMDS-RX-1_P: now reaches J?.4 (D1+)
- net TMDS-RX-1_P: now also U?.7 (TMDS_D1+)
- net TMDS-RX-1_N: now reaches J?.6 (D1-)
- net TMDS-RX-1_N: now also U?.30 (TMDS_D1-)
- net TMDS-RX-0_P: now reaches J?.7 (D0+)
- net TMDS-RX-0_P: now also U?.10 (TMDS_D0+)
- net TMDS-RX-0_N: now reaches J?.9 (D0-)
- net TMDS-RX-0_N: now also U?.27 (TMDS_D0-)
- net VCC5V0: now reaches U?.1 (VCC(5V0))
- net VCC5V0: now also R?.1
- net TMDS-RX-SCL: now reaches U?.17 (DDC_CLK_IN)
- net TMDS-RX-SCL: now also R?.2
- net TMDS-RX-SDA: now reaches U?.18 (DDC_DAT_IN)
- net TMDS-RX-SDA: now also R?.2
- net VCC3V3: now reaches U?.2 (VCC(3V3))
- net VCC3V3: now also R?.1
- net at U?.37 (TMDS_BIAS): now also C?.1
- net GND renamed VSS
- net VSS: now also C?.2, J?.11 (CLKS), J?.17 (DDC/CEC/HEC), J?.2 (D2S), J?.5 (D1S), J?.8 (D0S)
- new net: J?.1 (D2+), R?.2
- new net: J?.10 (CLK+), R?.2
- new net: J?.12 (CLK-), R?.2
- new net: J?.3 (D2-), R?.2
- new net: J?.6 (D1-), R?.2
- new net: J?.7 (D0+), R?.2
- new net: J?.9 (D0-), R?.2
- new net JA-CLK_N: R?.1
- new net JA-CLK_P: R?.1
- new net JA-D0_N: R?.1
- new net JA-D0_P: R?.1
- new net JA-D1_N: R?.1
- new net JA-D1_P: R?.1
- new net JA-D2_N: R?.1
- new net JA-D2_P: R?.1
- no-connect marks 0 -> 4
Other:
- note added: "HDMI P1"
- note added: "HDMI P2"
- note removed: "HDMI IN"
- moved on the sheet: J?, U?

Commit message: Issue #336
Parts:
- removed J?: HDMI, ~, symbol HDMI
- removed R? (x8): R, ~, symbol R
- added C?: C, ~, symbol C
- added J?: HDMI, ~, symbol HDMI
- added R? (x2): 1.5K, ~, symbol R
- added R? (x2): 47K, ~, symbol R
- added U?: IP4776CZ38, symbol IP4776CZ38
Connections:
- net labels added: P1-CLK+, P1-CLK-, P1-D0+, P1-D0-, P1-D1+, P1-D1-, P1-D2+, P1-D2-, P2-CLK+, P2-CLK-, P2-D0+, P2-D0-, P2-D1+, P2-D1-, P2-D2+, P2-D2-, TMDS-RX1-0_N, TMDS-RX1-0_P, TMDS-RX1-1_N, TMDS-RX1-1_P, TMDS-RX1-2_N, TMDS-RX1-2_P, TMDS-RX1-CLK_N, TMDS-RX1-CLK_P, TMDS-RX1-SCL, TMDS-RX1-SDA, TMDS-TX1-0_N, TMDS-TX1-0_P, TMDS-TX1-1_N, TMDS-TX1-1_P, TMDS-TX1-2_N, TMDS-TX1-2_P, TMDS-TX1-CLK_N, TMDS-TX1-CLK_P
- net labels removed: CLK+, CLK-, D0+, D0-, D1+, D1-, D2+, D2-, JA-CLK_N, JA-CLK_P, JA-D0_N, JA-D0_P, JA-D1_N, JA-D1_P, JA-D2_N, JA-D2_P, TMDS-RX-0_N, TMDS-RX-0_P, TMDS-RX-1_N, TMDS-RX-1_P, TMDS-RX-2_N, TMDS-RX-2_P, TMDS-RX-CLK_N, TMDS-RX-CLK_P, TMDS-RX-SCL, TMDS-RX-SDA
- wire segments 74 -> 108
- no-connect marks 4 -> 8
Other:
- moved on the sheet: C?, J?, R?, U?

Commit message: Issue #336
Parts:
- added C? (x2): C, ~, symbol C
- added J? (x2): HDMI, ~, symbol HDMI
- added J? (x4): DVI, ~, symbol DVI
- added R? (x4): 1.5K, ~, symbol R
- added R? (x4): 47K, ~, symbol R
- added U? (x2): IP4776CZ38, symbol IP4776CZ38
Connections:
- net labels added: P3-CLK+, P3-CLK-, P3-D0+, P3-D0-, P3-D1+, P3-D1-, P3-D2+, P3-D2-, P4-CLK+, P4-CLK-, P4-D0+, P4-D0-, P4-D1+, P4-D1-, P4-D2+, P4-D2-, TMDS-RX2-0_N, TMDS-RX2-0_P, TMDS-RX2-1_N, TMDS-RX2-1_P, TMDS-RX2-2_N, TMDS-RX2-2_P, TMDS-RX2-CLK_N, TMDS-RX2-CLK_P, TMDS-TX2-0_N, TMDS-TX2-0_P, TMDS-TX2-1_N, TMDS-TX2-1_P, TMDS-TX2-2_N, TMDS-TX2-2_P, TMDS-TX2-CLK_N, TMDS-TX2-CLK_P
- wire segments 108 -> 282
- no-connect marks 8 -> 44
Other:
- note added: "DVI-P1"
- note added: "DVI-P2"
- note added: "DVI-P3"
- note added: "DVI-P4"
- note added: "HDMI P3"
- note added: "HDMI P4"

Commit message: Issue #336
Parts:
- removed R? (x6): 1.5K, ~, symbol R
- removed R? (x6): 47K, ~, symbol R
- added R? (x3): 100K, ~, symbol R
- added R? (x4): 15K, ~, symbol R
- added R? (x4): 27K, ~, symbol R
- added R? (x4): 47K, ~, symbol R
- added R? (x6): 1.5K, ~, symbol R
Connections:
- net labels added: P1-CEC, P1-HOT, P1-SCL, P1-SDA, P2-CEC, P2-HOT, P2-SCL, P2-SDA, P3-CEC, P3-HOT, P3-SCL, P3-SDA, P4-CEC, P4-HOT, P4-SCL, P4-SDA, TMDS-RX1-CEC, TMDS-RX1-HOT, TMDS-RX2-CEC, TMDS-RX2-HOT, TMDS-RX2-SCL, TMDS-RX2-SDA, TMDS-TX1-CEC, TMDS-TX1-HOT, TMDS-TX1-SCL, TMDS-TX1-SDA, TMDS-TX2-CEC, TMDS-TX2-HOT, TMDS-TX2-SCL, TMDS-TX2-SDA
- net labels removed: DDC-SCL, DDC-SDA
- wire segments 282 -> 344
- no-connect marks 44 -> 32
Other:
- moved on the sheet: R?
