File: board/hdmi.sch (KiCad schematic (older format))
At the start: 41 parts

Commit message: Issue #336
Parts:
- added R148: 100K, ~, symbol R
- added R149, R150: 47K, ~, symbol R
- added R158, R159, R160, R161, R162, R163, R164, R165, R166, R167, R168, R169, R170, R171, R172, R173: 50R, ~, symbol R
- gave numbers to parts that had none: 41
Connections:
- wire segments 344 -> 395
Other:
- moved on the sheet: C30, C31, C32, C33, J3, J4, J5, J9, R100, R101, R102, R103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

Commit message: Issue #336
Connections:
- wire segments 395 -> 393
- no-connect marks 32 -> 34
Changed lines of the file:
@@
 Sheet 5 7
 Title ""
-Date "16 jul 2013"
+Date "18 jul 2013"
 Rev ""
 Comp ""
@@
 Text HLabel 2250 3300 0    60   BiDi ~ 0
 TMDS-RX1-SDA
-Text Label 7000 3400 0    60   ~ 0
-VCC5V0
 $Comp
 L HDMI J4
@@
 TMDS-RX2-CLK_N
 NoConn ~ 14950 3050
-Text Label 14400 3450 0    60   ~ 0
-VCC5V0
 $Comp
 L DVI J6
@@
 	7450 1800 7450 3800
 Wire Wire Line
-	7550 3400 7000 3400
-Wire Wire Line
 	6750 5600 6850 5600
 Connection ~ 6750 5600
@@
 Wire Wire Line
 	14850 1850 14850 3850
-Wire Wire Line
-	14950 3450 14400 3450
 Wire Wire Line
 	8850 6800 9400 6800
@@
 	13400 900  13400 850
 Connection ~ 13400 850
+NoConn ~ 7550 3400
+NoConn ~ 14950 3450
 $EndSCHEMATC

Commit message: Issue #346
Parts:
- removed J10, J6, J7, J8: DVI, ~, symbol DVI
- added J6, J7: DVI-STACKED, ~, symbol DVI-STACKED
Changed lines of the file:
@@
 Sheet 5 7
 Title ""
-Date "18 jul 2013"
+Date "30 jul 2013"
 Rev ""
 Comp ""
@@
 TMDS-RX2-CLK_N
 NoConn ~ 14950 3050
-$Comp
-L DVI J6
-U 1 1 51DA7B40
-P 9700 7850
-F 0 "J6" H 9650 9200 60  0000 C CNN
-F 1 "DVI" H 9650 6500 60  0000 C CNN
-F 2 "~" H 9700 7850 60  0000 C CNN
-F 3 "~" H 9700 7850 60  0000 C CNN
-	1    9700 7850
-	1    0    0    -1
-$EndComp
 Text Label 8850 6800 0    60   ~ 0
 P1-D2+
@@
 NoConn ~ 9400 8600
 NoConn ~ 9400 8700
-$Comp
-L DVI J7
-U 1 1 51DA90B3
-P 11500 7850
-F 0 "J7" H 11450 9200 60  0000 C CNN
-F 1 "DVI" H 11450 6500 60  0000 C CNN
-F 2 "~" H 11500 7850 60  0000 C CNN
-F 3 "~" H 11500 7850 60  0000 C CNN
-	1    11500 7850
-	1    0    0    -1
-$EndComp
 Text Label 10650 6800 0    60   ~ 0
 P2-D2+
@@
 NoConn ~ 11200 8600
 NoConn ~ 11200 8700
-$Comp
-L DVI J8
-U 1 1 51DA90E0
-P 13300 7850
-F 0 "J8" H 13250 9200 60  0000 C CNN
-F 1 "DVI" H 13250 6500 60  0000 C CNN
-F 2 "~" H 13300 7850 60  0000 C CNN
-F 3 "~" H 13300 7850 60  0000 C CNN
-	1    13300 7850
-	1    0    0    -1
-$EndComp
 Text Label 12450 6800 0    60   ~ 0
 P3-D2+
@@
 NoConn ~ 13000 8600
 NoConn ~ 13000 8700
-$Comp
-L DVI J10
-U 1 1 51DA910D
-P 15050 7850
-F 0 "J10" H 15000 9200 60  0000 C CNN
-F 1 "DVI" H 15000 6500 60  0000 C CNN
-F 2 "~" H 15050 7850 60  0000 C CNN
-F 3 "~" H 15050 7850 60  0000 C CNN
-	1    15050 7850
-	1    0    0    -1
-$EndComp
 Text Label 14200 6800 0    60   ~ 0
 P2-D2+
@@
 NoConn ~ 7550 3400
 NoConn ~ 14950 3450
+$Comp
+L DVI-STACKED J6
+U 1 1 51F942F4
+P 9700 7850
+F 0 "J6" H 9650 9200 60  0000 C CNN
+F 1 "DVI-STACKED" H 9650 6500 60  0000 C CNN
+F 2 "~" H 9700 7850 60  0000 C CNN
+F 3 "~" H 9700 7850 60  0000 C CNN
+	1    9700 7850
+	1    0    0    -1
+$EndComp
+$Comp
+L DVI-STACKED J6
+U 2 1 51F94303
+P 13300 7850
+F 0 "J6" H 13250 9200 60  0000 C CNN
+F 1 "DVI-STACKED" H 13250 6500 60  0000 C CNN
+F 2 "~" H 13300 7850 60  0000 C CNN
+F 3 "~" H 13300 7850 60  0000 C CNN
+	2    13300 7850
+	1    0    0    -1
+$EndComp
+$Comp
+L DVI-STACKED J7
+U 1 1 51F94310
+P 11500 7850
+F 0 "J7" H 11450 9200 60  0000 C CNN
+F 1 "DVI-STACKED" H 11450 6500 60  0000 C CNN
+F 2 "~" H 11500 7850 60  0000 C CNN
+F 3 "~" H 11500 7850 60  0000 C CNN
+	1    11500 7850
+	1    0    0    -1
+$EndComp
+$Comp
+L DVI-STACKED J7
+U 2 1 51F94316
+P 15050 7850
+F 0 "J7" H 15000 9200 60  0000 C CNN
+F 1 "DVI-STACKED" H 15000 6500 60  0000 C CNN
+F 2 "~" H 15050 7850 60  0000 C CNN
+F 3 "~" H 15050 7850 60  0000 C CNN
+	2    15050 7850
+	1    0    0    -1
+$EndComp
 $EndSCHEMATC

Commit message: Issue #344
Parts:
- renumbered C30 to C31, C31 to C33, C33 to C34, J3 to J2, J4 to J3, J5 to J4, J6 to J5, J7 to J6, J9 to J7, R171 to R100, R172 to R101, R173 to R102, R116 to R103, R92 to R60, R158 to R61, R94 to R62, R159 to R63, R97 to R64, R160 to R65, R93 to R66, R161 to R67, R95 to R68, R96 to R69, R98 to R70, R99 to R71, R100 to R72, R101 to R73, R103 to R74, R102 to R75, R107 to R76, R105 to R77, R104 to R78, R106 to R79, R108 to R80, R110 to R81, R162 to R82, R109 to R83, R163 to R84, R111 to R85, R164 to R86, R112 to R87, R165 to R88, R166 to R89, R167 to R90, R168 to R91, R169 to R92, R148 to R93, R149 to R94, R150 to R95, R113 to R96, R114 to R97, R170 to R98, R115 to R99, U5 to U4, U6 to U5, U7 to U6, U8 to U7
Connections:
- no-connect marks 34 -> 38

Commit message: Issue #510
Parts:
- renumbered C31 to C44, C32 to C45, C33 to C46, C34 to C47, R103 to R100, R60 to R57, R61 to R58, R62 to R59, R63 to R60, R64 to R61, R65 to R62, R66 to R63, R67 to R64, R68 to R65, R69 to R66, R70 to R67, R71 to R68, R72 to R69, R73 to R70, R74 to R71, R75 to R72, R76 to R73, R77 to R74, R78 to R75, R79 to R76, R80 to R77, R81 to R78, R82 to R79, R83 to R80, R84 to R81, R85 to R82, R86 to R83, R87 to R84, R88 to R85, R89 to R86, R90 to R87, R91 to R88, R92 to R89, R93 to R90, R94 to R91, R95 to R92, R96 to R93, R97 to R94, R98 to R95, R99 to R96, R100 to R97, R101 to R98, R102 to R99, U6 to U10, U7 to U11, U4 to U8, U5 to U9
