File: board/hdmi.sch (KiCad schematic (older format))
At the start: 148 parts, among them J2 HDMI, J3 HDMI, J4 HDMI, J5 DVI-STACKED, J6 DVI-STACKED, J7 HDMI, U10 IP4776CZ38, U11 IP4776CZ38, U8 IP4776CZ38, U9 IP4776CZ38

Commit message: Issue #1027 - Schematics final changes.
Parts:
- added C205, C206, C208, C210: 0.1mfd, ~, symbol C
- added C207, C209: 0.33mfd, ~, symbol C
- added R342, R343: 1K, ~, symbol R
- added R348, R349: 100K, ~, symbol R
- added U22, U23: ΜA78L00, symbol ΜA78L00
- R337, R338: value 10K -> 100R
Connections:
- net labels added: HDMI-TX1-VCC5V0, HDMI-TX2-VCC5V0
- wire segments 395 -> 424

Commit message: Issue #1027 - Schematics final changes.
Parts:
- added R361, R362: 10K, ~, symbol R
- R337, R338: value 100R -> 10K
Connections:
- wire segments 424 -> 426
Changed lines of the file:
@@
 Sheet 3 8
 Title "HDMI2USB"
-Date "15 apr 2014"
+Date "16 apr 2014"
 Rev ""
 Comp ""
@@
 Text Label 8750 8100 0    60   ~ 0
 P1-CLK-
-Text Label 8800 7100 0    60   ~ 0
-VCC5V0
 NoConn ~ 9800 6100
 NoConn ~ 9800 6200
@@
 Text Label 10400 8100 0    60   ~ 0
 P3-CLK-
-Text Label 10400 7100 0    60   ~ 0
-VCC5V0
 NoConn ~ 11450 6500
 NoConn ~ 11450 6900
@@
 P 14700 3500
 F 0 "R338" V 14750 3700 40  0000 C CNN
-F 1 "100R" V 14707 3501 40  0000 C CNN
+F 1 "10K" V 14707 3501 40  0000 C CNN
 F 2 "~" V 14630 3500 30  0000 C CNN
 F 3 "~" H 14700 3500 30  0000 C CNN
@@
 	0    -1   -1   0
 $EndComp
-$Comp
-L R R337
-U 1 1 5343B29C
-P 7150 3550
-F 0 "R337" V 7200 3750 40  0000 C CNN
-F 1 "100R" V 7157 3551 40  0000 C CNN
-F 2 "~" V 7080 3550 30  0000 C CNN
-F 3 "~" H 7150 3550 30  0000 C CNN
-	1    7150 3550
-	0    -1   -1   0
-$EndComp
 Text Label 8700 9550 0    39   ~ 0
 VCC5V0
@@
 	11450 6800 11350 6800
 Wire Wire Line
-	10400 7100 11450 7100
-Wire Wire Line
 	10950 7400 10400 7400
 Wire Wire Line
@@
 	14250 7050 15250 7050
 Wire Wire Line
-	8800 7100 9800 7100
-Wire Wire Line
 	6100 6800 7150 6800
 Wire Wire Line
@@
 	2550 1700 2250 1700
 Wire Wire Line
-	6250 3550 6900 3550
-Wire Wire Line
-	13800 3500 14450 3500
-Wire Wire Line
 	6850 3700 6850 3650
 Connection ~ 6850 3650
@@
 Wire Notes Line
 	10900 10500 10950 10500
-Text Label 6250 3550 0    39   ~ 0
-VCC5V0
-Text Label 13800 3500 0    39   ~ 0
-VCC5V0
 Text Label 6100 6800 0    39   ~ 0
 HDMI-TX1-VCC5V0
@@
 	500  500  15850 500
 Wire Notes Line
-	8250 500  8250 4500
-Wire Notes Line
 	500  4500 15850 4500
 Wire Notes Line
@@
 Wire Notes Line
 	900  4800 550  4800
+$Comp
+L R R337
+U 1 1 5343B29C
+P 7150 3550
+F 0 "R337" V 7200 3750 40  0000 C CNN
+F 1 "10K" V 7157 3551 40  0000 C CNN
+F 2 "~" V 7080 3550 30  0000 C CNN
+F 3 "~" H 7150 3550 30  0000 C CNN
+	1    7150 3550
+	0    -1   -1   0
+$EndComp
+Wire Wire Line
+	6900 3550 6350 3550
+Text Label 6350 3550 0    60   ~ 0
+GND
+Wire Wire Line
+	14450 3500 13900 3500
+Text Label 13900 3500 0    60   ~ 0
+GND
+$Comp
+L R R361
+U 1 1 534EA525
+P 9400 7100
+F 0 "R361" V 9450 7300 40  0000 C CNN
+F 1 "10K" V 9407 7101 40  0000 C CNN
+F 2 "~" V 9330 7100 30  0000 C CNN
+F 3 "~" H 9400 7100 30  0000 C CNN
+	1    9400 7100
+	0    -1   -1   0
+$EndComp
+Wire Wire Line
+	9650 7100 9800 7100
+Wire Wire Line
+	9150 7100 8750 7100
+$Comp
+L R R362
+U 1 1 534EAC48
+P 10950 7100
+F 0 "R362" V 11000 7300 40  0000 C CNN
+F 1 "10K" V 10957 7101 40  0000 C CNN
+F 2 "~" V 10880 7100 30  0000 C CNN
+F 3 "~" H 10950 7100 30  0000 C CNN
+	1    10950 7100
+	0    -1   -1   0
+$EndComp
+Wire Wire Line
+	11450 7100 11200 7100
+Wire Wire Line
+	10700 7100 10400 7100
+Text Label 8750 7100 0    60   ~ 0
+GND
+Text Label 10400 7100 0    60   ~ 0
+GND
 $EndSCHEMATC

Commit message: Issue #1027 - Schematics final changes.
Other:
- note added: "DVI IN 1"
- note added: "DVI IN 2"
- note added: "DVI OUT 1"
- note added: "DVI OUT 2"
- note added: "HDMI IN 1"
- note added: "HDMI IN 2"
- note added: "HDMI OUT 1"
- note added: "HDMI OUT 2"
- note added: "LDO OUT FOR"
- note added: "LDO OUT FOR TX1"
- note added: "LDO OUT FOR TX2"
- note removed: "DVI IN"
- note removed: "DVI OUT"
- note removed: "HDMI IN"
- note removed: "HDMI OUT"
- moved on the sheet: R199, R200, R201, R202, R203, R204, R205, R206, R207, R208, R209, R361

Commit message: Issue #1027 - Schematics final changes.
Changed lines of the file:
@@
 Sheet 3 8
 Title "HDMI2USB"
-Date "16 apr 2014"
+Date "17 apr 2014"
 Rev ""
 Comp ""
@@
 Text Label 14200 8050 0    60   ~ 0
 P2-CLK-
-Text Label 14250 7050 0    60   ~ 0
-VCC5V0
 NoConn ~ 15250 6050
 NoConn ~ 15250 6150
@@
 Text Label 12400 8050 0    60   ~ 0
 P4-CLK-
-Text Label 12400 7050 0    60   ~ 0
-VCC5V0
 NoConn ~ 13450 6050
 NoConn ~ 13450 6150
@@
 Text Notes 9150 9100 0    39   ~ 0
 HDMI OUT 1
+Text Label 12400 7050 0    39   ~ 0
+HDMI-TX2-VCC5V0
+Text Label 14250 7050 0    39   ~ 0
+HDMI-TX1-VCC5V0
 $EndSCHEMATC
