File: board/expansion connectors.sch (KiCad schematic (older format))
At the start: 44 parts, among them J2 VHDCI

Commit message: Issue #336
Parts:
- added R155, R156, R157: R, ~, symbol R
- gave numbers to parts that had none: 3
Connections:
- net labels added: TCK, TDO-FPGA/TDO-JTAG, TDO-USB/TDI-FPGA, TMS
- wire segments 163 -> 170
Changed lines of the file:
@@
 Sheet 6 7
 Title ""
-Date "13 jul 2013"
+Date "16 jul 2013"
 Rev ""
 Comp ""
@@
 Connection ~ 2250 2850
 $Comp
-L CONN_7X2 P?
+L CONN_7X2 P1
 U 1 1 51D7E6A3
 P 7800 1550
-F 0 "P?" H 7800 1950 60  0000 C CNN
+F 0 "P1" H 7800 1950 60  0000 C CNN
 F 1 "CONN_7X2" V 7800 1550 60  0000 C CNN
 F 2 "" H 7800 1550 60  0000 C CNN
@@
 VCC3V3
 $Comp
-L DVI J?
+L DVI J11
 U 1 1 520EC9D4
 P 7800 4150
-F 0 "J?" H 7750 5500 60  0000 C CNN
+F 0 "J11" H 7750 5500 60  0000 C CNN
 F 1 "DVI" H 7750 2800 60  0000 C CNN
 F 2 "~" H 7800 4150 60  0000 C CNN
@@
 $EndComp
 $Comp
-L DVI J?
+L DVI J12
 U 1 1 520EE54D
 P 8400 4150
-F 0 "J?" H 8350 5500 60  0000 C CNN
+F 0 "J12" H 8350 5500 60  0000 C CNN
 F 1 "DVI" H 8350 2800 60  0000 C CNN
 F 2 "~" H 8400 4150 60  0000 C CNN
@@
 Wire Wire Line
 	8700 4300 9350 4300
+$Comp
+L R R155
+U 1 1 51E938A6
+P 8800 1350
+F 0 "R155" V 8850 1150 40  0000 C CNN
+F 1 "R" V 8807 1351 40  0000 C CNN
+F 2 "~" V 8730 1350 30  0000 C CNN
+F 3 "~" H 8800 1350 30  0000 C CNN
+	1    8800 1350
+	0    -1   -1   0
+$EndComp
+Wire Wire Line
+	8200 1350 8550 1350
+Text GLabel 4950 2650 2    60   Input ~ 0
+VCC3V3
+$Comp
+L R R156
+U 1 1 51E93CA0
+P 8800 1450
+F 0 "R156" V 8850 1250 40  0000 C CNN
+F 1 "R" V 8807 1451 40  0000 C CNN
+F 2 "~" V 8730 1450 30  0000 C CNN
+F 3 "~" H 8800 1450 30  0000 C CNN
+	1    8800 1450
+	0    -1   -1   0
+$EndComp
+Wire Wire Line
+	8550 1450 8200 1450
+$Comp
+L R R157
+U 1 1 51E93D6E
+P 8800 1550
+F 0 "R157" V 8850 1350 40  0000 C CNN
+F 1 "R" V 8807 1551 40  0000 C CNN
+F 2 "~" V 8730 1550 30  0000 C CNN
+F 3 "~" H 8800 1550 30  0000 C CNN
+	1    8800 1550
+	0    -1   -1   0
+$EndComp
+Wire Wire Line
+	8200 1550 8550 1550
+Wire Wire Line
+	9050 1350 9150 1350
+Wire Wire Line
+	9050 1450 9150 1450
+Wire Wire Line
+	9050 1550 9150 1550
+Wire Wire Line
+	8200 1650 9150 1650
+Text HLabel 9150 1350 2    60   BiDi ~ 0
+TMS
+Text HLabel 9150 1450 2    60   BiDi ~ 0
+TCK
+Text HLabel 9150 1550 2    60   BiDi ~ 0
+TDO-FPGA/TDO-JTAG
+Text HLabel 9150 1650 2    60   BiDi ~ 0
+TDO-USB/TDI-FPGA
 $EndSCHEMATC

Commit message: Issue #336
Connections:
- wire segments 170 -> 169
- no-connect marks 6 -> 7
Changed lines of the file:
@@
 Sheet 6 7
 Title ""
-Date "16 jul 2013"
+Date "18 jul 2013"
 Rev ""
 Comp ""
@@
 NoConn ~ 7500 4900
 NoConn ~ 7500 5000
-Wire Wire Line
-	7500 4300 6850 4300
-Text Label 6850 4300 0    60   ~ 0
-VCC5V0
-Text GLabel 6850 4300 0    60   Input ~ 0
+Text GLabel 9350 4300 2    60   Input ~ 0
 VCC5V0
 Text Label 4950 2850 2    60   ~ 0
@@
 Text HLabel 9150 1650 2    60   BiDi ~ 0
 TDO-USB/TDI-FPGA
+NoConn ~ 7500 4300
 $EndSCHEMATC

Commit message: Issue #346
Parts:
- removed J11, J12: DVI, ~, symbol DVI
- added J8: DVI-STACKED, ~, symbol DVI-STACKED
Changed lines of the file:
@@
 Sheet 6 7
 Title ""
-Date "18 jul 2013"
+Date "30 jul 2013"
 Rev ""
 Comp ""
@@
 Text Label 8550 1250 2    60   ~ 0
 VCC3V3
-$Comp
-L DVI J11
-U 1 1 520EC9D4
-P 7800 4150
-F 0 "J11" H 7750 5500 60  0000 C CNN
-F 1 "DVI" H 7750 2800 60  0000 C CNN
-F 2 "~" H 7800 4150 60  0000 C CNN
-F 3 "~" H 7800 4150 60  0000 C CNN
-	1    7800 4150
-	1    0    0    -1
-$EndComp
-$Comp
-L DVI J12
-U 1 1 520EE54D
-P 8400 4150
-F 0 "J12" H 8350 5500 60  0000 C CNN
-F 1 "DVI" H 8350 2800 60  0000 C CNN
-F 2 "~" H 8400 4150 60  0000 C CNN
-F 3 "~" H 8400 4150 60  0000 C CNN
-	1    8400 4150
-	-1   0    0    -1
-$EndComp
 Text Notes 3550 850  2    60   ~ 0
 VHDCI EXPANSION
@@
 TDO-USB/TDI-FPGA
 NoConn ~ 7500 4300
+$Comp
+L DVI-STACKED J8
+U 1 1 51F96016
+P 7800 4150
+F 0 "J8" H 7750 5500 60  0000 C CNN
+F 1 "DVI-STACKED" H 7750 2800 60  0000 C CNN
+F 2 "~" H 7800 4150 60  0000 C CNN
+F 3 "~" H 7800 4150 60  0000 C CNN
+	1    7800 4150
+	1    0    0    -1
+$EndComp
+$Comp
+L DVI-STACKED J8
+U 2 1 51F96025
+P 8400 4150
+F 0 "J8" H 8350 5500 60  0000 C CNN
+F 1 "DVI-STACKED" H 8350 2800 60  0000 C CNN
+F 2 "~" H 8400 4150 60  0000 C CNN
+F 3 "~" H 8400 4150 60  0000 C CNN
+	2    8400 4150
+	-1   0    0    -1
+$EndComp
 $EndSCHEMATC

Commit message: Issue #344
Parts:
- renumbered J2 to J8, J8 to J9, R32 to R104, R33 to R105, R34 to R106, R35 to R107, R36 to R108, R37 to R109, R38 to R110, R39 to R111, R40 to R112, R41 to R113, R42 to R114, R43 to R115, R44 to R116, R45 to R117, R46 to R118, R47 to R119, R48 to R120, R49 to R121, R50 to R122, R51 to R123, R52 to R124, R53 to R125, R54 to R126, R55 to R127, R56 to R128, R57 to R129, R58 to R130, R59 to R131, R60 to R132, R61 to R133, R62 to R134, R63 to R135, R64 to R136, R65 to R137, R66 to R138, R67 to R139, R68 to R140, R69 to R141, R70 to R142, R71 to R143, R155 to R144, R156 to R145, R157 to R146

Commit message: Issue #510
Parts:
- renumbered R104 to R101, R105 to R102, R106 to R103, R107 to R104, R108 to R105, R109 to R106, R110 to R107, R111 to R108, R112 to R109, R113 to R110, R114 to R111, R115 to R112, R116 to R113, R117 to R114, R118 to R115, R119 to R116, R120 to R117, R121 to R118, R122 to R119, R123 to R120, R124 to R121, R125 to R122, R126 to R123, R127 to R124, R128 to R125, R129 to R126, R130 to R127, R131 to R128, R132 to R129, R133 to R130, R134 to R131, R135 to R132, R136 to R133, R137 to R134, R138 to R135, R139 to R136, R140 to R137, R141 to R138, R142 to R139, R143 to R140, R144 to R141, R145 to R142, R146 to R143
Changed lines of the file:
@@
 Sheet 6 7
 Title ""
-Date "11 aug 2013"
+Date "3 sep 2013"
 Rev ""
 Comp ""
@@
 	2500 1150 2250 1150
 $Comp
-L R R104
+L R R101
 U 1 1 51CD40FC
 P 2000 1150
-F 0 "R104" V 2050 950 40  0000 C CNN
+F 0 "R101" V 2050 950 40  0000 C CNN
 F 1 "R" V 2007 1151 40  0000 C CNN
 F 2 "~" V 1930 1150 30  0000 C CNN
@@
 $EndComp
 $Comp
-L R R105
+L R R102
 U 1 1 51CD4109
 P 2000 1350
-F 0 "R105" V 2050 1150 40  0000 C CNN
+F 0 "R102" V 2050 1150 40  0000 C CNN
 F 1 "R" V 2007 1351 40  0000 C CNN
 F 2 "~" V 1930 1350 30  0000 C CNN
@@
 	4050 1350 3800 1350
 $Comp
-L R R106
+L R R103
 U 1 1 51CD416D
 P 2000 1450
-F 0 "R106" V 1950 1650 40  0000 C CNN
+F 0 "R103" V 1950 1650 40  0000 C CNN
 F 1 "R" V 2007 1451 40  0000 C CNN
 F 2 "~" V 1930 1450 30  0000 C CNN
@@
 $EndComp
 $Comp
-L R R107
+L R R104
 U 1 1 51CD41F5
 P 2000 1650
-F 0 "R107" V 1950 1850 40  0000 C CNN
+F 0 "R104" V 1950 1850 40  0000 C CNN
 F 1 "R" V 2007 1651 40  0000 C CNN
 F 2 "~" V 1930 1650 30  0000 C CNN
@@
 $EndComp
 $Comp
-L R R108
+L R R105
 U 1 1 51CD41FB
 P 2000 1750
-F 0 "R108" V 1950 1950 40  0000 C CNN
+F 0 "R105" V 1950 1950 40  0000 C CNN
 F 1 "R" V 2007 1751 40  0000 C CNN
 F 2 "~" V 1930 1750 30  0000 C CNN
@@
 $EndComp
 $Comp
-L R R109
+L R R106
 U 1 1 51CD4224
 P 2000 1950
-F 0 "R109" V 2050 1750 40  0000 C CNN
+F 0 "R106" V 2050 1750 40  0000 C CNN
 F 1 "R" V 2007 1951 40  0000 C CNN
 F 2 "~" V 1930 1950 30  0000 C CNN
@@
 $EndComp
 $Comp
-L R R110
+L R R107
 U 1 1 51CD422A
 P 2000 2050
-F 0 "R110" V 1950 2250 40  0000 C CNN
+F 0 "R107" V 1950 2250 40  0000 C CNN
 F 1 "R" V 2007 2051 40  0000 C CNN
 F 2 "~" V 1930 2050 30  0000 C CNN
@@
 $EndComp
 $Comp
-L R R111
+L R R108
 U 1 1 51CD4230
 P 2000 2250
-F 0 "R111" V 1950 2450 40  0000 C CNN
+F 0 "R108" V 1950 2450 40  0000 C CNN
 F 1 "R" V 2007 2251 40  0000 C CNN
 F 2 "~" V 1930 2250 30  0000 C CNN
@@
 $EndComp
 $Comp
-L R R112
+L R R109
 U 1 1 51CD4236
 P 2000 2350
-F 0 "R112" V 1950 2550 40  0000 C CNN
+F 0 "R109" V 1950 2550 40  0000 C CNN
 F 1 "R" V 2007 2351 40  0000 C CNN
 F 2 "~" V 1930 2350 30  0000 C CNN
@@
 $EndComp
 $Comp
-L R R115
+L R R112
 U 1 1 51CD423C
 P 2000 3250
-F 0 "R115" V 2050 3050 40  0000 C CNN
+F 0 "R112" V 2050 3050 40  0000 C CNN
 F 1 "R" V 2007 3251 40  0000 C CNN
 F 2 "~" V 1930 3250 30  0000 C CNN
@@
 $EndComp
 $Comp
-L R R116
+L R R113
 U 1 1 51CD4242
 P 2000 3350
-F 0 "R116" V 1950 3550 40  0000 C CNN
+F 0 "R113" V 1950 3550 40  0000 C CNN
 F 1 "R" V 2007 3351 40  0000 C CNN
 F 2 "~" V 1930 3350 30  0000 C CNN
@@
 $EndComp
 $Comp
-L R R117
+L R R114
 U 1 1 51CD4248
 P 2000 3550
-F 0 "R117" V 1950 3750 40  0000 C CNN
+F 0 "R114" V 1950 3750 40  0000 C CNN
 F 1 "R" V 2007 3551 40  0000 C CNN
 F 2 "~" V 1930 3550 30  0000 C CNN
@@
 $EndComp
 $Comp
-L R R118
+L R R115
 U 1 1 51CD424E
 P 2000 3650
-F 0 "R118" V 1950 3850 40  0000 C CNN
+F 0 "R115" V 1950 3850 40  0000 C CNN
 F 1 "R" V 2007 3651 40  0000 C CNN
 F 2 "~" V 1930 3650 30  0000 C CNN
@@
 $EndComp
 $Comp
-L R R119
+L R R116
 U 1 1 51CD4254
 P 2000 3850
-F 0 "R119" V 2050 3650 40  0000 C CNN
+F 0 "R116" V 2050 3650 40  0000 C CNN
 F 1 "R" V 2007 3851 40  0000 C CNN
 F 2 "~" V 1930 3850 30  0000 C CNN
@@
 $EndComp
 $Comp
-L R R120
+L R R117
 U 1 1 51CD425A
 P 2000 3950
-F 0 "R120" V 1950 4150 40  0000 C CNN
+F 0 "R117" V 1950 4150 40  0000 C CNN
 F 1 "R" V 2007 3951 40  0000 C CNN
 F 2 "~" V 1930 3950 30  0000 C CNN
@@
 $EndComp
 $Comp
-L R R121
+L R R118
 U 1 1 51CD4260
 P 2000 4150
-F 0 "R121" V 1950 4350 40  0000 C CNN
+F 0 "R118" V 1950 4350 40  0000 C CNN
 F 1 "R" V 2007 4151 40  0000 C CNN
 F 2 "~" V 1930 4150 30  0000 C CNN
@@
 $EndComp
 $Comp
-L R R122
+L R R119
 U 1 1 51CD4266
 P 2000 4250
-F 0 "R122" V 1950 4450 40  0000 C CNN
+F 0 "R119" V 1950 4450 40  0000 C CNN
 F 1 "R" V 2007 4251 40  0000 C CNN
 F 2 "~" V 1930 4250 30  0000 C CNN
@@
 $EndComp
 $Comp
-L R R123
+L R R120
 U 1 1 51CD426C
 P 2000 4450
-F 0 "R123" V 1950 4650 40  0000 C CNN
+F 0 "R120" V 1950 4650 40  0000 C CNN
 F 1 "R" V 2007 4451 40  0000 C CNN
 F 2 "~" V 1930 4450 30  0000 C CNN
@@
 $EndComp
 $Comp
-L R R113
+L R R110
 U 1 1 51CD4272
 P 2000 2550
-F 0 "R113" V 1950 2750 40  0000 C CNN
+F 0 "R110" V 1950 2750 40  0000 C CNN
 F 1 "R" V 2007 2551 40  0000 C CNN
 F 2 "~" V 1930 2550 30  0000 C CNN
@@
 $EndComp
 $Comp
-L R R114
+L R R111
 U 1 1 51CD4278
 P 2000 3050
-F 0 "R114" V 1950 3250 40  0000 C CNN
+F 0 "R111" V 1950 3250 40  0000 C CNN
 F 1 "R" V 2007 3051 40  0000 C CNN
 F 2 "~" V 1930 3050 30  0000 C CNN
@@
 $EndComp
 $Comp
-L R R124
+L R R121
 U 1 1 51CD427E
 P 4300 1150
-F 0 "R124" V 4350 950 40  0000 C CNN
+F 0 "R121" V 4350 950 40  0000 C CNN
 F 1 "R" V 4307 1151 40  0000 C CNN
 F 2 "~" V 4230 1150 30  0000 C CNN
@@
 $EndComp
 $Comp
-L R R125
+L R R122
 U 1 1 51CD4284
 P 4300 1350
-F 0 "R125" V 4350 1150 40  0000 C CNN
+F 0 "R122" V 4350 1150 40  0000 C CNN
 F 1 "R" V 4307 1351 40  0000 C CNN
 F 2 "~" V 4230 1350 30  0000 C CNN
@@
 $EndComp
 $Comp
-L R R126
+L R R123
 U 1 1 51CD428A
 P 4300 1450
-F 0 "R126" V 4250 1650 40  0000 C CNN
+F 0 "R123" V 4250 1650 40  0000 C CNN
 F 1 "R" V 4307 1451 40  0000 C CNN
 F 2 "~" V 4230 1450 30  0000 C CNN
@@
 $EndComp
 $Comp
-L R R127
+L R R124
 U 1 1 51CD4290
 P 4300 1650
-F 0 "R127" V 4250 1850 40  0000 C CNN
+F 0 "R124" V 4250 1850 40  0000 C CNN
 F 1 "R" V 4307 1651 40  0000 C CNN
 F 2 "~" V 4230 1650 30  0000 C CNN
@@
 $EndComp
 $Comp
-L R R128
+L R R125
 U 1 1 51CD4296
 P 4300 1750
-F 0 "R128" V 4250 1950 40  0000 C CNN
+F 0 "R125" V 4250 1950 40  0000 C CNN
 F 1 "R" V 4307 1751 40  0000 C CNN
 F 2 "~" V 4230 1750 30  0000 C CNN
@@
 $EndComp
 $Comp
-L R R129
+L R R126
 U 1 1 51CD429C
 P 4300 1950
-F 0 "R129" V 4350 1750 40  0000 C CNN
+F 0 "R126" V 4350 1750 40  0000 C CNN
 F 1 "R" V 4307 1951 40  0000 C CNN
 F 2 "~" V 4230 1950 30  0000 C CNN
@@
 $EndComp
 $Comp
-L R R130
+L R R127
 U 1 1 51CD42A2
 P 4300 2050
-F 0 "R130" V 4250 2250 40  0000 C CNN
+F 0 "R127" V 4250 2250 40  0000 C CNN
 F 1 "R" V 4307 2051 40  0000 C CNN
 F 2 "~" V 4230 2050 30  0000 C CNN
@@
 $EndComp
 $Comp
-L R R131
+L R R128
 U 1 1 51CD42A8
 P 4300 2250
-F 0 "R131" V 4250 2450 40  0000 C CNN
+F 0 "R128" V 4250 2450 40  0000 C CNN
 F 1 "R" V 4307 2251 40  0000 C CNN
 F 2 "~" V 4230 2250 30  0000 C CNN
@@
 $EndComp
 $Comp
-L R R132
+L R R129
 U 1 1 51CD42AE
 P 4300 2350
-F 0 "R132" V 4250 2550 40  0000 C CNN
+F 0 "R129" V 4250 2550 40  0000 C CNN
 F 1 "R" V 4307 2351 40  0000 C CNN
 F 2 "~" V 4230 2350 30  0000 C CNN
@@
 $EndComp
 $Comp
-L R R135
+L R R132
 U 1 1 51CD42B4
 P 4300 3250
-F 0 "R135" V 4350 3050 40  0000 C CNN
+F 0 "R132" V 4350 3050 40  0000 C CNN
 F 1 "R" V 4307 3251 40  0000 C CNN
 F 2 "~" V 4230 3250 30  0000 C CNN
@@
 $EndComp
 $Comp
-L R R136
+L R R133
 U 1 1 51CD42BA
 P 4300 3350
-F 0 "R136" V 4250 3550 40  0000 C CNN
+F 0 "R133" V 4250 3550 40  0000 C CNN
 F 1 "R" V 4307 3351 40  0000 C CNN
 F 2 "~" V 4230 3350 30  0000 C CNN
@@
 $EndComp
 $Comp
-L R R137
+L R R134
 U 1 1 51CD42C0
 P 4300 3550
-F 0 "R137" V 4250 3750 40  0000 C CNN
+F 0 "R134" V 4250 3750 40  0000 C CNN
 F 1 "R" V 4307 3551 40  0000 C CNN
 F 2 "~" V 4230 3550 30  0000 C CNN
@@
 $EndComp
 $Comp
-L R R138
+L R R135
 U 1 1 51CD42C6
 P 4300 3650
-F 0 "R138" V 4250 3850 40  0000 C CNN
+F 0 "R135" V 4250 3850 40  0000 C CNN
 F 1 "R" V 4307 3651 40  0000 C CNN
 F 2 "~" V 4230 3650 30  0000 C CNN
@@
 $EndComp
 $Comp
-L R R139
+L R R136
 U 1 1 51CD42CC
 P 4300 3850
-F 0 "R139" V 4350 3650 40  0000 C CNN
+F 0 "R136" V 4350 3650 40  0000 C CNN
 F 1 "R" V 4307 3851 40  0000 C CNN
 F 2 "~" V 4230 3850 30  0000 C CNN
@@
 $EndComp
 $Comp
-L R R140
+L R R137
 U 1 1 51CD42D2
 P 4300 3950
-F 0 "R140" V 4250 4150 40  0000 C CNN
+F 0 "R137" V 4250 4150 40  0000 C CNN
 F 1 "R" V 4307 3951 40  0000 C CNN
 F 2 "~" V 4230 3950 30  0000 C CNN
@@
 $EndComp
 $Comp
-L R R141
+L R R138
 U 1 1 51CD42D8
 P 4300 4150
-F 0 "R141" V 4250 4350 40  0000 C CNN
+F 0 "R138" V 4250 4350 40  0000 C CNN
 F 1 "R" V 4307 4151 40  0000 C CNN
 F 2 "~" V 4230 4150 30  0000 C CNN
@@
 $EndComp
 $Comp
-L R R142
+L R R139
 U 1 1 51CD42DE
 P 4300 4250
-F 0 "R142" V 4250 4450 40  0000 C CNN
+F 0 "R139" V 4250 4450 40  0000 C CNN
 F 1 "R" V 4307 4251 40  0000 C CNN
 F 2 "~" V 4230 4250 30  0000 C CNN
@@
 $EndComp
 $Comp
-L R R143
+L R R140
 U 1 1 51CD42E4
 P 4300 4450
-F 0 "R143" V 4250 4650 40  0000 C CNN
+F 0 "R140" V 4250 4650 40  0000 C CNN
 F 1 "R" V 4307 4451 40  0000 C CNN
 F 2 "~" V 4230 4450 30  0000 C CNN
@@
 $EndComp
 $Comp
-L R R133
+L R R130
 U 1 1 51CD42EA
 P 4300 2550
-F 0 "R133" V 4250 2750 40  0000 C CNN
+F 0 "R130" V 4250 2750 40  0000 C CNN
 F 1 "R" V 4307 2551 40  0000 C CNN
 F 2 "~" V 4230 2550 30  0000 C CNN
@@
 $EndComp
 $Comp
-L R R134
+L R R131
 U 1 1 51CD42F0
 P 4300 3050
-F 0 "R134" V 4250 3250 40  0000 C CNN
+F 0 "R131" V 4250 3250 40  0000 C CNN
 F 1 "R" V 4307 3051 40  0000 C CNN
 F 2 "~" V 4230 3050 30  0000 C CNN
@@
 	8700 4300 9350 4300
 $Comp
-L R R144
+L R R141
 U 1 1 51E938A6
 P 8800 1350
-F 0 "R144" V 8850 1150 40  0000 C CNN
+F 0 "R141" V 8850 1150 40  0000 C CNN
 F 1 "R" V 8807 1351 40  0000 C CNN
 F 2 "~" V 8730 1350 30  0000 C CNN
@@
 VCC3V3
 $Comp
-L R R145
+L R R142
 U 1 1 51E93CA0
 P 8800 1450
-F 0 "R145" V 8850 1250 40  0000 C CNN
+F 0 "R142" V 8850 1250 40  0000 C CNN
 F 1 "R" V 8807 1451 40  0000 C CNN
 F 2 "~" V 8730 1450 30  0000 C CNN
@@
 	8550 1450 8200 1450
 $Comp
-L R R146
+L R R143
 U 1 1 51E93D6E
 P 8800 1550
-F 0 "R146" V 8850 1350 40  0000 C CNN
+F 0 "R143" V 8850 1350 40  0000 C CNN
 F 1 "R" V 8807 1551 40  0000 C CNN
 F 2 "~" V 8730 1550 30  0000 C CNN
