File: board/expansion connectors.sch (KiCad schematic (older format))
At the start: 16 parts, among them J8 VHDCI, J9 DVI-STACKED, P1 CONN_7X2

Commit message: Issue #1022 - Schematics final.
Parts:
- added Q1: NPN, ~, symbol NPN
- added R290, R293, R294, R295, R304: 2.2K, ~, symbol R
- added R291, R296, R298, R318, R323: 5.6K, ~, symbol R
- added R292, R297, R299, R319, R324: 10K, ~, symbol R
- added R300, R301, R302, R303, R305, R306, R315, R316, R317, R320, R321, R322: 50R, ~, symbol R
- R141, R142, R143: value R -> 100R
Connections:
- wire segments 129 -> 175
Other:
- moved on the sheet: J8, P1, R101, R102, R103, R104, R105, R106, R107, R108, R109, R110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

Commit message: Issue #993
Connections:
- wire segments 175 -> 216
Other:
- note added: "GTP RX DDC LEVEL SHIFTER"
- note added: "GTP RX EXPANSION"
- note added: "GTP TX DDC LEVEL SHIFTER"
- note added: "GTP TX EXPANSION"
- note added: "JTAG CONNECTOR"
- moved on the sheet: J8, P1, Q1, R101, R102, R103, R104, R105, R106, R107, R108, R109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

Commit message: Issue #1022 - Schematics final changes.
Parts:
- added R335: 10K, ~, symbol R
- added R336: 4.7K, ~, symbol R
Connections:
- wire segments 216 -> 219
- no-connect marks 7 -> 6
Changed lines of the file:
@@
 Sheet 4 8
 Title "HDMI2USB"
-Date "3 apr 2014"
+Date "7 apr 2014"
 Rev ""
 Comp ""
@@
 NoConn ~ 10250 5600
 NoConn ~ 10250 5700
-Text GLabel 12100 5000 2    60   Input ~ 0
+Text GLabel 12800 5000 2    60   Input ~ 0
 VCC5V0
 Text Label 5300 3550 2    39   ~ 0
@@
 Text Label 5300 3350 2    39   ~ 0
 VCC3V3
-Text Label 12100 5000 2    39   ~ 0
+Text Label 12800 5000 2    39   ~ 0
 VCC5V0
 $Comp
@@
 Text HLabel 10200 1850 2    60   BiDi ~ 0
 TDO-USB/TDI-FPGA
-NoConn ~ 10250 5000
 $Comp
 L DVI-STACKED J9
@@
 Wire Wire Line
 	8750 9100 8950 9100
+$Comp
+L R R335
+U 1 1 53435E5A
+P 9150 5000
+F 0 "R335" V 9200 4800 40  0000 C CNN
+F 1 "10K" V 9157 5001 40  0000 C CNN
+F 2 "~" V 9080 5000 30  0000 C CNN
+F 3 "~" H 9150 5000 30  0000 C CNN
+	1    9150 5000
+	0    -1   -1   0
+$EndComp
+Wire Wire Line
+	9400 5000 10250 5000
+Wire Wire Line
+	8650 5000 8900 5000
+Text Label 8650 5000 0    39   ~ 0
+GND
+$Comp
+L R R336
+U 1 1 534377F2
+P 12350 5000
+F 0 "R336" V 12400 4800 40  0000 C CNN
+F 1 "4.7K" V 12357 5001 40  0000 C CNN
+F 2 "~" V 12280 5000 30  0000 C CNN
+F 3 "~" H 12350 5000 30  0000 C CNN
+	1    12350 5000
+	0    -1   -1   0
+$EndComp
+Wire Wire Line
+	12800 5000 12600 5000
 $EndSCHEMATC
