File: board/expansion connectors.sch (KiCad schematic (older format))
At the start: 46 parts, among them J8 VHDCI, J9 DVI-STACKED, P1 CONN_7X2, Q1 NPN

Commit message: Issue #1027 - Schematics final changes.
Parts:
- added C211: 0.33mfd, ~, symbol C
- added C212: 0.1mfd, ~, symbol C
- added R350, R351, R352, R353, R354, R355, R356, R357, R358: 100R, ~, symbol R
- added R359: 100K, ~, symbol R
- added U24: ΜA78L00, symbol ΜA78L00
- R336: value 4.7K -> 1K
Connections:
- net labels added: GTP-TX-VCC5V0
- wire segments 219 -> 235
Other:
- note added: "=3.2V"
- note added: "SCL,SDA VOLTAGE CALCULATION"
- note added: "SCL/SDA = (10K(10+5.6)K)*5"

Commit message: Issue #1027 - Schematics final changes.
Parts:
- removed R336: 1K, ~, symbol R
Connections:
- wire segments 235 -> 234
Other:
- note added: "LDO OUT FOR GTP-TX"
Changed lines of the file:
@@
 GND
-$Comp
-L R R336
-U 1 1 534377F2
-P 12350 5000
-F 0 "R336" V 12300 4750 40  0000 C CNN
-F 1 "1K" V 12357 5001 40  0000 C CNN
-F 2 "~" V 12280 5000 30  0000 C CNN
-F 3 "~" H 12350 5000 30  0000 C CNN
-	1    12350 5000
-	0    -1   -1   0
-$EndComp
 $Comp
 L ΜA78L00 U24
@@
 Connection ~ 10150 6350
 Wire Wire Line
-	11450 5000 12100 5000
+	11450 5000 12550 5000
 Wire Wire Line
 	9250 1550 9600 1550
@@
 Wire Wire Line
 	8650 5000 8900 5000
-Wire Wire Line
-	12600 5000 13050 5000
 Wire Wire Line
 	12800 9200 12600 9200
@@
 	12750 9350 12750 9200
 Connection ~ 12750 9200
-Text Label 13050 5000 2    39   ~ 0
+Text Label 12550 5000 2    39   ~ 0
 GTP-TX-VCC5V0
 Wire Notes Line
@@
 Text Notes 13050 7850 0    39   ~ 0
 =3.2V
+Wire Notes Line
+	12450 8750 13400 8750
+Wire Notes Line
+	13400 8750 13400 8600
+Text Notes 12550 8700 0    39   ~ 0
+LDO OUT FOR GTP-TX
+Wire Notes Line
+	8200 2700 9250 2700
+Wire Notes Line
+	9250 2700 9250 2500
+Wire Notes Line
+	10850 2700 11800 2700
+Wire Notes Line
+	11800 2700 11800 2500
 $EndSCHEMATC

Commit message: Issue #1053 - Cypress routing
Connections:
- net labels added: GTP-RX_HOT, GTP-RX_SCL, GTP-RX_SDA, GTP-TX_HOT, GTP-TX_SCL, GTP-TX_SDA
Changed lines of the file:
@@
 Sheet 4 8
 Title "HDMI2USB"
-Date "17 apr 2014"
+Date "25 apr 2014"
 Rev ""
 Comp ""
@@
 GND
 Text Label 10350 7350 0    39   ~ 0
-GTP-RX-SDA
+GTP-RX_SDA
 Text Label 11550 7400 0    39   ~ 0
-GTP-RX-SCL
+GTP-RX_SCL
 $Comp
 L R R318
@@
 GND
 Text Label 9800 8450 2    39   ~ 0
-GTP-RX-HOT
-Text Label 9300 5200 2    39   ~ 0
-GTP-RX-HOT
+GTP-RX_HOT
 Text Label 9300 4300 2    39   ~ 0
-GTP-RX-SDA
+GTP-RX_SDA
 Text Label 9300 4200 2    39   ~ 0
-GTP-RX-SCL
+GTP-RX_SCL
 Text HLabel 11800 7950 0    60   BiDi ~ 0
 GTP-RX-SCL
 Text Label 9150 8850 0    39   ~ 0
-GTP-TX-SDA
+GTP-TX_SDA
 Text Label 10350 8950 0    39   ~ 0
-GTP-TX-SCL
+GTP-TX_SCL
 Text Label 11600 8850 0    39   ~ 0
-GTP-TX-HOT
+GTP-TX_HOT
 $Comp
 L NPN Q1
@@
 VCC5V0
 Text Label 12100 4300 0    39   ~ 0
-GTP-TX-SDA
+GTP-TX_SDA
 Text Label 12100 4200 0    39   ~ 0
-GTP-TX-SCL
+GTP-TX_SCL
 Text Label 12100 5200 0    39   ~ 0
-GTP-TX-HOT
+GTP-TX_HOT
 $Comp
 L R R301
@@
 Wire Notes Line
 	11800 2700 11800 2500
+Text Label 9300 5200 2    39   ~ 0
+GTP-RX_HOT
 $EndSCHEMATC

Commit message: Issue #1050
Connections:
- net labels added: R-EXP-IO10_N, R-EXP-IO10_P, R-EXP-IO11_N, R-EXP-IO11_P, R-EXP-IO12_N, R-EXP-IO12_P, R-EXP-IO13_N, R-EXP-IO13_P, R-EXP-IO14_N, R-EXP-IO14_P, R-EXP-IO15_N, R-EXP-IO15_P, R-EXP-IO16_N, R-EXP-IO16_P, R-EXP-IO17_N, R-EXP-IO17_P, R-EXP-IO18_N, R-EXP-IO18_P, R-EXP-IO19_N, R-EXP-IO19_P, R-EXP-IO1_N, R-EXP-IO1_P, R-EXP-IO20_N, R-EXP-IO20_P, R-EXP-IO2_N, R-EXP-IO2_P, R-EXP-IO3_N, R-EXP-IO3_P, R-EXP-IO4_N, R-EXP-IO4_P, R-EXP-IO5_N, R-EXP-IO5_P, R-EXP-IO6_N, R-EXP-IO6_P, R-EXP-IO7_N, R-EXP-IO7_P, R-EXP-IO8_N, R-EXP-IO8_P, R-EXP-IO9_N, R-EXP-IO9_P
Changed lines of the file:
@@
 LIBS:contrib
 LIBS:valves
-LIBS:xc6slx9-csg324
 LIBS:hdmi2usb
-LIBS:cypress-fx2
 LIBS:hdmi2usb-cache
 EELAYER 27 0
@@
 Sheet 4 8
 Title "HDMI2USB"
-Date "29 apr 2014"
+Date "2 may 2014"
 Rev ""
 Comp ""
@@
 $EndComp
 Text Label 2350 6850 2    39   ~ 0
-EXP-IO1_P
+R-EXP-IO1_P
 Text Label 2350 7050 2    39   ~ 0
-EXP-IO1_N
+R-EXP-IO1_N
 Text Label 2600 1850 2    39   ~ 0
-EXP-IO1_P
+R-EXP-IO1_P
 Text Label 4400 1850 0    39   ~ 0
-EXP-IO1_N
+R-EXP-IO1_N
 Text Label 2350 7450 2    39   ~ 0
-EXP-IO2_N
+R-EXP-IO2_N
 Text Label 2350 7250 2    39   ~ 0
-EXP-IO2_P
+R-EXP-IO2_P
 $Comp
 L RES_NET4 R102
@@
 $EndComp
 Text Label 2350 7850 2    39   ~ 0
-EXP-IO3_N
+R-EXP-IO3_N
 Text Label 2350 7650 2    39   ~ 0
-EXP-IO3_P
+R-EXP-IO3_P
 Text Label 2350 8250 2    39   ~ 0
-EXP-IO4_N
+R-EXP-IO4_N
 Text Label 2350 8050 2    39   ~ 0
-EXP-IO4_P
+R-EXP-IO4_P
 Text Label 4400 2150 0    39   ~ 0
-EXP-IO3_N
+R-EXP-IO3_N
 Text Label 4400 2050 0    39   ~ 0
-EXP-IO2_N
+R-EXP-IO2_N
 Text Label 4400 2350 0    39   ~ 0
-EXP-IO4_N
+R-EXP-IO4_N
 Text Label 2600 2050 2    39   ~ 0
-EXP-IO2_P
+R-EXP-IO2_P
 Text Label 2600 2150 2    39   ~ 0
-EXP-IO3_P
+R-EXP-IO3_P
 Text Label 2600 2350 2    39   ~ 0
-EXP-IO4_P
+R-EXP-IO4_P
 $Comp
 L RES_NET4 R103
@@
 EXP-IO13_P
 Text Label 3900 7050 2    39   ~ 0
-EXP-IO7_N
+R-EXP-IO7_N
 Text Label 3900 6850 2    39   ~ 0
-EXP-IO7_P
+R-EXP-IO7_P
 Text Label 3900 7450 2    39   ~ 0
-EXP-IO8_N
+R-EXP-IO8_N
 Text Label 3900 7250 2    39   ~ 0
-EXP-IO8_P
+R-EXP-IO8_P
 Text Label 3900 7850 2    39   ~ 0
-EXP-IO9_N
+R-EXP-IO9_N
 Text Label 3900 7650 2    39   ~ 0
-EXP-IO9_P
+R-EXP-IO9_P
 Text Label 3900 8250 2    39   ~ 0
-EXP-IO10_N
+R-EXP-IO10_N
 Text Label 3900 8050 2    39   ~ 0
-EXP-IO10_P
+R-EXP-IO10_P
 Text Label 3900 8650 2    39   ~ 0
-EXP-IO11_N
+R-EXP-IO11_N
 Text Label 3900 8450 2    39   ~ 0
-EXP-IO11_P
+R-EXP-IO11_P
 Text Label 3900 9050 2    39   ~ 0
-EXP-IO12_N
+R-EXP-IO12_N
 Text Label 3900 8850 2    39   ~ 0
-EXP-IO12_P
+R-EXP-IO12_P
 Text Label 6100 6550 2    39   ~ 0
-EXP-IO13_N
+R-EXP-IO13_N
 Text Label 6100 6350 2    39   ~ 0
-EXP-IO13_P
+R-EXP-IO13_P
 Text Label 6100 6950 2    39   ~ 0
-EXP-IO14_N
+R-EXP-IO14_N
 Text Label 6100 6750 2    39   ~ 0
-EXP-IO14_P
+R-EXP-IO14_P
 Text Label 6100 7350 2    39   ~ 0
-EXP-IO15_N
+R-EXP-IO15_N
 Text Label 6100 7150 2    39   ~ 0
-EXP-IO15_P
+R-EXP-IO15_P
 Text Label 6100 7750 2    39   ~ 0
-EXP-IO16_N
+R-EXP-IO16_N
 Text Label 6100 7550 2    39   ~ 0
-EXP-IO16_P
+R-EXP-IO16_P
 Text Label 6100 8700 2    39   ~ 0
-EXP-IO17_N
+R-EXP-IO17_N
 Text Label 6100 8500 2    39   ~ 0
-EXP-IO17_P
+R-EXP-IO17_P
 Text Label 6100 9100 2    39   ~ 0
-EXP-IO18_N
+R-EXP-IO18_N
 Text Label 6100 8900 2    39   ~ 0
-EXP-IO18_P
+R-EXP-IO18_P
 Text Label 6100 9500 2    39   ~ 0
-EXP-IO19_N
+R-EXP-IO19_N
 Text Label 6100 9300 2    39   ~ 0
-EXP-IO19_P
+R-EXP-IO19_P
 Text Label 6100 9900 2    39   ~ 0
-EXP-IO20_N
+R-EXP-IO20_N
 Text Label 6100 9700 2    39   ~ 0
-EXP-IO20_P
+R-EXP-IO20_P
 Text Label 2350 8650 2    39   ~ 0
-EXP-IO5_N
+R-EXP-IO5_N
 Text Label 2350 8450 2    39   ~ 0
-EXP-IO5_P
+R-EXP-IO5_P
 Text Label 2350 9050 2    39   ~ 0
-EXP-IO6_N
+R-EXP-IO6_N
 Text Label 2350 8850 2    39   ~ 0
-EXP-IO6_P
+R-EXP-IO6_P
 Text Label 4400 2450 0    39   ~ 0
-EXP-IO5_N
+R-EXP-IO5_N
 Text Label 2600 2450 2    39   ~ 0
-EXP-IO5_P
+R-EXP-IO5_P
 Text Label 4400 2650 0    39   ~ 0
-EXP-IO6_N
+R-EXP-IO6_N
 Text Label 2600 2650 2    39   ~ 0
-EXP-IO6_P
+R-EXP-IO6_P
 Text Label 4400 2750 0    39   ~ 0
-EXP-IO7_N
+R-EXP-IO7_N
 Text Label 2600 2750 2    39   ~ 0
-EXP-IO7_P
+R-EXP-IO7_P
 Text Label 4400 2950 0    39   ~ 0
-EXP-IO8_N
+R-EXP-IO8_N
 Text Label 2600 2950 2    39   ~ 0
-EXP-IO8_P
+R-EXP-IO8_P
 Text Label 4400 3050 0    39   ~ 0
-EXP-IO9_N
+R-EXP-IO9_N
 Text Label 2600 3050 2    39   ~ 0
-EXP-IO9_P
+R-EXP-IO9_P
 Text Label 4400 3250 0    39   ~ 0
-EXP-IO10_N
+R-EXP-IO10_N
 Text Label 2600 3250 2    39   ~ 0
-EXP-IO10_P
+R-EXP-IO10_P
 Text Label 4400 3750 0    39   ~ 0
-EXP-IO11_N
+R-EXP-IO11_N
 Text Label 2600 3750 2    39   ~ 0
-EXP-IO11_P
+R-EXP-IO11_P
 Text Label 4400 3950 0    39   ~ 0
-EXP-IO12_N
+R-EXP-IO12_N
 Text Label 2600 3950 2    39   ~ 0
-EXP-IO12_P
+R-EXP-IO12_P
 Text Label 4400 4050 0    39   ~ 0
-EXP-IO13_N
+R-EXP-IO13_N
 Text Label 2600 4050 2    39   ~ 0
-EXP-IO13_P
+R-EXP-IO13_P
 Text Label 4400 4250 0    39   ~ 0
-EXP-IO14_N
+R-EXP-IO14_N
 Text Label 2600 4250 2    39   ~ 0
-EXP-IO14_P
+R-EXP-IO14_P
 Text Label 4400 4350 0    39   ~ 0
-EXP-IO15_N
+R-EXP-IO15_N
 Text Label 2600 4350 2    39   ~ 0
-EXP-IO15_P
+R-EXP-IO15_P
 Text Label 4400 4550 0    39   ~ 0
-EXP-IO16_N
+R-EXP-IO16_N
 Text Label 2600 4550 2    39   ~ 0
-EXP-IO16_P
+R-EXP-IO16_P
 Text Label 4400 4650 0    39   ~ 0
-EXP-IO17_N
+R-EXP-IO17_N
 Text Label 2600 4650 2    39   ~ 0
-EXP-IO17_P
+R-EXP-IO17_P
 Text Label 4400 4850 0    39   ~ 0
-EXP-IO18_N
+R-EXP-IO18_N
 Text Label 2600 4850 2    39   ~ 0
-EXP-IO18_P
+R-EXP-IO18_P
 Text Label 4400 4950 0    39   ~ 0
-EXP-IO19_N
+R-EXP-IO19_N
 Text Label 2600 4950 2    39   ~ 0
-EXP-IO19_P
+R-EXP-IO19_P
 Text Label 4400 5150 0    39   ~ 0
-EXP-IO20_N
+R-EXP-IO20_N
 Text Label 2600 5150 2    39   ~ 0
-EXP-IO20_P
+R-EXP-IO20_P
 $Comp
 L R R291
