File: board/power.sch (KiCad schematic (older format))
At the start: 0 parts

Commit message: Issue #412
Parts:
- added U10, U11, U12: LMR10530, ~, symbol LMR10530
- added U13: LP2997, symbol LP2997
Changed lines of the file:
@@
 Sheet 3 7
 Title ""
-Date "31 jul 2013"
+Date "10 aug 2013"
 Rev ""
 Comp ""
@@
 Comment4 ""
 $EndDescr
+$Comp
+L LMR10530 U10
+U 1 1 52060750
+P 5650 2050
+F 0 "U10" H 5700 2350 60  0000 C CNN
+F 1 "LMR10530" H 5700 2950 60  0000 C CNN
+F 2 "~" H 3300 2250 60  0000 C CNN
+F 3 "~" H 3300 2250 60  0000 C CNN
+	1    5650 2050
+	1    0    0    -1
+$EndComp
+$Comp
+L LP2997 U13
+U 1 1 5206092A
+P 8050 5750
+F 0 "U13" H 8600 5350 60  0000 C CNN
+F 1 "LP2997" H 8250 6150 60  0000 C CNN
+F 2 "" H 8050 5750 60  0000 C CNN
+F 3 "" H 8050 5750 60  0000 C CNN
+	1    8050 5750
+	1    0    0    -1
+$EndComp
+$Comp
+L LMR10530 U11
+U 1 1 52060937
+P 5650 3900
+F 0 "U11" H 5700 4200 60  0000 C CNN
+F 1 "LMR10530" H 5700 4800 60  0000 C CNN
+F 2 "~" H 3300 4100 60  0000 C CNN
+F 3 "~" H 3300 4100 60  0000 C CNN
+	1    5650 3900
+	1    0    0    -1
+$EndComp
+$Comp
+L LMR10530 U12
+U 1 1 5206093D
+P 5750 5950
+F 0 "U12" H 5800 6250 60  0000 C CNN
+F 1 "LMR10530" H 5800 6850 60  0000 C CNN
+F 2 "~" H 3400 6150 60  0000 C CNN
+F 3 "~" H 3400 6150 60  0000 C CNN
+	1    5750 5950
+	1    0    0    -1
+$EndComp
 $EndSCHEMATC

Commit message: Issue #412 - Placement
Parts:
- removed U11, U12: LMR10530, ~, symbol LMR10530
- added C? (x13): C, ~, symbol C
- added D? (x3): DIODESCH, ~, symbol DIODESCH
- added L? (x3): INDUCTOR, ~, symbol INDUCTOR
- added R? (x9): R, ~, symbol R
- added U? (x2): LMR10530, ~, symbol LMR10530
Connections:
- net at U10.1 (VINC): now also U10.2 (EN), C?.1, R?.2
- net VCC5V0: now reaches U10.10 (VIND)
- net VCC5V0: now also U10.9 (VIND), U13.2 (~SD), U13.6 (AVIN), C?.1, C?.1, C?.1, C?.1, R?.1, R?.1, R?.1, U?.10 (VIND), U?.10 (VIND), U?.9 (VIND), U?.9 (VIND)
- net GND: now reaches U10.3 (SGND)
- net GND: now also U10.4 (NC), U10.6 (PGND), U13.1 (GND), C?.2, C?.2, C?.2, C?.2, C?.2, C?.2, C?.2, C?.2, C?.2, C?.2, C?.2, C?.2, C?.2, D?.1 (A), D?.1 (A), D?.1 (A), R?.2, R?.2, R?.2, U?.3 (SGND), U?.3 (SGND), U?.4 (NC), U?.4 (NC), U?.6 (PGND), U?.6 (PGND)
- net at U10.5 (FB): now also R?.1, R?.2
- net at U10.7 (SW): now also U10.8 (SW), D?.2 (K), L?.1
- net at U13.3 (VSEN): now also C?.1
- net DDR1V8: now reaches U13.5 (VDDQ)
- net DDR1V8: now also U13.7 (PVIN), C?.1, C?.1, L?.2, R?.1
- net DDR0V9: now reaches U13.8 (VTT)
- net DDR0V9: now also C?.1
- new net: C?.1, R?.2, U?.1 (VINC), U?.2 (EN) (x2)
- new net: R?.1, R?.2, U?.5 (FB) (x2)
- new net: D?.2 (K), L?.1, U?.7 (SW), U?.8 (SW) (x2)
- new net VCC1V2: C?.1, L?.2, R?.1
- new net VCC3V3: C?.1, L?.2, R?.1
- no-connect marks 0 -> 1
Other:
- moved on the sheet: U13

Commit message: Issue #510
Parts:
- gave numbers to parts that had none: 30
- renumbered U10 to U3, U13 to U6
Changed lines of the file:
@@
 Sheet 3 7
 Title ""
-Date "11 aug 2013"
+Date "3 sep 2013"
 Rev ""
 Comp ""
@@
 $EndDescr
 $Comp
-L LMR10530 U10
+L LMR10530 U3
 U 1 1 52060750
 P 5650 2050
-F 0 "U10" H 5700 2350 60  0000 C CNN
+F 0 "U3" H 5700 2350 60  0000 C CNN
 F 1 "LMR10530" H 5700 2950 60  0000 C CNN
 F 2 "~" H 3300 2250 60  0000 C CNN
@@
 $EndComp
 $Comp
-L LP2997 U13
+L LP2997 U6
 U 1 1 5206092A
 P 9200 3000
-F 0 "U13" H 9750 2600 60  0000 C CNN
+F 0 "U6" H 9750 2600 60  0000 C CNN
 F 1 "LP2997" H 9400 3400 60  0000 C CNN
 F 2 "" H 9200 3000 60  0000 C CNN
@@
 DDR1V8
 $Comp
-L C C?
+L C C23
 U 1 1 52080654
 P 8500 3350
-F 0 "C?" H 8500 3450 40  0000 L CNN
+F 0 "C23" H 8500 3450 40  0000 L CNN
 F 1 "C" H 8506 3265 40  0000 L CNN
 F 2 "~" H 8538 3200 30  0000 C CNN
@@
 GND
 $Comp
-L C C?
+L C C22
 U 1 1 52080681
 P 8250 3350
-F 0 "C?" H 8250 3450 40  0000 L CNN
+F 0 "C22" H 8250 3450 40  0000 L CNN
 F 1 "C" H 8256 3265 40  0000 L CNN
 F 2 "~" H 8288 3200 30  0000 C CNN
@@
 $EndComp
 $Comp
-L C C?
+L C C24
 U 1 1 52080705
 P 10200 3350
-F 0 "C?" H 10200 3450 40  0000 L CNN
+F 0 "C24" H 10200 3450 40  0000 L CNN
 F 1 "C" H 10206 3265 40  0000 L CNN
 F 2 "~" H 10238 3200 30  0000 C CNN
@@
 DDR0V9
 $Comp
-L C C?
+L C C25
 U 1 1 5208074C
 P 10400 3350
-F 0 "C?" H 10400 3450 40  0000 L CNN
+F 0 "C25" H 10400 3450 40  0000 L CNN
 F 1 "C" H 10406 3265 40  0000 L CNN
 F 2 "~" H 10438 3200 30  0000 C CNN
@@
 VCC5V0
 $Comp
-L R R?
+L R R35
 U 1 1 52080807
 P 4900 1750
-F 0 "R?" V 4980 1750 40  0000 C CNN
+F 0 "R35" V 4980 1750 40  0000 C CNN
 F 1 "R" V 4907 1751 40  0000 C CNN
 F 2 "~" V 4830 1750 30  0000 C CNN
@@
 $EndComp
 $Comp
-L C C?
+L C C13
 U 1 1 52080896
 P 4750 1750
-F 0 "C?" H 4750 1850 40  0000 L CNN
+F 0 "C13" H 4750 1850 40  0000 L CNN
 F 1 "C" H 4756 1665 40  0000 L CNN
 F 2 "~" H 4788 1600 30  0000 C CNN
@@
 $EndComp
 $Comp
-L C C?
+L C C16
 U 1 1 5208097C
 P 4900 2400
-F 0 "C?" H 4900 2500 40  0000 L CNN
+F 0 "C16" H 4900 2500 40  0000 L CNN
 F 1 "C" H 4906 2315 40  0000 L CNN
 F 2 "~" H 4938 2250 30  0000 C CNN
@@
 GND
 $Comp
-L R R?
+L R R38
 U 1 1 52080A6E
 P 7350 1550
-F 0 "R?" V 7430 1550 40  0000 C CNN
+F 0 "R38" V 7430 1550 40  0000 C CNN
 F 1 "R" V 7357 1551 40  0000 C CNN
 F 2 "~" V 7280 1550 30  0000 C CNN
@@
 	6300 1850 7350 1850
 $Comp
-L R R?
+L R R39
 U 1 1 52080B4B
 P 7350 2200
-F 0 "R?" V 7430 2200 40  0000 C CNN
+F 0 "R39" V 7430 2200 40  0000 C CNN
 F 1 "R" V 7357 2201 40  0000 C CNN
 F 2 "~" V 7280 2200 30  0000 C CNN
@@
 Connection ~ 6400 2700
 $Comp
-L C C?
+L C C19
 U 1 1 52080BC0
 P 7600 1750
-F 0 "C?" H 7600 1850 40  0000 L CNN
+F 0 "C19" H 7600 1850 40  0000 L CNN
 F 1 "C" H 7606 1665 40  0000 L CNN
 F 2 "~" H 7638 1600 30  0000 C CNN
@@
 Connection ~ 6600 2700
 $Comp
-L INDUCTOR L?
+L INDUCTOR L1
 U 1 1 52080C7C
 P 6750 1250
-F 0 "L?" V 6700 1250 40  0000 C CNN
+F 0 "L1" V 6700 1250 40  0000 C CNN
 F 1 "INDUCTOR" V 6850 1250 40  0000 C CNN
 F 2 "~" H 6750 1250 60  0000 C CNN
@@
 Connection ~ 7350 2700
 $Comp
-L DIODESCH D?
+L DIODESCH D1
 U 1 1 52080D95
 P 6400 1550
-F 0 "D?" H 6400 1650 40  0000 C CNN
+F 0 "D1" H 6400 1650 40  0000 C CNN
 F 1 "DIODESCH" H 6400 1450 40  0000 C CNN
 F 2 "~" H 6400 1550 60  0000 C CNN
@@
 GND
 $Comp
-L LMR10530 U?
+L LMR10530 U4
 U 1 1 52080E26
 P 5650 3950
-F 0 "U?" H 5700 4250 60  0000 C CNN
+F 0 "U4" H 5700 4250 60  0000 C CNN
 F 1 "LMR10530" H 5700 4850 60  0000 C CNN
 F 2 "~" H 3300 4150 60  0000 C CNN
@@
 VCC5V0
 $Comp
-L R R?
+L R R36
 U 1 1 52080E2D
 P 4900 3650
-F 0 "R?" V 4980 3650 40  0000 C CNN
+F 0 "R36" V 4980 3650 40  0000 C CNN
 F 1 "R" V 4907 3651 40  0000 C CNN
 F 2 "~" V 4830 3650 30  0000 C CNN
@@
 $EndComp
 $Comp
-L C C?
+L C C14
 U 1 1 52080E33
 P 4750 3650
-F 0 "C?" H 4750 3750 40  0000 L CNN
+F 0 "C14" H 4750 3750 40  0000 L CNN
 F 1 "C" H 4756 3565 40  0000 L CNN
 F 2 "~" H 4788 3500 30  0000 C CNN
@@
 $EndComp
 $Comp
-L C C?
+L C C17
 U 1 1 52080E39
 P 4900 4300
-F 0 "C?" H 4900 4400 40  0000 L CNN
+F 0 "C17" H 4900 4400 40  0000 L CNN
 F 1 "C" H 4906 4215 40  0000 L CNN
 F 2 "~" H 4938 4150 30  0000 C CNN
@@
 GND
 $Comp
-L R R?
+L R R40
 U 1 1 52080E40
 P 7350 3450
-F 0 "R?" V 7430 3450 40  0000 C CNN
+F 0 "R40" V 7430 3450 40  0000 C CNN
 F 1 "R" V 7357 3451 40  0000 C CNN
 F 2 "~" V 7280 3450 30  0000 C CNN
@@
 	6300 3750 7350 3750
 $Comp
-L R R?
+L R R41
 U 1 1 52080E62
 P 7350 4100
-F 0 "R?" V 7430 4100 40  0000 C CNN
+F 0 "R41" V 7430 4100 40  0000 C CNN
 F 1 "R" V 7357 4101 40  0000 C CNN
 F 2 "~" V 7280 4100 30  0000 C CNN
@@
 Connection ~ 6400 4600
 $Comp
-L C C?
+L C C20
 U 1 1 52080E6B
 P 7600 3650
-F 0 "C?" H 7600 3750 40  0000 L CNN
+F 0 "C20" H 7600 3750 40  0000 L CNN
 F 1 "C" H 7606 3565 40  0000 L CNN
 F 2 "~" H 7638 3500 30  0000 C CNN
@@
 Connection ~ 6600 4600
 $Comp
-L INDUCTOR L?
+L INDUCTOR L2
 U 1 1 52080E75
 P 6750 3150
-F 0 "L?" V 6700 3150 40  0000 C CNN
+F 0 "L2" V 6700 3150 40  0000 C CNN
 F 1 "INDUCTOR" V 6850 3150 40  0000 C CNN
 F 2 "~" H 6750 3150 60  0000 C CNN
@@
 Connection ~ 7350 4600
 $Comp
-L DIODESCH D?
+L DIODESCH D2
 U 1 1 52080E7D
 P 6400 3450
-F 0 "D?" H 6400 3550 40  0000 C CNN
+F 0 "D2" H 6400 3550 40  0000 C CNN
 F 1 "DIODESCH" H 6400 3350 40  0000 C CNN
 F 2 "~" H 6400 3450 60  0000 C CNN
@@
 GND
 $Comp
-L LMR10530 U?
+L LMR10530 U5
 U 1 1 52080E87
 P 5650 5800
-F 0 "U?" H 5700 6100 60  0000 C CNN
+F 0 "U5" H 5700 6100 60  0000 C CNN
 F 1 "LMR10530" H 5700 6700 60  0000 C CNN
 F 2 "~" H 3300 6000 60  0000 C CNN
@@
 VCC5V0
 $Comp
-L R R?
+L R R37
 U 1 1 52080E8E
 P 4900 5500
-F 0 "R?" V 4980 5500 40  0000 C CNN
+F 0 "R37" V 4980 5500 40  0000 C CNN
 F 1 "R" V 4907 5501 40  0000 C CNN
 F 2 "~" V 4830 5500 30  0000 C CNN
@@
 $EndComp
 $Comp
-L C C?
+L C C15
 U 1 1 52080E94
 P 4750 5500
-F 0 "C?" H 4750 5600 40  0000 L CNN
+F 0 "C15" H 4750 5600 40  0000 L CNN
 F 1 "C" H 4756 5415 40  0000 L CNN
 F 2 "~" H 4788 5350 30  0000 C CNN
@@
 $EndComp
 $Comp
-L C C?
+L C C18
 U 1 1 52080E9A
 P 4900 6150
-F 0 "C?" H 4900 6250 40  0000 L CNN
+F 0 "C18" H 4900 6250 40  0000 L CNN
 F 1 "C" H 4906 6065 40  0000 L CNN
 F 2 "~" H 4938 6000 30  0000 C CNN
@@
 GND
 $Comp
-L R R?
+L R R42
 U 1 1 52080EA1
 P 7350 5300
-F 0 "R?" V 7430 5300 40  0000 C CNN
+F 0 "R42" V 7430 5300 40  0000 C CNN
 F 1 "R" V 7357 5301 40  0000 C CNN
 F 2 "~" V 7280 5300 30  0000 C CNN
@@
 	6300 5600 7350 5600
 $Comp
-L R R?
+L R R43
 U 1 1 52080EC3
 P 7350 5950
-F 0 "R?" V 7430 5950 40  0000 C CNN
+F 0 "R43" V 7430 5950 40  0000 C CNN
 F 1 "R" V 7357 5951 40  0000 C CNN
 F 2 "~" V 7280 5950 30  0000 C CNN
@@
 Connection ~ 6400 6450
 $Comp
-L C C?
+L C C21
 U 1 1 52080ECC
 P 7600 5500
-F 0 "C?" H 7600 5600 40  0000 L CNN
+F 0 "C21" H 7600 5600 40  0000 L CNN
 F 1 "C" H 7606 5415 40  0000 L CNN
 F 2 "~" H 7638 5350 30  0000 C CNN
@@
 Connection ~ 6600 6450
 $Comp
-L INDUCTOR L?
+L INDUCTOR L3
 U 1 1 52080ED6
 P 6750 5000
-F 0 "L?" V 6700 5000 40  0000 C CNN
+F 0 "L3" V 6700 5000 40  0000 C CNN
 F 1 "INDUCTOR" V 6850 5000 40  0000 C CNN
 F 2 "~" H 6750 5000 60  0000 C CNN
@@
 Connection ~ 7350 6450
 $Comp
-L DIODESCH D?
+L DIODESCH D3
 U 1 1 52080EDE
 P 6400 5300
-F 0 "D?" H 6400 5400 40  0000 C CNN
+F 0 "D3" H 6400 5400 40  0000 C CNN
 F 1 "DIODESCH" H 6400 5200 40  0000 C CNN
 F 2 "~" H 6400 5300 60  0000 C CNN
