File: board/power.sch (KiCad schematic (older format))
At the start: 149 parts, among them CON1 BARREL_JACK, CON2 BARREL_JACK, P47 CONN_2, U14 TPS53319, U15 GBU15005-G, U16 TPS54560, U3 TPS54625, U4 TPS54625, U5 TPS54625, U6 TPS51200

Commit message: Issue #1022 - Schematics final.
Changed lines of the file:
@@
 Sheet 6 8
 Title "SP6N02"
-Date "28 mar 2014"
+Date "31 mar 2014"
 Rev "V1"
 Comp "Numato Lab"
@@
 $EndComp
 $Comp
-L GND #PWR13
+L GND #PWR04
 U 1 1 52DD9648
 P 11300 7700
-F 0 "#PWR13" H 11300 7700 30  0001 C CNN
+F 0 "#PWR04" H 11300 7700 30  0001 C CNN
 F 1 "GND" H 11300 7630 30  0001 C CNN
 F 2 "" H 11300 7700 60  0000 C CNN
@@
 $EndComp
 $Comp
-L GND #PWR17
+L GND #PWR05
 U 1 1 52DD9786
 P 12800 5350
-F 0 "#PWR17" H 12800 5350 30  0001 C CNN
+F 0 "#PWR05" H 12800 5350 30  0001 C CNN
 F 1 "GND" H 12800 5280 30  0001 C CNN
 F 2 "" H 12800 5350 60  0000 C CNN
@@
 $EndComp
 $Comp
-L GND #PWR16
+L GND #PWR06
 U 1 1 52DD9A04
 P 11500 1100
-F 0 "#PWR16" H 11500 1100 30  0001 C CNN
+F 0 "#PWR06" H 11500 1100 30  0001 C CNN
 F 1 "GND" H 11500 1030 30  0001 C CNN
 F 2 "" H 11500 1100 60  0000 C CNN
@@
 $EndComp
 $Comp
-L GND #PWR8
+L GND #PWR07
 U 1 1 52DD9A0A
 P 9400 2950
-F 0 "#PWR8" H 9400 2950 30  0001 C CNN
+F 0 "#PWR07" H 9400 2950 30  0001 C CNN
 F 1 "GND" H 9400 2880 30  0001 C CNN
 F 2 "" H 9400 2950 60  0000 C CNN
@@
 $EndComp
 $Comp
-L GND #PWR4
+L GND #PWR08
 U 1 1 52E1FEA6
 P 4000 1950
-F 0 "#PWR4" H 4000 1950 30  0001 C CNN
+F 0 "#PWR08" H 4000 1950 30  0001 C CNN
 F 1 "GND" H 4000 1880 30  0001 C CNN
 F 2 "" H 4000 1950 60  0000 C CNN
@@
 $EndComp
 $Comp
-L TPS51200 U6
-U 1 1 52E4CA5E
-P 12150 9350
-F 0 "U6" H 12100 8950 60  0000 C CNN
-F 1 "TPS51200" H 12150 9650 60  0000 C CNN
-F 2 "" H 12200 9000 60  0000 C CNN
-F 3 "" H 12200 9000 60  0000 C CNN
-	1    12150 9350
-	1    0    0    -1
-$EndComp
-$Comp
 L R R41
 U 1 1 52E4CA64
@@
 $EndComp
 $Comp
-L GND #PWR12
+L GND #PWR09
 U 1 1 52E4CA76
 P 10900 8600
-F 0 "#PWR12" H 10900 8600 30  0001 C CNN
+F 0 "#PWR09" H 10900 8600 30  0001 C CNN
 F 1 "GND" H 10900 8530 30  0001 C CNN
 F 2 "" H 10900 8600 60  0000 C CNN
@@
 $EndComp
 $Comp
-L GND #PWR9
+L GND #PWR010
 U 1 1 52E4CA88
 P 10450 9800
-F 0 "#PWR9" H 10450 9800 30  0001 C CNN
+F 0 "#PWR010" H 10450 9800 30  0001 C CNN
 F 1 "GND" H 10450 9730 30  0001 C CNN
 F 2 "" H 10450 9800 60  0000 C CNN
@@
 $EndComp
 $Comp
-L GND #PWR21
+L GND #PWR011
 U 1 1 52E4CAA0
 P 13800 9800
-F 0 "#PWR21" H 13800 9800 30  0001 C CNN
+F 0 "#PWR011" H 13800 9800 30  0001 C CNN
 F 1 "GND" H 13800 9730 30  0001 C CNN
 F 2 "" H 13800 9800 60  0000 C CNN
@@
 $EndComp
 $Comp
-L GND #PWR20
+L GND #PWR012
 U 1 1 52E4CAAC
 P 13200 9300
-F 0 "#PWR20" H 13200 9300 30  0001 C CNN
+F 0 "#PWR012" H 13200 9300 30  0001 C CNN
 F 1 "GND" H 13200 9230 30  0001 C CNN
 F 2 "" H 13200 9300 60  0000 C CNN
@@
 $EndComp
 $Comp
-L GND #PWR14
+L GND #PWR013
 U 1 1 52E4CAB8
 P 11350 9950
-F 0 "#PWR14" H 11350 9950 30  0001 C CNN
+F 0 "#PWR013" H 11350 9950 30  0001 C CNN
 F 1 "GND" H 11350 9880 30  0001 C CNN
 F 2 "" H 11350 9950 60  0000 C CNN
@@
 VCC3V3
 $Comp
-L GND #PWR18
+L GND #PWR014
 U 1 1 52E4CABF
 P 12800 9700
-F 0 "#PWR18" H 12800 9700 30  0001 C CNN
+F 0 "#PWR014" H 12800 9700 30  0001 C CNN
 F 1 "GND" H 12800 9630 30  0001 C CNN
 F 2 "" H 12800 9700 60  0000 C CNN
@@
 $EndComp
 $Comp
-L GND #PWR19
+L GND #PWR015
 U 1 1 52E4CACB
 P 13100 9950
-F 0 "#PWR19" H 13100 9950 30  0001 C CNN
+F 0 "#PWR015" H 13100 9950 30  0001 C CNN
 F 1 "GND" H 13100 9880 30  0001 C CNN
 F 2 "" H 13100 9950 60  0000 C CNN
@@
 $EndComp
 $Comp
-L GND #PWR10
+L GND #PWR016
 U 1 1 52F26CB0
 P 10650 3700
-F 0 "#PWR10" H 10650 3700 30  0001 C CNN
+F 0 "#PWR016" H 10650 3700 30  0001 C CNN
 F 1 "GND" H 10650 3630 30  0001 C CNN
 F 2 "" H 10650 3700 60  0000 C CNN
@@
 $EndComp
 $Comp
-L GND #PWR11
+L GND #PWR017
 U 1 1 52F2BB58
 P 10900 6200
-F 0 "#PWR11" H 10900 6200 30  0001 C CNN
+F 0 "#PWR017" H 10900 6200 30  0001 C CNN
 F 1 "GND" H 10900 6130 30  0001 C CNN
 F 2 "" H 10900 6200 60  0000 C CNN
@@
 $EndComp
 $Comp
-L GND #PWR15
+L GND #PWR018
 U 1 1 52F2C00C
 P 11450 6150
-F 0 "#PWR15" H 11450 6150 30  0001 C CNN
+F 0 "#PWR018" H 11450 6150 30  0001 C CNN
 F 1 "GND" H 11450 6080 30  0001 C CNN
 F 2 "" H 11450 6150 60  0000 C CNN
@@
 $EndComp
 $Comp
-L GND #PWR6
+L GND #PWR019
 U 1 1 52FA3E62
 P 6250 9400
-F 0 "#PWR6" H 6250 9400 30  0001 C CNN
+F 0 "#PWR019" H 6250 9400 30  0001 C CNN
 F 1 "GND" H 6250 9330 30  0001 C CNN
 F 2 "" H 6250 9400 60  0000 C CNN
@@
 $EndComp
 $Comp
-L GND #PWR3
+L GND #PWR020
 U 1 1 52FA3EB9
 P 1900 7900
-F 0 "#PWR3" H 1900 7900 30  0001 C CNN
+F 0 "#PWR020" H 1900 7900 30  0001 C CNN
 F 1 "GND" H 1900 7830 30  0001 C CNN
 F 2 "" H 1900 7900 60  0000 C CNN
@@
 $EndComp
 $Comp
-L GND #PWR23
+L GND #PWR021
 U 1 1 530E4356
 P 15100 10050
-F 0 "#PWR23" H 15100 10050 30  0001 C CNN
+F 0 "#PWR021" H 15100 10050 30  0001 C CNN
 F 1 "GND" H 15100 9980 30  0001 C CNN
 F 2 "" H 15100 10050 60  0000 C CNN
@@
 $EndComp
 $Comp
-L GND #PWR24
+L GND #PWR022
 U 1 1 530E4D62
 P 15250 7650
-F 0 "#PWR24" H 15250 7650 30  0001 C CNN
+F 0 "#PWR022" H 15250 7650 30  0001 C CNN
 F 1 "GND" H 15250 7580 30  0001 C CNN
 F 2 "" H 15250 7650 60  0000 C CNN
@@
 $EndComp
 $Comp
-L GND #PWR22
+L GND #PWR023
 U 1 1 530E5A14
 P 15000 5400
-F 0 "#PWR22" H 15000 5400 30  0001 C CNN
+F 0 "#PWR023" H 15000 5400 30  0001 C CNN
 F 1 "GND" H 15000 5330 30  0001 C CNN
 F 2 "" H 15000 5400 60  0000 C CNN
@@
 $EndComp
 $Comp
-L GND #PWR25
+L GND #PWR024
 U 1 1 530E6979
 P 15300 3150
-F 0 "#PWR25" H 15300 3150 30  0001 C CNN
+F 0 "#PWR024" H 15300 3150 30  0001 C CNN
 F 1 "GND" H 15300 3080 30  0001 C CNN
 F 2 "" H 15300 3150 60  0000 C CNN
@@
 $EndComp
 $Comp
-L GND #PWR7
+L GND #PWR025
 U 1 1 530E7C33
 P 8050 3100
-F 0 "#PWR7" H 8050 3100 30  0001 C CNN
+F 0 "#PWR025" H 8050 3100 30  0001 C CNN
 F 1 "GND" H 8050 3030 30  0001 C CNN
 F 2 "" H 8050 3100 60  0000 C CNN
@@
 PICADC0
 $Comp
-L GND #PWR5
+L GND #PWR026
 U 1 1 53108904
 P 4050 9550
-F 0 "#PWR5" H 4050 9550 30  0001 C CNN
+F 0 "#PWR026" H 4050 9550 30  0001 C CNN
 F 1 "GND" H 4050 9480 30  0001 C CNN
 F 2 "" H 4050 9550 60  0000 C CNN
@@
 	1    0    0    -1
 $EndComp
-Wire Wire Line
-	11100 4100 10950 4100
+$Comp
+L DIODESCH D28
+U 1 1 532F293D
+P 6400 1350
+F 0 "D28" H 6400 1450 40  0000 C CNN
+F 1 "DIODESCH" H 6400 1550 40  0000 C CNN
+F 2 "~" H 6400 1350 60  0000 C CNN
+F 3 "~" H 6400 1350 60  0000 C CNN
+	1    6400 1350
+	1    0    0    -1
+$EndComp
+$Comp
+L DIODESCH D31
+U 1 1 532F294A
+P 6450 2300
+F 0 "D31" H 6450 2400 40  0000 C CNN
+F 1 "DIODESCH" H 6450 2200 40  0000 C CNN
+F 2 "~" H 6450 2300 60  0000 C CNN
+F 3 "~" H 6450 2300 60  0000 C CNN
+	1    6450 2300
+	1    0    0    -1
+$EndComp
+$Comp
+L DIODESCH D30
+U 1 1 532F2950
+P 6450 2000
+F 0 "D30" H 6450 2100 40  0000 C CNN
+F 1 "DIODESCH" H 6450 1900 40  0000 C CNN
+F 2 "~" H 6450 2000 60  0000 C CNN
+F 3 "~" H 6450 2000 60  0000 C CNN
+	1    6450 2000
+	1    0    0    -1
+$EndComp
+$Comp
+L DIODESCH D29
+U 1 1 532F2956
+P 6400 1550
+F 0 "D29" H 6400 1650 40  0000 C CNN
+F 1 "DIODESCH" H 6400 1450 40  0000 C CNN
+F 2 "~" H 6400 1550 60  0000 C CNN
+F 3 "~" H 6400 1550 60  0000 C CNN
+	1    6400 1550
+	1    0    0    -1
+$EndComp
+$Comp
+L FUSE F1
+U 1 1 532F3994
+P 7050 1800
+F 0 "F1" H 7150 1850 40  0000 C CNN
+F 1 "FUSE" H 6950 1750 40  0000 C CNN
+F 2 "~" H 7050 1800 60  0000 C CNN
+F 3 "~" H 7050 1800 60  0000 C CNN
+	1    7050 1800
+	1    0    0    -1
+$EndComp
 Wire Wire Line
 	10950 4100 10950 4000
@@
 	10750 1600 10600 1600
 Connection ~ 10600 1600
-Wire Wire Line
-	10750 1700 10600 1700
 Connection ~ 10600 1700
 Wire Wire Line
@@
 	11450 9550 11450 9000
 Wire Wire Line
-	11450 9000 12750 9000
-Wire Wire Line
-	12750 9000 12750 9150
+	11450 9000 12800 9000
 Wire Wire Line
 	12750 9250 13200 9250
@@
 Wire Wire Line
 	8000 1800 8100 1800
-$Comp
-L DIODESCH D28
-U 1 1 532F293D
-P 6400 1350
-F 0 "D28" H 6400 1450 40  0000 C CNN
-F 1 "DIODESCH" H 6400 1550 40  0000 C CNN
-F 2 "~" H 6400 1350 60  0000 C CNN
-F 3 "~" H 6400 1350 60  0000 C CNN
-	1    6400 1350
-	1    0    0    -1
-$EndComp
-$Comp
-L DIODESCH D31
-U 1 1 532F294A
-P 6450 2300
-F 0 "D31" H 6450 2400 40  0000 C CNN
-F 1 "DIODESCH" H 6450 2200 40  0000 C CNN
-F 2 "~" H 6450 2300 60  0000 C CNN
-F 3 "~" H 6450 2300 60  0000 C CNN
-	1    6450 2300
-	1    0    0    -1
-$EndComp
-$Comp
-L DIODESCH D30
-U 1 1 532F2950
-P 6450 2000
-F 0 "D30" H 6450 2100 40  0000 C CNN
-F 1 "DIODESCH" H 6450 1900 40  0000 C CNN
-F 2 "~" H 6450 2000 60  0000 C CNN
-F 3 "~" H 6450 2000 60  0000 C CNN
-	1    6450 2000
-	1    0    0    -1
-$EndComp
-$Comp
-L DIODESCH D29
-U 1 1 532F2956
-P 6400 1550
-F 0 "D29" H 6400 1650 40  0000 C CNN
-F 1 "DIODESCH" H 6400 1450 40  0000 C CNN
-F 2 "~" H 6400 1550 60  0000 C CNN
-F 3 "~" H 6400 1550 60  0000 C CNN
-	1    6400 1550
-	1    0    0    -1
-$EndComp
 Wire Wire Line
 	6200 1350 6200 1550
@@
 Connection ~ 6600 1450
 Connection ~ 6650 2150
-$Comp
-L FUSE F1
-U 1 1 532F3994
-P 7050 1800
-F 0 "F1" H 7150 1850 40  0000 C CNN
-F 1 "FUSE" H 6950 1750 40  0000 C CNN
-F 2 "~" H 7050 1800 60  0000 C CNN
-F 3 "~" H 7050 1800 60  0000 C CNN
-	1    7050 1800
-	1    0    0    -1
-$EndComp
 Wire Wire Line
 	6800 1800 6750 1800
@@
 Wire Wire Line
 	10750 2000 10600 2000
+Wire Wire Line
+	11100 4100 10950 4100
+$Comp
+L TPS51200 U6
+U 1 1 52E4CA5E
+P 12150 9350
+F 0 "U6" H 12100 8950 60  0000 C CNN
+F 1 "TPS51200" H 12150 9650 60  0000 C CNN
+F 2 "" H 12200 9000 60  0000 C CNN
+F 3 "" H 12200 9000 60  0000 C CNN
+	1    12150 9350
+	1    0    0    -1
+$EndComp
+Wire Wire Line
+	12800 9000 12800 9150
+Connection ~ 12800 9150
+Wire Wire Line
+	10750 1700 10600 1700
 $EndSCHEMATC

Commit message: Issue #993
Parts:
- removed R119, R120, R123, R124, R133, R134, R135, R136, R137, R138, R139, R140: 10K, symbol R
- added D33: LED, ~, symbol LED
- added R328: 2.2K, symbol R
Connections:
- net GND: now also D33.2 (K)
- net VCC12V0_RS-: now also R328.1
- new net: D33.1 (A), R328.2

Commit message: Issue #1022 - Schematics final changes.
Parts:
- R117, R118, R125, R126, R127, R128, R129, R130, R131, R132: value 0.2E 2W -> 0.03E
- R121, R122: value 0.2E 2W -> 0.008E
Connections:
- net VCC12V0_RS- renamed VCC12V0
Changed lines of the file:
@@
 Sheet 8 8
 Title "HDMI2USB"
-Date "3 apr 2014"
+Date "7 apr 2014"
 Rev "V1"
 Comp "Numato Lab"
@@
 	1    0    0    -1
 $EndComp
-Text Label 8100 1800 0    60   ~ 0
+Text Label 8000 1800 0    39   ~ 0
 VCC12V0
 Text Label 5600 2000 0    60   ~ 0
@@
 P 14700 8750
 F 0 "R127" V 14780 8750 50  0000 C CNN
-F 1 "0.2E 2W" V 14700 8750 50  0000 C CNN
+F 1 "0.03E" V 14700 8750 39  0000 C CNN
 F 2 "" H 14700 8750 60  0000 C CNN
 F 3 "" H 14700 8750 60  0000 C CNN
@@
 P 14900 8750
 F 0 "R132" V 14980 8750 50  0000 C CNN
-F 1 "0.2E 2W" V 14900 8750 50  0000 C CNN
+F 1 "0.03E" V 14900 8750 39  0000 C CNN
 F 2 "" H 14900 8750 60  0000 C CNN
 F 3 "" H 14900 8750 60  0000 C CNN
@@
 P 5850 8000
 F 0 "R117" V 5930 8000 50  0000 C CNN
-F 1 "0.2E 2W" V 5850 8000 50  0000 C CNN
+F 1 "0.03E" V 5850 8000 39  0000 C CNN
 F 2 "" H 5850 8000 60  0000 C CNN
 F 3 "" H 5850 8000 60  0000 C CNN
@@
 P 5850 8200
 F 0 "R118" V 5930 8200 50  0000 C CNN
-F 1 "0.2E 2W" V 5850 8200 50  0000 C CNN
+F 1 "0.03E" V 5850 8200 39  0000 C CNN
 F 2 "" H 5850 8200 60  0000 C CNN
 F 3 "" H 5850 8200 60  0000 C CNN
@@
 P 7700 1700
 F 0 "R121" V 7780 1700 50  0000 C CNN
-F 1 "0.2E 2W" V 7700 1700 50  0000 C CNN
+F 1 "0.008E" V 7700 1700 39  0000 C CNN
 F 2 "" H 7700 1700 60  0000 C CNN
 F 3 "" H 7700 1700 60  0000 C CNN
@@
 P 7700 1900
 F 0 "R122" V 7780 1900 50  0000 C CNN
-F 1 "0.2E 2W" V 7700 1900 50  0000 C CNN
+F 1 "0.008E" V 7700 1900 39  0000 C CNN
 F 2 "" H 7700 1900 60  0000 C CNN
 F 3 "" H 7700 1900 60  0000 C CNN
@@
 P 14850 6050
 F 0 "R130" V 14930 6050 50  0000 C CNN
-F 1 "0.2E 2W" V 14850 6050 50  0000 C CNN
+F 1 "0.03E" V 14850 6050 39  0000 C CNN
 F 2 "" H 14850 6050 60  0000 C CNN
 F 3 "" H 14850 6050 60  0000 C CNN
@@
 P 14850 6250
 F 0 "R131" V 14930 6250 50  0000 C CNN
-F 1 "0.2E 2W" V 14850 6250 50  0000 C CNN
+F 1 "0.03E" V 14850 6250 39  0000 C CNN
 F 2 "" H 14850 6250 60  0000 C CNN
 F 3 "" H 14850 6250 60  0000 C CNN
@@
 P 14750 1650
 F 0 "R128" V 14830 1650 50  0000 C CNN
-F 1 "0.2E 2W" V 14750 1650 50  0000 C CNN
+F 1 "0.03E" V 14750 1650 39  0000 C CNN
 F 2 "" H 14750 1650 60  0000 C CNN
 F 3 "" H 14750 1650 60  0000 C CNN
@@
 P 14750 1850
 F 0 "R129" V 14830 1850 50  0000 C CNN
-F 1 "0.2E 2W" V 14750 1850 50  0000 C CNN
+F 1 "0.03E" V 14750 1850 39  0000 C CNN
 F 2 "" H 14750 1850 60  0000 C CNN
 F 3 "" H 14750 1850 60  0000 C CNN
@@
 P 14600 3800
 F 0 "R125" V 14680 3800 50  0000 C CNN
-F 1 "0.2E 2W" V 14600 3800 50  0000 C CNN
+F 1 "0.03E" V 14600 3800 39  0000 C CNN
 F 2 "" H 14600 3800 60  0000 C CNN
 F 3 "" H 14600 3800 60  0000 C CNN
@@
 P 14600 4000
 F 0 "R126" V 14680 4000 50  0000 C CNN
-F 1 "0.2E 2W" V 14600 4000 50  0000 C CNN
+F 1 "0.03E" V 14600 4000 39  0000 C CNN
 F 2 "" H 14600 4000 60  0000 C CNN
 F 3 "" H 14600 4000 60  0000 C CNN
@@
 Connection ~ 1550 2100
 Wire Wire Line
-	8000 1800 8100 1800
+	8000 1800 8250 1800
 Wire Wire Line
 	6200 1350 6200 1550
@@
 Text Notes 800  3400 0    79   ~ 16
 Conference Model
+Text GLabel 8250 1800 2    39   Output ~ 0
+VCC12V0
 $EndSCHEMATC
