File: board/HDMI2USB.kicad_pcb (KiCad board)
At the start: 10 copper layers, 170 x 170 mm, 460 parts, among them CON1 BARREL_JACK, CON2 BARREL_JACK, J1 USB_MICRO_B, J2 HDMI, J3 HDMI, J4 HDMI, J5 HDMI, J6 RJ45(HFJ11-1GO1ERL), J7 USB_MICRO_B, J8 DISPLAY_PORT, J9 DISPLAY_PORT, P1 CONN_2, P10 CONN_1, P11 CONN_1, P12 CONN_1, P13 CONN_1, P2 CONN_1, P3 CONN_7X2, P4 CONN_1, P5 CONN_1, P6 CONN_1, P7 CONN_1, P8 CONN_1, P9 CONN_1, SW1 SW_PUSH, U1 MT41J128M16, U10 XC6SLX150T, U11 MICRO_SD, U12 TPS51200, U13 IP4776CZ38, U14 IP4776CZ38, U15 IP4776CZ38, U16 ΜA78L00, U17 FXO-HC536R, U18 USB3340, U19 MCP1825, U2 CY7C68013A_100AC, U20 RTL8211E-VB, U21 IP4776CZ38, U22 ΜA78L00, U23 24AA02E48, U3 W25Q128FVEIG, U4 GBU15005-G, U5 7805, U6 TPS54560, U7 TPS53319, U8 TPS54625, U9 TPS54625, X1 CRYSTAL, X2 50MHz

Commit message: Issue #1412 - Placement
Parts:
- C62: footprint SM1210L -> SM0603
- C64: footprint SM0805 -> SM0603
- R30: value 20K -> 20K5%- 0.05W
- moved R14 197.5 mm to (198.7, 213.2), turned to 270 degrees
- moved R15 196.3 mm to (200.4, 213.2), turned to 270 degrees
- moved R23 195.0 mm to (202.2, 213.2), turned to 270 degrees
- moved R24 193.7 mm to (204.0, 213.2), turned to 270 degrees
- moved R26 192.5 mm to (205.8, 213.2), turned to 270 degrees
- moved R31 191.2 mm to (207.5, 213.2), turned to 270 degrees
- moved R27 190.0 mm to (209.3, 213.2), turned to 270 degrees
- moved R28 188.8 mm to (211.1, 213.2), turned to 270 degrees
- moved C62 188.5 mm to (223.8, 198.6)
- moved C64 173.2 mm to (223.8, 203.7), turned to 0 degrees
- moved R32 170.6 mm to (217.2, 193.6), turned to 0 degrees
- moved R37 169.4 mm to (217.2, 191.8), turned to 0 degrees
- moved J7 168.5 mm to (212.6, 228.8), turned to 0 degrees
- moved R34 168.2 mm to (217.2, 190.1), turned to 0 degrees
- moved R33 167.0 mm to (217.2, 188.3), turned to 0 degrees
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Connections:
- net /DDR3/DDR0_ZQ renamed N-00000174
- C173 pad 1: VCC5V0 -> VCC12V0
- C177 pad 1: VCC5V0 -> VCC12V0
- C38 pad 1: N-00000364 -> VCC12V0
- J1 pad 1: N-00000348 -> /USB/USB_5V
- J9 pad 17: (no net) -> /DisplayPort/RXAUXCH_N
- JP1 pad 1: /SPI_Flash/FPGA_M0_CMP_MISO -> /FPGA_Bank_1_2/FPGA_M0_CMP_MISO
- JP2 pad 1: /SPI_Flash/FPGA_M1 -> /FPGA_Bank_1_2/FPGA_M1
- R14 pad 2: /FPGA_Power/TDO_FPGA/TDO-JTAG -> /SPI_Flash/TDO-FPGA/TDO-JTAG
- R23 pad 2: /USB/TDO-USB/TDI-FPGA -> /SPI_Flash/TDO-USB/TDI-FPGA
- R27 pad 2: /FPGA_Power/INIT_B -> /FPGA_Bank_1_2/INIT_B
- R30 pad 2: N-00000364 -> /USB/USB_5V
- R37 pad 1: N-00000363 -> N-00000348
- R40 pad 2: /SPI_Flash/FPGA_M0_CMP_MISO -> /FPGA_Bank_1_2/FPGA_M0_CMP_MISO
- R41 pad 1: /SPI_Flash/FPGA_M1 -> /FPGA_Bank_1_2/FPGA_M1
- R52 pad 2: /FPGA_Power/INIT_B -> /FPGA_Bank_1_2/INIT_B
- R53 pad 1: (no net) -> /FPGA_Bank_0_3/HSWAP
- R76 pad 2: (no net) -> /FPGA_Power/TMS
- R81 pad 2: (no net) -> /FPGA_Power/TCK
- R82 pad 2: (no net) -> /SPI_Flash/TDO-FPGA/TDO-JTAG
- R83 pad 2: (no net) -> /SPI_Flash/TDO-USB/TDI-FPGA
- R86 pad 1: (no net) -> /Ethernet/ETH_FPGA_CLK
- U10 pad AA12: (no net) -> /Ethernet/ETH_RXCLK
- U10 pad AA21: (no net) -> /FPGA_Bank_1_2/FPGA_M0_CMP_MISO
- U10 pad AB12: (no net) -> /Ethernet/ETH_TXCLK
- U10 pad B21: (no net) -> /FPGA_Bank_1_2/CY_PA4
- U10 pad B22: (no net) -> /FPGA_Bank_1_2/CY_PA5
- U10 pad C20: (no net) -> /FPGA_Bank_1_2/CY_FD0
- U10 pad C22: (no net) -> /FPGA_Bank_1_2/CY_FD1
- U10 pad C3: (no net) -> /FPGA_Bank_0_3/HSWAP
- U10 pad D19: (no net) -> /DisplayPort/RXAUXCH_N
- U10 pad D21: (no net) -> /FPGA_Bank_1_2/CY_FD4
- U10 pad D22: (no net) -> /FPGA_Bank_1_2/CY_FD5
- U10 pad E18: /USB/TDO-USB/TDI-FPGA -> /SPI_Flash/TDO-USB/TDI-FPGA
- U10 pad E20: (no net) -> /FPGA_Bank_1_2/CY_FD12
- U10 pad E22: (no net) -> /FPGA_Bank_1_2/CY_FD13
- U10 pad F18: (no net) -> /FPGA_Bank_1_2/CY_PA0
- U10 pad F19: (no net) -> /FPGA_Bank_1_2/CY_PA1
- U10 pad F20: (no net) -> /FPGA_Bank_1_2/CY_FD7
- U10 pad F21: (no net) -> /FPGA_Bank_1_2/CY_FD10
- U10 pad F22: (no net) -> /FPGA_Bank_1_2/CY_FD11
- U10 pad G17: /FPGA_Power/TDO_FPGA/TDO-JTAG -> /SPI_Flash/TDO-FPGA/TDO-JTAG
- U10 pad G19: (no net) -> /FPGA_Bank_1_2/CY_FD6
- U10 pad G20: (no net) -> /FPGA_Bank_1_2/CY_T0
- U10 pad G22: (no net) -> /FPGA_Bank_1_2/CYPRESS-RESET
- U10 pad H16: (no net) -> /FPGA_Bank_1_2/CY_PA2
- U10 pad H17: (no net) -> /FPGA_Bank_1_2/CY_PA3
- U10 pad H18: (no net) -> /FPGA_Bank_1_2/CY_FD8
- U10 pad H19: (no net) -> /FPGA_Bank_1_2/CY_FD9
- U10 pad H20: (no net) -> /FPGA_Bank_1_2/CY_FD15
- U10 pad J16: (no net) -> /FPGA_Bank_1_2/CY_PA6
- U10 pad J17: (no net) -> /FPGA_Bank_1_2/CY_PA7
- U10 pad J19: (no net) -> /FPGA_Bank_1_2/CY_FD14
- U10 pad K16: (no net) -> /FPGA_Bank_1_2/CY_FD3
- U10 pad K18: (no net) -> /FPGA_Bank_1_2/CY_WR
- U10 pad K19: (no net) -> /FPGA_Bank_1_2/CY_RD
- U10 pad L15: (no net) -> /FPGA_Bank_1_2/CY_FD2
- U10 pad M16: (no net) -> /FPGA_Bank_1_2/CY_RD2
- U10 pad M17: (no net) -> /FPGA_Bank_1_2/CY_CTL2
- U10 pad M18: (no net) -> /FPGA_Bank_1_2/CY_CTL3
- U10 pad N15: (no net) -> /FPGA_Bank_1_2/CY_RD3
- U10 pad N16: (no net) -> /FPGA_Bank_1_2/CY_CTL0
- U10 pad P16: (no net) -> /FPGA_Bank_1_2/CY_CTL1
- U10 pad P17: (no net) -> /FPGA_Bank_1_2/CY_RXD0
- U10 pad P18: (no net) -> /FPGA_Bank_1_2/CY_RXD1
- U10 pad P19: (no net) -> /FPGA_Bank_1_2/CY_RD0
- U10 pad P20: (no net) -> /FPGA_Bank_1_2/CY-IFCLK
- U10 pad R15: (no net) -> /FPGA_Bank_1_2/CY_CTL4
- U10 pad R16: (no net) -> /FPGA_Bank_1_2/CY_CTL5
- U10 pad R17: (no net) -> /FPGA_Bank_1_2/CY_TXD0
- U10 pad R19: (no net) -> /FPGA_Bank_1_2/CY_RD1
- U10 pad T17: (no net) -> /FPGA_Bank_1_2/CY_TXD1
- U10 pad T19: (no net) -> /FPGA_Bank_1_2/CY_INT5
- U10 pad T20: (no net) -> /FPGA_Bank_1_2/CY_RD5
- U10 pad U10: (no net) -> /Ethernet/MAC_SCL
- U10 pad U19: (no net) -> /FPGA_Bank_1_2/CY_RD4
- U10 pad U20: (no net) -> /FPGA_Bank_1_2/CY_PC0
- U10 pad U22: (no net) -> /FPGA_Bank_1_2/CY_PC1
- U10 pad V21: (no net) -> /FPGA_Bank_1_2/CY_PC2
- U10 pad V22: (no net) -> /FPGA_Bank_1_2/CY_PC3
- U10 pad W20: (no net) -> /FPGA_Bank_1_2/CY_PC4
- U10 pad W22: (no net) -> /FPGA_Bank_1_2/CY_PC5
- U10 pad Y13: (no net) -> /Ethernet/ETH_FPGA_CLK
- U10 pad Y19: (no net) -> /FPGA_Bank_1_2/FPGA_M1
- U10 pad Y21: (no net) -> /FPGA_Bank_1_2/CY_PC6
- U10 pad Y22: (no net) -> /FPGA_Bank_1_2/CY_PC7
- U10 pad Y4: (no net) -> /FPGA_Bank_1_2/INIT_B
- U16 pad 3: VCC5V0 -> VCC12V0
- U18 pad 17: VCC5V0 -> /USB/CPEN
- U2 pad 23: (no net) -> /FPGA_Bank_1_2/CY_T0
- U2 pad 26: (no net) -> /FPGA_Bank_1_2/CY-IFCLK
- U2 pad 27: N-00000363 -> N-00000348
- U2 pad 3: (no net) -> /FPGA_Bank_1_2/CY_RD0
- U2 pad 31: (no net) -> /FPGA_Bank_1_2/CY_RD
- U2 pad 32: (no net) -> /FPGA_Bank_1_2/CY_WR
- U2 pad 34: (no net) -> /FPGA_Bank_1_2/CY_FD0
- U2 pad 35: (no net) -> /FPGA_Bank_1_2/CY_FD1
- U2 pad 36: (no net) -> /FPGA_Bank_1_2/CY_FD2
- U2 pad 37: (no net) -> /FPGA_Bank_1_2/CY_FD3
- U2 pad 4: (no net) -> /FPGA_Bank_1_2/CY_RD1
- U2 pad 40: (no net) -> /FPGA_Bank_1_2/CY_TXD1
- U2 pad 41: (no net) -> /FPGA_Bank_1_2/CY_RXD1
- U2 pad 42: (no net) -> /FPGA_Bank_1_2/CY_TXD0
- U2 pad 43: (no net) -> /FPGA_Bank_1_2/CY_RXD0
- U2 pad 44: (no net) -> /FPGA_Bank_1_2/CY_FD4
- U2 pad 45: (no net) -> /FPGA_Bank_1_2/CY_FD5
- U2 pad 46: (no net) -> /FPGA_Bank_1_2/CY_FD6
- U2 pad 47: (no net) -> /FPGA_Bank_1_2/CY_FD7
- U2 pad 5: (no net) -> /FPGA_Bank_1_2/CY_RD2
- U2 pad 51: (no net) -> /FPGA_Bank_1_2/CY_CTL3
- U2 pad 52: (no net) -> /FPGA_Bank_1_2/CY_CTL4
- U2 pad 54: (no net) -> /FPGA_Bank_1_2/CY_CTL0
- U2 pad 55: (no net) -> /FPGA_Bank_1_2/CY_CTL1
- U2 pad 56: (no net) -> /FPGA_Bank_1_2/CY_CTL2
- U2 pad 57: (no net) -> /FPGA_Bank_1_2/CY_PC0
- U2 pad 58: (no net) -> /FPGA_Bank_1_2/CY_PC1
- U2 pad 59: (no net) -> /FPGA_Bank_1_2/CY_PC2
- U2 pad 6: (no net) -> /FPGA_Bank_1_2/CY_RD3
- U2 pad 60: (no net) -> /FPGA_Bank_1_2/CY_PC3
- U2 pad 61: (no net) -> /FPGA_Bank_1_2/CY_PC4
- U2 pad 62: (no net) -> /FPGA_Bank_1_2/CY_PC5
- U2 pad 63: (no net) -> /FPGA_Bank_1_2/CY_PC6
- U2 pad 64: (no net) -> /FPGA_Bank_1_2/CY_PC7
- U2 pad 67: (no net) -> /FPGA_Bank_1_2/CY_PA0
- U2 pad 68: (no net) -> /FPGA_Bank_1_2/CY_PA1
- U2 pad 69: (no net) -> /FPGA_Bank_1_2/CY_PA2
- U2 pad 7: (no net) -> /FPGA_Bank_1_2/CY_RD4
- U2 pad 70: (no net) -> /FPGA_Bank_1_2/CY_PA3
- U2 pad 71: (no net) -> /FPGA_Bank_1_2/CY_PA4
- U2 pad 72: (no net) -> /FPGA_Bank_1_2/CY_PA5
- U2 pad 73: (no net) -> /FPGA_Bank_1_2/CY_PA6
- U2 pad 74: (no net) -> /FPGA_Bank_1_2/CY_PA7
- U2 pad 76: (no net) -> /FPGA_Bank_1_2/CY_CTL5
- U2 pad 77: (no net) -> /FPGA_Bank_1_2/CYPRESS-RESET
- U2 pad 8: (no net) -> /FPGA_Bank_1_2/CY_RD5
- U2 pad 80: (no net) -> /FPGA_Bank_1_2/CY_FD8
- U2 pad 81: (no net) -> /FPGA_Bank_1_2/CY_FD9
- U2 pad 82: (no net) -> /FPGA_Bank_1_2/CY_FD10
- U2 pad 83: (no net) -> /FPGA_Bank_1_2/CY_FD11
- U2 pad 84: (no net) -> /FPGA_Bank_1_2/CY_INT5
- U2 pad 95: (no net) -> /FPGA_Bank_1_2/CY_FD12
- U2 pad 96: (no net) -> /FPGA_Bank_1_2/CY_FD13
- U2 pad 97: (no net) -> /FPGA_Bank_1_2/CY_FD14
- U2 pad 98: (no net) -> /FPGA_Bank_1_2/CY_FD15
- U20 pad 22: (no net) -> /Ethernet/ETH_TXCLK
- U22 pad 3: VCC5V0 -> VCC12V0
Routing:
- net (no net): track 819.2 -> 563.1 mm, vias 96 -> 63
- net /FPGA_Bank_1_2/CY_PA0: track 0.00 -> 59.2 mm, vias 0 -> 2
- net /FPGA_Bank_1_2/CY_CTL5: track 0.00 -> 44.4 mm, vias 0 -> 2
- net /FPGA_Bank_1_2/CY_FD8: track 0.00 -> 43.0 mm, vias 0 -> 2
- net /FPGA_Bank_1_2/CY_PA2: track 0.00 -> 41.7 mm, vias 0 -> 2
- net /FPGA_Bank_1_2/CY_FD9: track 0.00 -> 40.8 mm, vias 0 -> 2
- net /FPGA_Bank_1_2/CY_PA6: track 0.00 -> 40.8 mm, vias 0 -> 2
- net /FPGA_Bank_1_2/CY_PA7: track 0.00 -> 40.7 mm, vias 0 -> 2
- net /FPGA_Bank_1_2/CY_PA1: track 0.00 -> 40.6 mm, vias 0 -> 2
- net /FPGA_Bank_1_2/CY_FD10: track 0.00 -> 38.5 mm, vias 0 -> 2
- net /FPGA_Bank_1_2/CYPRESS-RESET: track 0.00 -> 37.6 mm, vias 0 -> 1
- net /FPGA_Bank_1_2/CY_PA3: track 0.00 -> 37.6 mm, vias 0 -> 2
- net /FPGA_Bank_1_2/CY_FD11: track 0.00 -> 37.5 mm, vias 0 -> 2
- net /FPGA_Bank_1_2/CY_PA4: track 0.00 -> 36.8 mm, vias 0 -> 1
- net /FPGA_Bank_1_2/CY_PA5: track 0.00 -> 36.2 mm, vias 0 -> 1
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- added copper zone on F.Cu, net N-00000391
- added copper zone on F.Cu, net N-00000398
- added copper zone on F.Cu, net N-00000401
- added copper zone on F.Cu, net N-00000413
- removed copper zone on F.Cu, net N-00000370
- removed copper zone on F.Cu, net N-00000403
- removed copper zone on F.Cu, net N-00000408
- removed copper zone on F.Cu, net N-00000409
Other:
- board size 170 x 170 mm -> 205 x 170 mm

Commit message: Issue #1608 - Placement
Parts:
- R76: footprint SM0402 -> SM0603
- U11: moved to F.Cu
- moved C134 190.5 mm to (89.9, 128.0)
- moved C139 190.5 mm to (93.7, 128.0)
- moved C140 190.5 mm to (93.7, 128.0)
- moved C141 190.5 mm to (85.3, 121.2)
- moved C144 190.5 mm to (79.5, 121.4)
- moved C145 190.5 mm to (89.9, 128.0)
- moved C152 190.5 mm to (85.6, 134.1)
- moved C158 190.5 mm to (84.8, 119.6)
- moved C164 190.5 mm to (75.7, 127.3)
- moved C167 190.5 mm to (75.7, 127.3)
- moved C80 190.5 mm to (88.6, 133.3)
- moved R103 190.5 mm to (80.3, 121.4)
- moved R104 190.5 mm to (82.5, 120.4)
- moved R114 190.5 mm to (83.1, 119.6)
- moved U9 190.5 mm to (83.8, 126.5)
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Connections:
- U10 pad AA4: /FPGA_Bank_1_2/SD_DAT2 -> /FPGA_Bank_1_2/SD_DAT3
- U10 pad AB4: /FPGA_Bank_1_2/SD_DAT3 -> /FPGA_Bank_1_2/SD_DAT2
- U10 pad M17: /FPGA_Bank_1_2/CY_CTL2 -> /FPGA_Bank_1_2/CY_CTL4
- U10 pad R15: /FPGA_Bank_1_2/CY_CTL4 -> /FPGA_Bank_1_2/CY_CTL2
Routing:
- net /Ethernet/ETH_RXCLK: track 0.66 -> 129.5 mm, vias 1 -> 2
- net (no net): track 563.1 -> 434.3 mm
- net /FPGA_Bank_1_2/SD_DAT3: track 14.7 -> 123.1 mm
- net /FPGA_Bank_1_2/SD_DAT0: track 18.6 -> 125.4 mm
- net /FPGA_Bank_1_2/SD_DAT2: track 15.9 -> 122.5 mm
- net /FPGA_Bank_1_2/SD_DAT1: track 15.8 -> 122.2 mm
- net /FPGA_Bank_1_2/SD_CMD: track 23.1 -> 129.0 mm
- net /FPGA_Bank_1_2/SD_CLK: track 20.7 -> 126.6 mm
- net /FPGA_Bank_1_2/CY_RD3: track 0.88 -> 86.8 mm, vias 1 -> 2
- net /FPGA_Bank_1_2/CY_RD2: track 1.58 -> 85.1 mm
- net /FPGA_Bank_1_2/CY_RD0: track 0.88 -> 77.4 mm, vias 1 -> 2
- net /FPGA_Bank_1_2/CY_RD1: track 1.60 -> 70.4 mm
- net /FPGA_Bank_1_2/CY_RD4: track 0.88 -> 69.0 mm, vias 1 -> 2
- net /FPGA_Bank_1_2/CY_RD5: track 0.88 -> 68.5 mm, vias 1 -> 2
- net /SPI_Flash/TDO-FPGA/TDO-JTAG: track 19.0 -> 77.7 mm, vias 1 -> 2
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Other:
- board size 205 x 170 mm -> 215 x 155 mm
