File: board/DDR3.sch (KiCad schematic (older format))
At the start: 56 parts, among them U1 MT41J128M16

Commit message: Issue #1670
Other:
- note added: "DDR3"
Changed lines of the file:
@@
 Sheet 5 12
 Title "HDMI2USB"
-Date "25 mar 2015"
+Date "30 mar 2015"
 Rev "Rev2"
 Comp ""
@@
 Wire Wire Line
 	2000 9500 5050 9500
+Text Notes 10550 800  0    118  ~ 24
+DDR3
 $EndSCHEMATC

Commit message: Issue #1585
Parts:
- R12: value R -> 240R
Changed lines of the file:
@@
 LIBS:contrib
 LIBS:valves
-LIBS:hdmi2usb
-LIBS:timvideos-pcie-8x
 LIBS:HDMI2USB-cache
 EELAYER 27 0
@@
 Sheet 5 12
 Title "HDMI2USB"
-Date "30 mar 2015"
+Date "1 apr 2015"
 Rev "Rev2"
 Comp ""
@@
 $EndComp
 $Comp
-L GND #PWR31
+L GND #PWR032
 U 1 1 52D6229F
 P 11850 5300
-F 0 "#PWR31" H 11850 5300 30  0001 C CNN
+F 0 "#PWR032" H 11850 5300 30  0001 C CNN
 F 1 "GND" H 11850 5230 30  0001 C CNN
 F 2 "" H 11850 5300 60  0000 C CNN
@@
 $EndComp
 $Comp
-L GND #PWR32
+L GND #PWR033
 U 1 1 52D622F7
 P 11850 6350
-F 0 "#PWR32" H 11850 6350 30  0001 C CNN
+F 0 "#PWR033" H 11850 6350 30  0001 C CNN
 F 1 "GND" H 11850 6280 30  0001 C CNN
 F 2 "" H 11850 6350 60  0000 C CNN
@@
 P 12250 1300
 F 0 "R12" V 12330 1300 50  0000 C CNN
-F 1 "R" V 12250 1300 50  0000 C CNN
+F 1 "240R" V 12250 1300 50  0000 C CNN
 F 2 "" H 12250 1300 60  0000 C CNN
 F 3 "" H 12250 1300 60  0000 C CNN
@@
 $EndComp
 $Comp
-L GND #PWR34
+L GND #PWR034
 U 1 1 52D66B0B
 P 12500 1400
-F 0 "#PWR34" H 12500 1400 30  0001 C CNN
+F 0 "#PWR034" H 12500 1400 30  0001 C CNN
 F 1 "GND" H 12500 1330 30  0001 C CNN
 F 2 "" H 12500 1400 60  0000 C CNN
@@
 $EndComp
 $Comp
-L GND #PWR33
+L GND #PWR035
 U 1 1 52D66E65
 P 12100 4100
-F 0 "#PWR33" H 12100 4100 30  0001 C CNN
+F 0 "#PWR035" H 12100 4100 30  0001 C CNN
 F 1 "GND" H 12100 4030 30  0001 C CNN
 F 2 "" H 12100 4100 60  0000 C CNN
@@
 $EndComp
 $Comp
-L GND #PWR29
+L GND #PWR036
 U 1 1 52D6755F
 P 7450 5650
-F 0 "#PWR29" H 7450 5650 30  0001 C CNN
+F 0 "#PWR036" H 7450 5650 30  0001 C CNN
 F 1 "GND" H 7450 5580 30  0001 C CNN
 F 2 "" H 7450 5650 60  0000 C CNN
@@
 $EndComp
 $Comp
-L GND #PWR30
+L GND #PWR037
 U 1 1 52D69B15
 P 8450 8650
-F 0 "#PWR30" H 8450 8650 30  0001 C CNN
+F 0 "#PWR037" H 8450 8650 30  0001 C CNN
 F 1 "GND" H 8450 8580 30  0001 C CNN
 F 2 "" H 8450 8650 60  0000 C CNN
@@
 	5050 9500 5050 9600
 $Comp
-L GND #PWR28
+L GND #PWR038
 U 1 1 52E83C38
 P 5050 9600
-F 0 "#PWR28" H 5050 9600 30  0001 C CNN
+F 0 "#PWR038" H 5050 9600 30  0001 C CNN
 F 1 "GND" H 5050 9530 30  0001 C CNN
 F 2 "" H 5050 9600 60  0000 C CNN
