File: board/Ethernet.sch (KiCad schematic (older format))
At the start: 55 parts, among them J6 RJ45(HFJ11-1GO1ERL), U19 MCP1825, U20 RTL8211E-VB, U23 24AA02E48, X2 50MHz

Commit message: Issue #1683
Parts:
- removed R86: 0R, ~, symbol R
- added K1: CONN_3, symbol CONN_3
Connections:
- net GND: now also K1.3 (P3); no longer U23.3 (A2)
- net VCC3V3: now also K1.1 (P1)
- new net: K1.2 (PM), U23.3 (A2)
Changed lines of the file:
@@
 Sheet 8 12
 Title "HDMI2USB"
-Date "23 mar 2015"
+Date "25 mar 2015"
 Rev "Rev2"
 Comp "Numato Lab"
@@
 Text Label 7200 1700 0    47   ~ 0
 ETH_VCC3V3
-Text Label 11850 8200 2    39   ~ 0
-FPGA_CLK
-$Comp
-L R R86
-U 1 1 54980368
-P 11300 8200
-F 0 "R86" V 11380 8200 40  0000 C CNN
-F 1 "0R" V 11307 8201 40  0000 C CNN
-F 2 "~" V 11230 8200 30  0000 C CNN
-F 3 "~" H 11300 8200 30  0000 C CNN
-	1    11300 8200
-	0    1    1    0
-$EndComp
 Entry Wire Line
 	6350 3900 6450 4000
@@
 	14350 8550 14600 8550
 Connection ~ 13650 7950
-Connection ~ 12850 8550
-Wire Wire Line
-	12950 8550 12850 8550
 Wire Wire Line
 	12950 8450 12850 8450
 Wire Wire Line
-	12850 8450 12850 9150
-Wire Wire Line
-	12950 8650 12850 8650
-Connection ~ 12850 8650
+	12600 8650 12950 8650
 Wire Wire Line
 	15000 8350 15000 8400
@@
 Connection ~ 3800 8400
 Wire Wire Line
-	12850 9150 13650 9150
-Wire Wire Line
 	13650 7950 13650 8150
 Connection ~ 3800 9600
@@
 	5500 1800 5500 1850
 Connection ~ 5500 1850
-Wire Wire Line
-	11850 8200 11550 8200
 Wire Wire Line
 	7650 1700 7650 2350
@@
 Text HLabel 5750 5200 0    47   Input ~ 0
 ETH_RESET_B
-Text HLabel 11850 8200 2    47   Input ~ 0
-ETH_FPGA_CLK
 Text HLabel 5700 4800 0    47   Input ~ 0
 ETH_MDC
@@
 NoConn ~ 10750 4600
 NoConn ~ 6800 5750
+Wire Wire Line
+	12950 8550 12600 8550
+Wire Wire Line
+	12850 8450 12850 8550
+Connection ~ 12850 8550
+Text Label 12600 8550 0    60   ~ 0
+GND
+$Comp
+L CONN_3 K1
+U 1 1 55123FA6
+P 12250 8650
+F 0 "K1" V 12200 8650 50  0000 C CNN
+F 1 "CONN_3" V 12300 8650 40  0000 C CNN
+F 2 "" H 12250 8650 60  0000 C CNN
+F 3 "" H 12250 8650 60  0000 C CNN
+	1    12250 8650
+	-1   0    0    1
+$EndComp
+Text Label 12900 8750 2    47   ~ 0
+VCC3V3
+Wire Wire Line
+	12600 8750 12900 8750
 $EndSCHEMATC

Commit message: Issue #1585
Other:
- note added: "JUSBPROM"
Changed lines of the file:
@@
 LIBS:contrib
 LIBS:valves
-LIBS:hdmi2usb
-LIBS:timvideos-pcie-8x
 LIBS:HDMI2USB-cache
 EELAYER 27 0
@@
 Sheet 8 12
 Title "HDMI2USB"
-Date "30 mar 2015"
+Date "1 apr 2015"
 Rev "Rev2"
 Comp "Numato Lab"
@@
 MAC_SCL
 $Comp
-L GND #PWR37
+L GND #PWR039
 U 1 1 53CC9E90
 P 14600 8600
-F 0 "#PWR37" H 14600 8600 30  0001 C CNN
+F 0 "#PWR039" H 14600 8600 30  0001 C CNN
 F 1 "GND" H 14600 8530 30  0001 C CNN
 F 2 "" H 14600 8600 60  0001 C CNN
@@
 $EndComp
 $Comp
-L GND #PWR38
+L GND #PWR040
 U 1 1 53CC9E9C
 P 15000 8400
-F 0 "#PWR38" H 15000 8400 30  0001 C CNN
+F 0 "#PWR040" H 15000 8400 30  0001 C CNN
 F 1 "GND" H 15000 8330 30  0001 C CNN
 F 2 "" H 15000 8400 60  0001 C CNN
@@
 $EndComp
 $Comp
-L GND #PWR36
+L GND #PWR041
 U 1 1 53CC9EA2
 P 13650 9300
-F 0 "#PWR36" H 13650 9300 30  0001 C CNN
+F 0 "#PWR041" H 13650 9300 30  0001 C CNN
 F 1 "GND" H 13650 9230 30  0001 C CNN
 F 2 "" H 13650 9300 60  0001 C CNN
@@
 $EndComp
 $Comp
-L GND #PWR35
+L GND #PWR042
 U 1 1 54772306
 P 3500 9650
-F 0 "#PWR35" H 3500 9650 30  0001 C CNN
+F 0 "#PWR042" H 3500 9650 30  0001 C CNN
 F 1 "GND" H 3500 9580 30  0001 C CNN
 F 2 "" H 3500 9650 60  0001 C CNN
@@
 Wire Wire Line
 	12600 8750 12900 8750
+Text Notes 13200 8300 0    39   ~ 0
+JUSBPROM
 $EndSCHEMATC

Commit message: Issue #1713
Parts:
- removed R72: 0R, ~, symbol R
Changed lines of the file:
@@
 Sheet 8 12
 Title "HDMI2USB"
-Date "2 apr 2015"
+Date "7 apr 2015"
 Rev "Rev2"
 Comp "Numato Lab"
@@
 MAC_SCL
 $Comp
-L GND #PWR039
+L GND #PWR040
 U 1 1 53CC9E90
 P 14600 8600
-F 0 "#PWR039" H 14600 8600 30  0001 C CNN
+F 0 "#PWR040" H 14600 8600 30  0001 C CNN
 F 1 "GND" H 14600 8530 30  0001 C CNN
 F 2 "" H 14600 8600 60  0001 C CNN
@@
 $EndComp
 $Comp
-L GND #PWR040
+L GND #PWR041
 U 1 1 53CC9E9C
 P 15000 8400
-F 0 "#PWR040" H 15000 8400 30  0001 C CNN
+F 0 "#PWR041" H 15000 8400 30  0001 C CNN
 F 1 "GND" H 15000 8330 30  0001 C CNN
 F 2 "" H 15000 8400 60  0001 C CNN
@@
 $EndComp
 $Comp
-L GND #PWR041
+L GND #PWR042
 U 1 1 53CC9EA2
 P 13650 9300
-F 0 "#PWR041" H 13650 9300 30  0001 C CNN
+F 0 "#PWR042" H 13650 9300 30  0001 C CNN
 F 1 "GND" H 13650 9230 30  0001 C CNN
 F 2 "" H 13650 9300 60  0001 C CNN
@@
 XTAL2_50MHZ
 $Comp
-L R R72
-U 1 1 5477065F
-P 9600 8700
-F 0 "R72" V 9680 8700 40  0000 C CNN
-F 1 "0R" V 9607 8701 40  0000 C CNN
-F 2 "~" V 9530 8700 30  0000 C CNN
-F 3 "~" H 9600 8700 30  0000 C CNN
-	1    9600 8700
-	-1   0    0    1
-$EndComp
-$Comp
 L MCP1825 U19
 U 1 1 547713E1
@@
 $EndComp
 $Comp
-L GND #PWR042
+L GND #PWR043
 U 1 1 54772306
 P 3500 9650
-F 0 "#PWR042" H 3500 9650 30  0001 C CNN
+F 0 "#PWR043" H 3500 9650 30  0001 C CNN
 F 1 "GND" H 3500 9580 30  0001 C CNN
 F 2 "" H 3500 9650 60  0001 C CNN
@@
 Wire Wire Line
 	6050 5850 5850 5850
-Wire Wire Line
-	9600 8450 9600 8200
-Wire Wire Line
-	9600 8950 9600 9150
-Wire Wire Line
-	9600 9150 10950 9150
-Connection ~ 9900 9150
-Connection ~ 9600 8200
 Wire Wire Line
 	2550 9000 2550 8800
@@
 Text Notes 13200 8300 0    39   ~ 0
 JUSBPROM
+Text GLabel 13350 7950 0    39   Input ~ 0
+VCC3V3
+Wire Wire Line
+	9900 9150 10950 9150
 $EndSCHEMATC
