File: board/FPGA_Bank_1_2.sch (KiCad schematic (older format))
At the start: 3 parts, among them SW1 SW_PUSH, U10 XC6SLX45T

Commit message: Issue #1713
Connections:
- net ETH_MDIO: now also U10.T8 (*IO_L57P_2); no longer U10.U8 (*IO_L57N_2)
- net ETH_RESET_B: now also U10.U8 (*IO_L57N_2); no longer U10.T8 (*IO_L57P_2)
- net SD_CLK: now also U10.T7 (IO_L64P_D8_2); no longer U10.U6 (IO_L64N_D9_2)
- net SD_CMD: now also U10.U6 (IO_L64N_D9_2); no longer U10.T7 (IO_L64P_D8_2)
- net SD_DAT0: now also U10.AA4 (IO_L63P_2); no longer U10.Y5 (IO_L62P_D5_2)
- net SD_DAT1: now also U10.AB4 (IO_L63N_2); no longer U10.AB5 (IO_L62N_D6_2)
- net SD_DAT2: now also U10.AB5 (IO_L62N_D6_2); no longer U10.AB4 (IO_L63N_2)
- net SD_DAT3: now also U10.Y5 (IO_L62P_D5_2); no longer U10.AA4 (IO_L63P_2)
- net TMDS_RX1_1_N: now also U10.H22 (IO_L37N_A6_M1A1_1); no longer U10.L19 (IO_L38N_A4_M1CLKN_1)
- net TMDS_RX1_1_P: now also U10.H21 (IO_L37P_A7_M1A0_1); no longer U10.K20 (IO_L38P_A5_M1CLK_1)
- net TMDS_RX1_2_N: now also U10.L19 (IO_L38N_A4_M1CLKN_1); no longer U10.H22 (IO_L37N_A6_M1A1_1)
- net TMDS_RX1_2_P: now also U10.K20 (IO_L38P_A5_M1CLK_1); no longer U10.H21 (IO_L37P_A7_M1A0_1)
- net TMDS_RX1_CEC: now also U10.K17 (IO_L36P_A9_M1BA0_1); no longer U10.V19 (IO_L74P_AWAKE_1)
- net TMDS_RX1_HOT: now also U10.V19 (IO_L74P_AWAKE_1); no longer U10.T18 (*IO_L73N_1)
- net TMDS_RX1_SCL: now also U10.L17 (IO_L36N_A8_M1BA1_1); no longer U10.K17 (IO_L36P_A9_M1BA0_1)
- net TMDS_RX1_SDA: now also U10.T18 (*IO_L73N_1); no longer U10.L17 (IO_L36N_A8_M1BA1_1)
- net TMDS_RX2_CEC: now also U10.T22 (IO_L48N_M1DQ9_1); no longer U10.T21 (IO_L48P_HDC_M1DQ8_1)
- net TMDS_RX2_HOT: now also U10.R20 (IO_L47P_FWE_B_M1DQ0_1); no longer U10.T22 (IO_L48N_M1DQ9_1)
- net TMDS_RX2_SCL: now also U10.T21 (IO_L48P_HDC_M1DQ8_1); no longer U10.R20 (IO_L47P_FWE_B_M1DQ0_1)
- net TMDS_TX1_CEC: now also U10.W10 (*IO_L44P_2); no longer U10.Y7 (IO_L47P_2)
- net TMDS_TX1_SCL: now also U10.Y7 (IO_L47P_2); no longer U10.W10 (*IO_L44P_2)
- net TMDS_TX2_CEC: now also U10.AA18 (IO_L14P_D11_2); no longer U10.AB18 (IO_L14N_D12_2)
- net TMDS_TX2_HOT: now also U10.AB18 (IO_L14N_D12_2); no longer U10.AA18 (IO_L14P_D11_2)
- net USB_D2: now also U10.Y18 (*IO_L5N_2); no longer U10.W17 (*IO_L5P_2)
- net USB_D3: now also U10.W17 (*IO_L5P_2); no longer U10.Y18 (*IO_L5N_2)
Changed lines of the file:
@@
 Sheet 12 12
 Title "HDMI2USB"
-Date "2 apr 2015"
+Date "7 apr 2015"
 Rev "Rev2"
 Comp ""
@@
 Text HLabel 6350 9700 2    60   Output ~ 0
 INIT_B
+Text HLabel 6350 9300 2    60   BiDi ~ 0
+SD_DAT0
+Text HLabel 6350 9400 2    60   BiDi ~ 0
+SD_DAT1
+Text HLabel 6200 9200 2    60   BiDi ~ 0
+SD_DAT2
 Text HLabel 6200 9100 2    60   BiDi ~ 0
-SD_DAT0
-Text HLabel 6200 9200 2    60   BiDi ~ 0
-SD_DAT1
-Text HLabel 6350 9400 2    60   BiDi ~ 0
-SD_DAT2
-Text HLabel 6350 9300 2    60   BiDi ~ 0
 SD_DAT3
-Text HLabel 6350 9500 2    60   BiDi ~ 0
+Text HLabel 6350 9600 2    60   BiDi ~ 0
 SD_CMD
-Text HLabel 6350 9600 2    60   Output ~ 0
+Text HLabel 6350 9500 2    60   Output ~ 0
 SD_CLK
 Text HLabel 6100 5600 2    39   Input ~ 0
@@
 	8250 14500 8250 14600
 $Comp
-L GND #PWR053
+L GND #PWR054
 U 1 1 53857D31
 P 8250 14600
-F 0 "#PWR053" H 8250 14600 30  0001 C CNN
+F 0 "#PWR054" H 8250 14600 30  0001 C CNN
 F 1 "GND" H 8250 14530 30  0001 C CNN
 F 2 "" H 8250 14600 60  0000 C CNN
@@
 Text HLabel 6100 6000 2    60   BiDi ~ 0
 TMDS_TX1_CLK_N
-Text HLabel 6100 6900 2    60   BiDi ~ 0
+Text HLabel 6100 7500 2    60   BiDi ~ 0
 TMDS_TX1_SCL
 Text HLabel 6100 7000 2    60   BiDi ~ 0
 TMDS_TX1_SDA
-Text HLabel 6100 7500 2    60   BiDi ~ 0
+Text HLabel 6100 6900 2    60   BiDi ~ 0
 TMDS_TX1_CEC
 Text HLabel 6100 7600 2    60   BiDi ~ 0
@@
 Text HLabel 6100 3600 2    60   BiDi ~ 0
 TMDS_TX2_SDA
+Text HLabel 6100 3300 2    60   BiDi ~ 0
+TMDS_TX2_CEC
 Text HLabel 6100 3400 2    60   BiDi ~ 0
-TMDS_TX2_CEC
-Text HLabel 6100 3300 2    60   BiDi ~ 0
 TMDS_TX2_HOT
 Text HLabel 12450 5150 2    60   BiDi ~ 0
@@
 Text HLabel 12450 5250 2    60   BiDi ~ 0
 TMDS_RX1_0_N
+Text HLabel 12450 4750 2    60   BiDi ~ 0
+TMDS_RX1_1_P
+Text HLabel 12450 4850 2    60   BiDi ~ 0
+TMDS_RX1_1_N
 Text HLabel 12450 4950 2    60   BiDi ~ 0
-TMDS_RX1_1_P
+TMDS_RX1_2_P
 Text HLabel 12450 5050 2    60   BiDi ~ 0
-TMDS_RX1_1_N
-Text HLabel 12450 4750 2    60   BiDi ~ 0
-TMDS_RX1_2_P
-Text HLabel 12450 4850 2    60   BiDi ~ 0
 TMDS_RX1_2_N
 Text HLabel 12450 5350 2    60   BiDi ~ 0
@@
 Text HLabel 12450 5450 2    60   BiDi ~ 0
 TMDS_RX1_CLK_N
+Text HLabel 12450 4650 2    60   BiDi ~ 0
+TMDS_RX1_SCL
+Text HLabel 13300 9650 2    60   BiDi ~ 0
+TMDS_RX1_SDA
 Text HLabel 12450 4550 2    60   BiDi ~ 0
-TMDS_RX1_SCL
-Text HLabel 12450 4650 2    60   BiDi ~ 0
-TMDS_RX1_SDA
+TMDS_RX1_CEC
 Text HLabel 13300 9750 2    60   BiDi ~ 0
-TMDS_RX1_CEC
-Text HLabel 13300 9650 2    60   BiDi ~ 0
 TMDS_RX1_HOT
 Text HLabel 12450 6150 2    60   BiDi ~ 0
@@
 Text HLabel 12450 6050 2    60   BiDi ~ 0
 TMDS_RX2_CLK_N
-Text HLabel 12450 6750 2    60   BiDi ~ 0
+Text HLabel 12450 6950 2    60   BiDi ~ 0
 TMDS_RX2_SCL
 Text HLabel 12450 6850 2    60   BiDi ~ 0
 TMDS_RX2_SDA
-Text HLabel 12450 6950 2    60   BiDi ~ 0
+Text HLabel 12450 7050 2    60   BiDi ~ 0
 TMDS_RX2_CEC
-Text HLabel 12450 7050 2    60   BiDi ~ 0
+Text HLabel 12450 6750 2    60   BiDi ~ 0
 TMDS_RX2_HOT
 Text HLabel 12450 5750 2    39   BiDi ~ 0
@@
 Text HLabel 6100 8500 2    47   Input ~ 0
 ETH_MDC
+Text HLabel 6100 8300 2    47   Input ~ 0
+ETH_MDIO
 Text HLabel 6100 8400 2    47   Input ~ 0
-ETH_MDIO
-Text HLabel 6100 8300 2    47   Input ~ 0
 ETH_RESET_B
 Text HLabel 6100 8200 2    47   Input ~ 0
@@
 Text Label 7150 2400 0    39   ~ 0
 USB_D1
+Text Label 7150 2600 0    39   ~ 0
+USB_D2
 Text Label 7150 2500 0    39   ~ 0
-USB_D2
-Text Label 7150 2600 0    39   ~ 0
 USB_D3
 Text Label 7150 2700 0    39   ~ 0
