File: board/FPGA_Power.sch (KiCad schematic (older format))
At the start: 67 parts, among them U10 XC6SLX150T

Commit message: Issue #1683
Parts:
- U10: value XC6SLX150T -> XC6SLX45T
Changed lines of the file:
@@
 $Descr A2 23386 16535
 encoding utf-8
-Sheet 4 12
+Sheet 3 12
 Title "HDMI2USB"
-Date "23 mar 2015"
+Date "25 mar 2015"
 Rev "Rev2"
 Comp ""
@@
 P 5450 4750
 F 0 "U10" H 4500 8800 60  0000 C CNN
-F 1 "XC6SLX150T" H 4800 -2550 60  0000 C CNN
+F 1 "XC6SLX45T" H 4800 -2550 60  0000 C CNN
 F 2 "~" H 5500 4750 60  0000 C CNN
 F 3 "~" H 5500 4750 60  0000 C CNN
@@
 P 17400 7900
 F 0 "U10" H 16450 11950 60  0000 C CNN
-F 1 "XC6SLX150T" H 16750 600 60  0000 C CNN
+F 1 "XC6SLX45T" H 16750 600 60  0000 C CNN
 F 2 "~" H 17450 7900 60  0000 C CNN
 F 3 "~" H 17450 7900 60  0000 C CNN
