File: board/FPGA_Power.sch (KiCad schematic (older format))
At the start: 67 parts, among them U10 XC6SLX45T

Commit message: Issue #1647 - Final changes
Parts:
- removed C100, C104, C106: 0.1UF, symbol C
Connections:
- net GND: now also C108.1, C110.1, C112.1, C114.1, C116.1, C118.1; no longer C108.2, C110.2, C112.2, C114.2, C116.2, C118.2
- net VCC1V5: no longer C108.1, C110.1, C112.1, C114.1, C116.1, C118.1
- net VCC3V3: now also C108.2, C110.2, C112.2, C114.2, C116.2, C118.2
Other:
- moved on the sheet: C102, C108, C110, C112, C114, C116, C118, C127
Changed lines of the file:
@@
 $EndComp
 $Comp
-L C C100
-U 1 1 52DE5492
+L C C102
+U 1 1 52DE5498
 P 11200 14400
-F 0 "C100" H 11250 14500 50  0000 L CNN
+F 0 "C102" H 11250 14500 50  0000 L CNN
 F 1 "0.1UF" H 11200 14300 50  0000 L CNN
 F 2 "" H 11200 14400 60  0000 C CNN
@@
 $EndComp
 $Comp
-L C C102
-U 1 1 52DE5498
-P 11450 14400
-F 0 "C102" H 11500 14500 50  0000 L CNN
-F 1 "0.1UF" H 11450 14300 50  0000 L CNN
-F 2 "" H 11450 14400 60  0000 C CNN
-F 3 "" H 11450 14400 60  0000 C CNN
-	1    11450 14400
-	1    0    0    -1
-$EndComp
-$Comp
-L C C104
-U 1 1 52DE549E
-P 11700 14400
-F 0 "C104" H 11750 14500 50  0000 L CNN
-F 1 "0.1UF" H 11700 14300 50  0000 L CNN
-F 2 "" H 11700 14400 60  0000 C CNN
-F 3 "" H 11700 14400 60  0000 C CNN
-	1    11700 14400
-	1    0    0    -1
-$EndComp
-$Comp
-L C C106
-U 1 1 52DE54F4
-P 11950 14400
-F 0 "C106" H 12000 14500 50  0000 L CNN
-F 1 "0.1UF" H 11950 14300 50  0000 L CNN
-F 2 "" H 11950 14400 60  0000 C CNN
-F 3 "" H 11950 14400 60  0000 C CNN
-	1    11950 14400
-	1    0    0    -1
-$EndComp
-$Comp
 L C C108
 U 1 1 52DE54FA
-P 12200 14400
-F 0 "C108" H 12250 14500 50  0000 L CNN
-F 1 "0.1UF" H 12200 14300 50  0000 L CNN
-F 2 "" H 12200 14400 60  0000 C CNN
-F 3 "" H 12200 14400 60  0000 C CNN
-	1    12200 14400
+P 14950 14850
+F 0 "C108" H 15000 14950 50  0000 L CNN
+F 1 "0.1UF" H 14950 14750 50  0000 L CNN
+F 2 "" H 14950 14850 60  0000 C CNN
+F 3 "" H 14950 14850 60  0000 C CNN
+	1    14950 14850
 	1    0    0    -1
 $EndComp
@@
 L C C110
 U 1 1 52DE5500
-P 12450 14400
-F 0 "C110" H 12500 14500 50  0000 L CNN
-F 1 "0.1UF" H 12450 14300 50  0000 L CNN
-F 2 "" H 12450 14400 60  0000 C CNN
-F 3 "" H 12450 14400 60  0000 C CNN
-	1    12450 14400
+P 15200 14850
+F 0 "C110" H 15250 14950 50  0000 L CNN
+F 1 "0.1UF" H 15200 14750 50  0000 L CNN
+F 2 "" H 15200 14850 60  0000 C CNN
+F 3 "" H 15200 14850 60  0000 C CNN
+	1    15200 14850
 	1    0    0    -1
 $EndComp
@@
 L C C112
 U 1 1 52DE5506
-P 12700 14400
-F 0 "C112" H 12750 14500 50  0000 L CNN
-F 1 "0.1UF" H 12700 14300 50  0000 L CNN
-F 2 "" H 12700 14400 60  0000 C CNN
-F 3 "" H 12700 14400 60  0000 C CNN
-	1    12700 14400
+P 15450 14850
+F 0 "C112" H 15500 14950 50  0000 L CNN
+F 1 "0.1UF" H 15450 14750 50  0000 L CNN
+F 2 "" H 15450 14850 60  0000 C CNN
+F 3 "" H 15450 14850 60  0000 C CNN
+	1    15450 14850
 	1    0    0    -1
 $EndComp
@@
 L C C114
 U 1 1 52DE550C
-P 12950 14400
-F 0 "C114" H 13000 14500 50  0000 L CNN
-F 1 "0.1UF" H 12950 14300 50  0000 L CNN
-F 2 "" H 12950 14400 60  0000 C CNN
-F 3 "" H 12950 14400 60  0000 C CNN
-	1    12950 14400
+P 15700 14850
+F 0 "C114" H 15750 14950 50  0000 L CNN
+F 1 "0.1UF" H 15700 14750 50  0000 L CNN
+F 2 "" H 15700 14850 60  0000 C CNN
+F 3 "" H 15700 14850 60  0000 C CNN
+	1    15700 14850
 	1    0    0    -1
 $EndComp
@@
 	9200 14200 9200 14150
 Wire Wire Line
-	13200 14150 13200 14200
-Wire Wire Line
-	12950 14200 12950 14150
-Connection ~ 12950 14150
-Wire Wire Line
-	12700 14200 12700 14150
-Connection ~ 12700 14150
-Wire Wire Line
-	12450 14200 12450 14150
-Connection ~ 12450 14150
-Wire Wire Line
-	12200 14200 12200 14150
-Connection ~ 12200 14150
-Wire Wire Line
-	11950 14200 11950 14150
-Connection ~ 11950 14150
-Wire Wire Line
-	11700 14200 11700 14150
-Connection ~ 11700 14150
-Wire Wire Line
-	11450 14200 11450 14150
-Connection ~ 11450 14150
+	11450 14150 11450 14200
 Wire Wire Line
 	11200 14200 11200 14150
@@
 	11450 14650 11450 14600
 Connection ~ 11450 14650
-Wire Wire Line
-	11700 14650 11700 14600
 Connection ~ 11700 14650
-Wire Wire Line
-	11950 14650 11950 14600
 Connection ~ 11950 14650
-Wire Wire Line
-	12200 14650 12200 14600
 Connection ~ 12200 14650
-Wire Wire Line
-	12450 14650 12450 14600
 Connection ~ 12450 14650
-Wire Wire Line
-	12700 14650 12700 14600
 Connection ~ 12700 14650
-Wire Wire Line
-	12950 14650 12950 14600
 Connection ~ 12950 14650
-Wire Wire Line
-	13200 14650 13200 14600
 Wire Wire Line
 	12200 15150 12200 15050
@@
 L C C127
 U 1 1 52DEC671
-P 13700 14400
-F 0 "C127" H 13750 14500 50  0000 L CNN
-F 1 "0.1UF" H 13700 14300 50  0000 L CNN
-F 2 "" H 13700 14400 60  0000 C CNN
-F 3 "" H 13700 14400 60  0000 C CNN
-	1    13700 14400
+P 11450 14400
+F 0 "C127" H 11500 14500 50  0000 L CNN
+F 1 "0.1UF" H 11450 14300 50  0000 L CNN
+F 2 "" H 11450 14400 60  0000 C CNN
+F 3 "" H 11450 14400 60  0000 C CNN
+	1    11450 14400
 	1    0    0    -1
 $EndComp
@@
 L C C116
 U 1 1 52DEC9D2
-P 13200 14400
-F 0 "C116" H 13250 14500 50  0000 L CNN
-F 1 "0.1UF" H 13200 14300 50  0000 L CNN
-F 2 "" H 13200 14400 60  0000 C CNN
-F 3 "" H 13200 14400 60  0000 C CNN
-	1    13200 14400
+P 15950 14850
+F 0 "C116" H 16000 14950 50  0000 L CNN
+F 1 "0.1UF" H 15950 14750 50  0000 L CNN
+F 2 "" H 15950 14850 60  0000 C CNN
+F 3 "" H 15950 14850 60  0000 C CNN
+	1    15950 14850
 	1    0    0    -1
 $EndComp
@@
 L C C118
 U 1 1 52DEC9D8
-P 13450 14400
-F 0 "C118" H 13500 14500 50  0000 L CNN
-F 1 "0.1UF" H 13450 14300 50  0000 L CNN
-F 2 "" H 13450 14400 60  0000 C CNN
-F 3 "" H 13450 14400 60  0000 C CNN
-	1    13450 14400
+P 16200 14850
+F 0 "C118" H 16250 14950 50  0000 L CNN
+F 1 "0.1UF" H 16200 14750 50  0000 L CNN
+F 2 "" H 16200 14850 60  0000 C CNN
+F 3 "" H 16200 14850 60  0000 C CNN
+	1    16200 14850
 	1    0    0    -1
 $EndComp
@@
 $EndComp
 Wire Wire Line
-	13450 14600 13450 14650
-Wire Wire Line
-	13700 14600 13700 14650
-Wire Wire Line
 	14700 14650 14700 14600
 Wire Wire Line
@@
 Connection ~ 14950 14650
 Wire Wire Line
-	13450 14150 13450 14200
-Wire Wire Line
 	16200 14150 16200 14200
-Wire Wire Line
-	13700 14150 13700 14200
 Wire Wire Line
 	14700 14200 14700 14150
@@
 	2150 15100 2300 15100
 Connection ~ 2150 14950
-Connection ~ 13200 14150
-Connection ~ 13700 14150
-Connection ~ 13450 14150
 Wire Wire Line
 	14200 14150 17200 14150
@@
 $EndComp
 Wire Wire Line
-	8550 15150 14700 15150
+	8550 15150 16200 15150
 Wire Wire Line
 	14200 14650 14700 14650
@@
 	14450 14200 14450 14150
 Connection ~ 14700 14150
-Wire Wire Line
-	9050 14150 13700 14150
 Wire Wire Line
 	14200 14150 14200 14200
@@
 Text HLabel 1600 14650 0    50   Input ~ 10
 DONE
+Wire Wire Line
+	14950 15150 14950 15050
+Connection ~ 14700 15150
+Wire Wire Line
+	15200 15150 15200 15050
+Connection ~ 14950 15150
+Wire Wire Line
+	15450 15150 15450 15050
+Connection ~ 15200 15150
+Wire Wire Line
+	15700 15150 15700 15050
+Connection ~ 15450 15150
+Wire Wire Line
+	15950 15150 15950 15050
+Connection ~ 15700 15150
+Wire Wire Line
+	16200 15150 16200 15050
+Connection ~ 15950 15150
+Wire Wire Line
+	9050 14150 11450 14150
 $EndSCHEMATC

Commit message: Issue #1961 - Adding initial "populate" field to all components.
Parts:
- C101, C102, C103, C105, C107, C108, C109, C110, C111, C112, C114, C115, C116, C117, C118, C119, C120, C121, C122, C123, C124, C125, C126, C127, C128, C129, C130, C131, C190, C213, C215, C221, C236, C237, C242, C243, C82, C83, C84, C85, C86, C87, C88, C89, C90, C91, C92, C93, C94, C95, C96, C97, C98, C99, D1, R29, R52, R53, R55, R56, R57, R58, R59, U10: Populate (none) -> Yes
