File: board/SPI.sch (KiCad schematic (older format))
At the start: 28 parts, among them P3 CONN_7X2, U11 MICRO_SD, U17 FXO-HC536R, U3 W25Q128FVEIG

Commit message: Issue #1585
Parts:
- added C241: 0.1UF, symbol C
- added C244: 15PF, symbol C
- added P14: CONN_5X2, symbol CONN_5X2
- added R116, R118, R119, R93: 1K, symbol R
- added R117: 1M, symbol R
- added R86: 4K7, symbol R
- added SW2: SW_PUSH, ~, symbol SW_PUSH
- added U26: CB3LV-3I-27M0000, ~, symbol FXO-HC536R
Connections:
- net GND: now also C241.1, C244.1, R116.1, R119.2, U26.2 (GND)
- net VCC3V3: now also C241.2, R86.1, U26.4 (VCC)
- new net: R86.2, U26.1 (E/D)
- new net: P14.1, R93.2
- new net: P14.2, R118.1
- new net: P14.5, R116.2
- new net: P14.7, SW2.1
- new net: P14.8, R119.1, SW2.2
- new net 27MHz: C244.2, U26.3 (OUT)
- new net PCIO0: R118.2
- new net PCIO1: P14.3
- new net PCIO2: P14.4
- new net PCIO3: P14.6, R117.1
- new net VCC1V5: R117.2, R93.1
- no-connect marks 2 -> 4
Other:
- note added: "27MHz"
- moved on the sheet: C188, C189, JP1, JP2, P3, R40, R41, R76, R80, R81, R82, R83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

Commit message: Issue #1647 - Final changes
Parts:
- removed SW2: SW_PUSH, ~, symbol SW_PUSH
Connections:
- net CYPRESS_RESET: now reaches P14.7
Changed lines of the file:
@@
 LIBS:contrib
 LIBS:valves
+LIBS:hdmi2usb
+LIBS:timvideos-pcie-8x
 LIBS:HDMI2USB-cache
 EELAYER 27 0
@@
 Sheet 4 12
 Title "HDMI2USB"
-Date "1 apr 2015"
+Date "2 apr 2015"
 Rev "Rev2"
 Comp ""
@@
 	1    0    0    -1
 $EndComp
-$Comp
-L SW_PUSH SW2
-U 1 1 551DEF80
-P 9150 6400
-F 0 "SW2" H 9300 6510 50  0000 C CNN
-F 1 "SW_PUSH" H 9150 6320 50  0000 C CNN
-F 2 "~" H 9150 6400 60  0000 C CNN
-F 3 "~" H 9150 6400 60  0000 C CNN
-	1    9150 6400
-	1    0    0    -1
-$EndComp
-Wire Wire Line
-	9700 5900 9700 6400
-Wire Wire Line
-	9700 6400 9450 6400
-Wire Wire Line
-	8850 6400 8700 6400
-Wire Wire Line
-	8700 6400 8700 5900
 Wire Wire Line
 	8700 5900 8800 5900
@@
 Text HLabel 10450 5800 2    39   BiDi ~ 0
 PCIO3
+Text HLabel 8700 5900 0    39   Output ~ 0
+CYPRESS_RESET
 $EndSCHEMATC
