File: board/HDMI.sch (KiCad schematic (older format))
At the start: 82 parts, among them J2 HDMI, J3 HDMI, J4 HDMI, J5 HDMI, P10 CONN_1, P2 CONN_1, P4 CONN_1, P5 CONN_1, P6 CONN_1, P7 CONN_1, P8 CONN_1, P9 CONN_1, U13 IP4776CZ38, U14 IP4776CZ38, U15 IP4776CZ38, U16 ΜA78L00, U21 IP4776CZ38, U22 ΜA78L00

Commit message: Issue #1647 - Final changes
Parts:
- added C251: 0.33mfd, ~, symbol C
- added C252, C253, C254: 0.1mfd, ~, symbol C
- added R121, R122: 100K, ~, symbol R
- added U30, U31: ΜA78L00, symbol ΜA78L00
- C183: value 0.1mfd -> 0.33mfd
Connections:
- net GND: no longer C183.2, C205.2, C206.2, C208.2
- net HDMI-TX1-VCC5V0: now also C205.1, U13.1 (VCC(5V0))
- net HDMI-TX2-VCC5V0: now also U14.1 (VCC(5V0)), C252.1
- net VCC12V0: now also C183.1, C251.1, U30.3 (IN), U31.3 (IN)
- net VCC5V0: no longer C183.1, C205.1, C206.1, C208.1, U13.1 (VCC(5V0)), U14.1 (VCC(5V0)), U15.1 (VCC(5V0)), U21.1 (VCC(5V0))
- net at C173.2, C175.2, R195.2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: now also C205.2
- net at C177.2, C181.2, R202.2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: now also C252.2
- new net: C183.2, C206.2, C208.2, R121.2, U30.2 (C)
- new net: C251.2, C253.2, C254.2, R122.2, U31.2 (C)
- new net HDMI-RX1-VCC5V0: C206.1, C208.1, R121.1, U15.1 (VCC(5V0)), U30.1 (OUT)
- new net HDMI-RX2-VCC5V0: C253.1, C254.1, R122.1, U21.1 (VCC(5V0)), U31.1 (OUT)

Commit message: Issue #1713
Parts:
- removed C251: 0.33mfd, ~, symbol C
- removed C253, C254: 0.1mfd, ~, symbol C
- removed R122: 100K, ~, symbol R
- removed U31: ΜA78L00, symbol ΜA78L00
Connections:
- net HDMI-RX2-VCC5V0 is gone; now on net HDMI_VCC5V0: U21.1 (VCC(5V0))
- net HDMI-TX1-VCC5V0: no longer U13.1 (VCC(5V0))
- net HDMI-TX2-VCC5V0: no longer U14.1 (VCC(5V0))
- net HDMI-RX1-VCC5V0 renamed HDMI_VCC5V0
- net HDMI_VCC5V0: now also U13.1 (VCC(5V0)), U14.1 (VCC(5V0))
Changed lines of the file:
@@
 Sheet 7 12
 Title "HDMI2USB"
-Date "2 apr 2015"
+Date "7 apr 2015"
 Rev "Rev2"
 Comp ""
@@
 $EndComp
 Text Label 10850 7750 2    39   ~ 0
-HDMI-RX1-VCC5V0
+HDMI_VCC5V0
 $Comp
 L C C183
@@
 	1    0    0    -1
 $EndComp
-Text Label 11050 7700 0    39   ~ 0
-VCC12V0
-$Comp
-L ΜA78L00 U31
-U 1 1 551E1F04
-P 12050 7700
-F 0 "U31" H 12350 7400 60  0000 C CNN
-F 1 "ΜA78L00" H 11900 7950 60  0000 C CNN
-F 2 "" H 12050 7700 60  0000 C CNN
-F 3 "" H 12050 7700 60  0000 C CNN
-	1    12050 7700
-	1    0    0    -1
-$EndComp
-Text Label 13150 7700 2    39   ~ 0
-HDMI-RX2-VCC5V0
-$Comp
-L C C251
-U 1 1 551E1F0B
-P 11300 8000
-F 0 "C251" H 11300 8100 40  0000 L CNN
-F 1 "0.33mfd" H 11306 7915 40  0000 L CNN
-F 2 "~" H 11338 7850 30  0000 C CNN
-F 3 "~" H 11300 8000 60  0000 C CNN
-	1    11300 8000
-	1    0    0    -1
-$EndComp
-$Comp
-L C C254
-U 1 1 551E1F11
-P 12750 8100
-F 0 "C254" H 12750 8200 40  0000 L CNN
-F 1 "0.1mfd" H 12756 8015 40  0000 L CNN
-F 2 "~" H 12788 7950 30  0000 C CNN
-F 3 "~" H 12750 8100 60  0000 C CNN
-	1    12750 8100
-	1    0    0    -1
-$EndComp
-$Comp
-L R R122
-U 1 1 551E1F17
-P 13050 8100
-F 0 "R122" V 13100 7900 40  0000 C CNN
-F 1 "100K" V 13057 8101 40  0000 C CNN
-F 2 "~" V 12980 8100 30  0000 C CNN
-F 3 "~" H 13050 8100 30  0000 C CNN
-	1    13050 8100
-	1    0    0    -1
-$EndComp
 Text Notes 8750 7300 0    39   ~ 0
 LDO OUT FOR
-Text Notes 11050 7300 0    39   ~ 0
-LDO OUT FOR
-Text Notes 11500 7300 0    39   ~ 0
-HDMI IN 2
 Text Notes 9200 7300 0    39   ~ 0
 HDMI IN 1
@@
 	10750 8550 10750 8400
 Connection ~ 10450 8550
-Wire Wire Line
-	11050 7700 11400 7700
-Wire Wire Line
-	12700 7700 13150 7700
-Wire Wire Line
-	11300 7800 11300 7700
-Connection ~ 11300 7700
-Wire Wire Line
-	12050 8250 12050 8500
-Wire Wire Line
-	11300 8500 13050 8500
-Wire Wire Line
-	11300 8500 11300 8200
-Wire Wire Line
-	12750 8300 12750 8500
-Connection ~ 12050 8500
-Wire Wire Line
-	12750 7900 12750 7700
-Connection ~ 12750 7700
-Wire Wire Line
-	13050 7850 13050 7700
-Connection ~ 13050 7700
-Wire Wire Line
-	13050 8500 13050 8350
-Connection ~ 12750 8500
-Wire Notes Line
-	8350 7200 13250 7200
-Wire Notes Line
-	13250 7200 13250 8700
-Wire Notes Line
-	13250 8700 8700 8700
-Wire Notes Line
-	10950 7200 10950 8700
-Wire Notes Line
-	10950 8700 11000 8700
+Wire Notes Line
+	10950 8700 10950 7200
 Wire Notes Line
 	8350 7300 9950 7300
 Wire Notes Line
 	9950 7300 9950 7200
-Wire Notes Line
-	10950 7300 12050 7300
-Wire Notes Line
-	12050 7300 12050 7200
 Text GLabel 8750 7750 0    39   Input ~ 0
 VCC12V0
@@
 	8350 7200 8350 8700
 Wire Notes Line
-	8350 8700 8750 8700
+	8350 8700 10950 8700
 $Comp
 L C C206
@@
 	10250 8350 10250 8550
 Connection ~ 10250 8550
-$Comp
-L C C253
-U 1 1 551E1F56
-P 12500 8100
-F 0 "C253" H 12500 8200 40  0000 L CNN
-F 1 "0.1mfd" H 12506 8015 40  0000 L CNN
-F 2 "~" H 12538 7950 30  0000 C CNN
-F 3 "~" H 12500 8100 60  0000 C CNN
-	1    12500 8100
-	1    0    0    -1
-$EndComp
-Wire Wire Line
-	12500 7900 12500 7800
-Wire Wire Line
-	12500 7800 12750 7800
-Connection ~ 12750 7800
-Wire Wire Line
-	12500 8300 12500 8500
-Connection ~ 12500 8500
+Text Label 1700 8250 0    39   ~ 0
+HDMI_VCC5V0
+Text Label 2000 1700 0    39   ~ 0
+HDMI_VCC5V0
 Text Label 9750 1650 0    39   ~ 0
-HDMI-RX2-VCC5V0
-Text Label 2000 1700 0    39   ~ 0
-HDMI-RX1-VCC5V0
+HDMI_VCC5V0
+Wire Notes Line
+	10950 7200 8350 7200
 Text Label 1700 5050 0    39   ~ 0
-HDMI-TX1-VCC5V0
-Text Label 1700 8250 0    39   ~ 0
-HDMI-TX2-VCC5V0
+HDMI_VCC5V0
 $EndSCHEMATC

Commit message: Issue #1647 - Final changes
Connections:
- net VCC5V0 is gone; now on net HDMI_VCC5V0: R137.1, R138.1, R139.1, R140.1, R141.1, R142.1, R153.1, R196.1, R197.1, R205.1
Other:
- note added: "LDO FOR IP4776CZ38"
Changed lines of the file:
@@
 	-1   0    0    1
 $EndComp
-Text Label 4850 10800 2    60   ~ 0
-VCC5V0
 $Comp
 L R R129
@@
 	-1   0    0    1
 $EndComp
-Text Label 4850 7550 2    60   ~ 0
-VCC5V0
 $Comp
 L R R148
@@
 	-1   0    0    1
 $EndComp
-Text Label 5100 4450 2    60   ~ 0
-VCC5V0
 $Comp
 L R R151
@@
 	-1   0    0    1
 $EndComp
-Text Label 12850 4400 2    60   ~ 0
-VCC5V0
 $Comp
 L R R204
@@
 	-1   0    0    1
 $EndComp
-Text Label 6250 4300 0    60   ~ 0
-VCC5V0
 $Comp
 L R R205
@@
 	-1   0    0    1
 $EndComp
-Text Label 13750 4200 0    60   ~ 0
-VCC5V0
 $Comp
 L ΜA78L00 U16
@@
 	4350 10650 4350 10800
 Wire Wire Line
-	4350 10800 4850 10800
+	4350 10800 4900 10800
 Wire Wire Line
 	4500 10650 4500 10800
@@
 	4350 7400 4350 7550
 Wire Wire Line
-	4350 7550 4850 7550
+	4350 7550 4950 7550
 Wire Wire Line
 	4500 7400 4500 7550
@@
 	4600 4300 4600 4450
 Wire Wire Line
-	4600 4450 5100 4450
+	4600 4450 5150 4450
 Wire Wire Line
 	4750 4300 4750 4450
@@
 	12350 4250 12350 4400
 Wire Wire Line
-	12350 4400 12850 4400
+	12350 4400 12900 4400
 Wire Wire Line
 	12500 4250 12500 4400
@@
 $EndComp
 Text Notes 8750 7300 0    39   ~ 0
-LDO OUT FOR
-Text Notes 9200 7300 0    39   ~ 0
-HDMI IN 1
+LDO FOR IP4776CZ38
 Wire Wire Line
 	8750 7750 9100 7750
@@
 Text Label 1700 5050 0    39   ~ 0
 HDMI_VCC5V0
+Text Label 4900 10800 2    39   ~ 0
+HDMI_VCC5V0
+Text Label 4950 7550 2    39   ~ 0
+HDMI_VCC5V0
+Text Label 5150 4450 2    39   ~ 0
+HDMI_VCC5V0
+Text Label 6250 4300 0    39   ~ 0
+HDMI_VCC5V0
+Text Label 12900 4400 2    39   ~ 0
+HDMI_VCC5V0
+Text Label 13750 4200 0    39   ~ 0
+HDMI_VCC5V0
 $EndSCHEMATC
