File: board/HDMI.sch (KiCad schematic (older format))
At the start: 85 parts, among them J2 HDMI, J3 HDMI, J4 HDMI, J5 HDMI, P10 CONN_1, P2 CONN_1, P4 CONN_1, P5 CONN_1, P6 CONN_1, P7 CONN_1, P8 CONN_1, P9 CONN_1, U13 IP4776CZ38, U14 IP4776CZ38, U15 IP4776CZ38, U16 ΜA78L00, U21 IP4776CZ38, U22 ΜA78L00, U30 ΜA78L00

Commit message: Issue #1804 - Adding RX/TX direction fields.
Parts:
- J2, J5: Direction (none) -> TX
- J3, J4: Direction (none) -> RX
Changed lines of the file:
@@
 F 2 "~" H 7900 2750 60  0000 C CNN
 F 3 "~" H 7900 2750 60  0000 C CNN
+F 4 "RX" H 7900 2750 60  0001 C CNN "Direction"
 	1    7950 2750
 	1    0    0    -1
@@
 F 2 "~" H 7650 6000 60  0000 C CNN
 F 3 "~" H 7650 6000 60  0000 C CNN
+F 4 "RX" H 7650 6000 60  0001 C CNN "Direction"
 	1    7700 6000
 	1    0    0    -1
@@
 F 2 "~" H 7550 9150 60  0000 C CNN
 F 3 "~" H 7550 9150 60  0000 C CNN
+F 4 "TX" H 7550 9150 60  0001 C CNN "Direction"
 	1    7600 9150
 	1    0    0    -1
@@
 F 2 "~" H 15450 2700 60  0000 C CNN
 F 3 "~" H 15450 2700 60  0000 C CNN
+F 4 "TX" H 15450 2700 60  0001 C CNN "Direction"
 	1    15500 2700
 	1    0    0    -1

Commit message: Issue #1804 - Fixing RX/TX direction fields.
Parts:
- J3: Direction RX -> TX
- J5: Direction TX -> RX
Changed lines of the file:
@@
 F 2 "~" H 7650 6000 60  0000 C CNN
 F 3 "~" H 7650 6000 60  0000 C CNN
-F 4 "RX" H 7650 6000 60  0001 C CNN "Direction"
+F 4 "TX" H 7650 6000 60  0001 C CNN "Direction"
 	1    7700 6000
 	1    0    0    -1
@@
 F 2 "~" H 15450 2700 60  0000 C CNN
 F 3 "~" H 15450 2700 60  0000 C CNN
-F 4 "TX" H 15450 2700 60  0001 C CNN "Direction"
+F 4 "RX" H 15450 2700 60  0001 C CNN "Direction"
 	1    15500 2700
 	1    0    0    -1

Commit message: Issue #1849 - Gerber files
Parts:
- J2, J3: Direction TX -> (none)
- J4, J5: Direction RX -> (none)
Changed lines of the file:
@@
 F 2 "~" H 7900 2750 60  0000 C CNN
 F 3 "~" H 7900 2750 60  0000 C CNN
-F 4 "RX" H 7900 2750 60  0001 C CNN "Direction"
 	1    7950 2750
 	1    0    0    -1
@@
 F 2 "~" H 7650 6000 60  0000 C CNN
 F 3 "~" H 7650 6000 60  0000 C CNN
-F 4 "TX" H 7650 6000 60  0001 C CNN "Direction"
 	1    7700 6000
 	1    0    0    -1
@@
 F 2 "~" H 7550 9150 60  0000 C CNN
 F 3 "~" H 7550 9150 60  0000 C CNN
-F 4 "TX" H 7550 9150 60  0001 C CNN "Direction"
 	1    7600 9150
 	1    0    0    -1
@@
 F 2 "~" H 15450 2700 60  0000 C CNN
 F 3 "~" H 15450 2700 60  0000 C CNN
-F 4 "RX" H 15450 2700 60  0001 C CNN "Direction"
 	1    15500 2700
 	1    0    0    -1
